File: pt.kicad_sch (KiCad schematic)
At the start: 7 parts, among them J5 PT

Commit message: Lots of cleanup and updates; Waiting on PR approval for GPS filter
Parts:
- renumbered C38 to C46, D19 to D21, J5 to J10, U22 to U25

Commit message: 8.02 Update; Also changed VRMs and added some notes
Parts:
- renumbered C46 to C39, D21 to D16, J10 to J6, R52 to R68, R53 to R69, R54 to R70, U25 to U29

Commit message: ECU essentially reviewable
Parts:
- renumbered D16 to D23, R68 to R72, R69 to R73, R70 to R74, U29 to U28

Commit message: addressed PR comments
Parts:
- renumbered D23 to D22

Commit message: Updated schematic with IOC
Parts:
- J6: footprint TerminalBlock:TerminalBlock_bornier-3_P5.08mm -> Connector_PinHeader_2.54mm:PinHeader_1x03_P2.54mm_Vertical
Changed lines of the file:
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@@
 			)
 		)
-		(property "Footprint" "TerminalBlock:TerminalBlock_bornier-3_P5.08mm"
+		(property "Footprint" "Connector_PinHeader_2.54mm:PinHeader_1x03_P2.54mm_Vertical"
 			(at 102.87 92.71 0)
 			(effects
