File: rocket2-ecu.kicad_pcb (KiCad board)
At the start: 4 copper layers, 0 parts

Commit message: Add PCB outline
Parts:
- added REF**: MountingHole_4.3mm_M4_Pad_Via, MountingHole:MountingHole_4.3mm_M4_Pad_Via, F.Cu at (215.0, 60.0)
- added REF**: MountingHole_4.3mm_M4_Pad_Via, MountingHole:MountingHole_4.3mm_M4_Pad_Via, F.Cu at (85.0, 60.0)
- added REF**: MountingHole_4.3mm_M4_Pad_Via, MountingHole:MountingHole_4.3mm_M4_Pad_Via, F.Cu at (215.0, 140.0)
- added REF**: MountingHole_4.3mm_M4_Pad_Via, MountingHole:MountingHole_4.3mm_M4_Pad_Via, F.Cu at (85.0, 140.0)
Other:
- board outline added: 150 x 100 mm
Changed lines of the file:
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@@
   )
   (net 0 "")
+  (footprint "MountingHole:MountingHole_4.3mm_M4_Pad_Via" (layer "F.Cu")
+    (at 215 60)
+    (descr "Mounting Hole 4.3mm, M4")
+    (tags "mounting hole 4.3mm m4")
+    (attr exclude_from_pos_files exclude_from_bom)
+    (fp_text reference "REF**" (at 0 -5.3) (layer "F.SilkS") hide
+        (effects (font (size 1 1) (thickness 0.15)))
+    )
+    (fp_text value "MountingHole_4.3mm_M4_Pad_Via" (at 0 5.3) (layer "F.Fab")
+        (effects (font (size 1 1) (thickness 0.15)))
+    )
+    (fp_text user "${REFERENCE}" (at 0 0) (layer "F.Fab")
+        (effects (font (size 1 1) (thickness 0.15)))
+    )
+    (fp_circle (center 0 0) (end 4.3 0)
+      (stroke (width 0.15) (type solid)) (fill none) (layer "Cmts.User"))
+    (fp_circle (center 0 0) (end 4.55 0)
+      (stroke (width 0.05) (type solid)) (fill none) (layer "F.CrtYd"))
+    (pad "1" thru_hole circle (at -3.225 0) (size 0.9 0.9) (drill 0.6) (layers "*.Cu" "*.Mask"))
+    (pad "1" thru_hole circle (at -2.280419 -2.280419) (size 0.9 0.9) (drill 0.6) (layers "*.Cu" "*.Mask"))
+    (pad "1" thru_hole circle (at -2.280419 2.280419) (size 0.9 0.9) (drill 0.6) (layers "*.Cu" "*.Mask"))
+    (pad "1" thru_hole circle (at 0 -3.225) (size 0.9 0.9) (drill 0.6) (layers "*.Cu" "*.Mask"))
+    (pad "1" thru_hole circle (at 0 0) (size 8.6 8.6) (drill 4.3) (layers "*.Cu" "*.Mask"))
+    (pad "1" thru_hole circle (at 0 3.225) (size 0.9 0.9) (drill 0.6) (layers "*.Cu" "*.Mask"))
+    (pad "1" thru_hole circle (at 2.280419 -2.280419) (size 0.9 0.9) (drill 0.6) (layers "*.Cu" "*.Mask"))
+    (pad "1" thru_hole circle (at 2.280419 2.280419) (size 0.9 0.9) (drill 0.6) (layers "*.Cu" "*.Mask"))
+    (pad "1" thru_hole circle (at 3.225 0) (size 0.9 0.9) (drill 0.6) (layers "*.Cu" "*.Mask"))
+  )
+  (footprint "MountingHole:MountingHole_4.3mm_M4_Pad_Via" (layer "F.Cu")
+    (at 85 60)
+    (descr "Mounting Hole 4.3mm, M4")
+    (tags "mounting hole 4.3mm m4")
+    (attr exclude_from_pos_files exclude_from_bom)
+    (fp_text reference "REF**" (at 0 -5.3) (layer "F.SilkS") hide
+        (effects (font (size 1 1) (thickness 0.15)))
+    )
+    (fp_text value "MountingHole_4.3mm_M4_Pad_Via" (at 0 5.3) (layer "F.Fab")
+        (effects (font (size 1 1) (thickness 0.15)))
+    )
+    (fp_text user "${REFERENCE}" (at 0 0) (layer "F.Fab")
+        (effects (font (size 1 1) (thickness 0.15)))
+    )
+    (fp_circle (center 0 0) (end 4.3 0)
+      (stroke (width 0.15) (type solid)) (fill none) (layer "Cmts.User"))
+    (fp_circle (center 0 0) (end 4.55 0)
+      (stroke (width 0.05) (type solid)) (fill none) (layer "F.CrtYd"))
+    (pad "1" thru_hole circle (at -3.225 0) (size 0.9 0.9) (drill 0.6) (layers "*.Cu" "*.Mask"))
+    (pad "1" thru_hole circle (at -2.280419 -2.280419) (size 0.9 0.9) (drill 0.6) (layers "*.Cu" "*.Mask"))
+    (pad "1" thru_hole circle (at -2.280419 2.280419) (size 0.9 0.9) (drill 0.6) (layers "*.Cu" "*.Mask"))
+    (pad "1" thru_hole circle (at 0 -3.225) (size 0.9 0.9) (drill 0.6) (layers "*.Cu" "*.Mask"))
+    (pad "1" thru_hole circle (at 0 0) (size 8.6 8.6) (drill 4.3) (layers "*.Cu" "*.Mask"))
+    (pad "1" thru_hole circle (at 0 3.225) (size 0.9 0.9) (drill 0.6) (layers "*.Cu" "*.Mask"))
+    (pad "1" thru_hole circle (at 2.280419 -2.280419) (size 0.9 0.9) (drill 0.6) (layers "*.Cu" "*.Mask"))
+    (pad "1" thru_hole circle (at 2.280419 2.280419) (size 0.9 0.9) (drill 0.6) (layers "*.Cu" "*.Mask"))
+    (pad "1" thru_hole circle (at 3.225 0) (size 0.9 0.9) (drill 0.6) (layers "*.Cu" "*.Mask"))
+  )
+  (footprint "MountingHole:MountingHole_4.3mm_M4_Pad_Via" (layer "F.Cu")
+    (at 215 140)
+    (descr "Mounting Hole 4.3mm, M4")
+    (tags "mounting hole 4.3mm m4")
+    (attr exclude_from_pos_files exclude_from_bom)
+    (fp_text reference "REF**" (at 0 -5.3) (layer "F.SilkS") hide
+        (effects (font (size 1 1) (thickness 0.15)))
+    )
+    (fp_text value "MountingHole_4.3mm_M4_Pad_Via" (at 0 5.3) (layer "F.Fab")
+        (effects (font (size 1 1) (thickness 0.15)))
+    )
+    (fp_text user "${REFERENCE}" (at 0 0) (layer "F.Fab")
+        (effects (font (size 1 1) (thickness 0.15)))
+    )
+    (fp_circle (center 0 0) (end 4.3 0)
+      (stroke (width 0.15) (type solid)) (fill none) (layer "Cmts.User"))
+    (fp_circle (center 0 0) (end 4.55 0)
+      (stroke (width 0.05) (type solid)) (fill none) (layer "F.CrtYd"))
+    (pad "1" thru_hole circle (at -3.225 0) (size 0.9 0.9) (drill 0.6) (layers "*.Cu" "*.Mask"))
+    (pad "1" thru_hole circle (at -2.280419 -2.280419) (size 0.9 0.9) (drill 0.6) (layers "*.Cu" "*.Mask"))
+    (pad "1" thru_hole circle (at -2.280419 2.280419) (size 0.9 0.9) (drill 0.6) (layers "*.Cu" "*.Mask"))
+    (pad "1" thru_hole circle (at 0 -3.225) (size 0.9 0.9) (drill 0.6) (layers "*.Cu" "*.Mask"))
+    (pad "1" thru_hole circle (at 0 0) (size 8.6 8.6) (drill 4.3) (layers "*.Cu" "*.Mask"))
+    (pad "1" thru_hole circle (at 0 3.225) (size 0.9 0.9) (drill 0.6) (layers "*.Cu" "*.Mask"))
+    (pad "1" thru_hole circle (at 2.280419 -2.280419) (size 0.9 0.9) (drill 0.6) (layers "*.Cu" "*.Mask"))
+    (pad "1" thru_hole circle (at 2.280419 2.280419) (size 0.9 0.9) (drill 0.6) (layers "*.Cu" "*.Mask"))
+    (pad "1" thru_hole circle (at 3.225 0) (size 0.9 0.9) (drill 0.6) (layers "*.Cu" "*.Mask"))
+  )
+  (footprint "MountingHole:MountingHole_4.3mm_M4_Pad_Via" (layer "F.Cu")
+    (at 85 140)
+    (descr "Mounting Hole 4.3mm, M4")
+    (tags "mounting hole 4.3mm m4")
+    (attr exclude_from_pos_files exclude_from_bom)
+    (fp_text reference "REF**" (at 0 -5.3) (layer "F.SilkS") hide
+        (effects (font (size 1 1) (thickness 0.15)))
+    )
+    (fp_text value "MountingHole_4.3mm_M4_Pad_Via" (at 0 5.3) (layer "F.Fab")
+        (effects (font (size 1 1) (thickness 0.15)))
+    )
+    (fp_text user "${REFERENCE}" (at 0 0) (layer "F.Fab")
+        (effects (font (size 1 1) (thickness 0.15)))
+    )
+    (fp_circle (center 0 0) (end 4.3 0)
+      (stroke (width 0.15) (type solid)) (fill none) (layer "Cmts.User"))
+    (fp_circle (center 0 0) (end 4.55 0)
+      (stroke (width 0.05) (type solid)) (fill none) (layer "F.CrtYd"))
+    (pad "1" thru_hole circle (at -3.225 0) (size 0.9 0.9) (drill 0.6) (layers "*.Cu" "*.Mask"))
+    (pad "1" thru_hole circle (at -2.280419 -2.280419) (size 0.9 0.9) (drill 0.6) (layers "*.Cu" "*.Mask"))
+    (pad "1" thru_hole circle (at -2.280419 2.280419) (size 0.9 0.9) (drill 0.6) (layers "*.Cu" "*.Mask"))
+    (pad "1" thru_hole circle (at 0 -3.225) (size 0.9 0.9) (drill 0.6) (layers "*.Cu" "*.Mask"))
+    (pad "1" thru_hole circle (at 0 0) (size 8.6 8.6) (drill 4.3) (layers "*.Cu" "*.Mask"))
+    (pad "1" thru_hole circle (at 0 3.225) (size 0.9 0.9) (drill 0.6) (layers "*.Cu" "*.Mask"))
+    (pad "1" thru_hole circle (at 2.280419 -2.280419) (size 0.9 0.9) (drill 0.6) (layers "*.Cu" "*.Mask"))
+    (pad "1" thru_hole circle (at 2.280419 2.280419) (size 0.9 0.9) (drill 0.6) (layers "*.Cu" "*.Mask"))
+    (pad "1" thru_hole circle (at 3.225 0) (size 0.9 0.9) (drill 0.6) (layers "*.Cu" "*.Mask"))
+  )
+  (gr_arc (start 215 50) (mid 222.071068 52.928932) (end 225 60)
+    (stroke (width 0.1) (type default)) (layer "Edge.Cuts"))
+  (gr_line (start 215 150) (end 85 150)
+    (stroke (width 0.1) (type default)) (layer "Edge.Cuts"))
+  (gr_arc (start 225 140) (mid 222.071068 147.071068) (end 215 150)
+    (stroke (width 0.1) (type default)) (layer "Edge.Cuts"))
+  (gr_arc (start 75 60) (mid 77.928932 52.928932) (end 85 50)
+    (stroke (width 0.1) (type default)) (layer "Edge.Cuts"))
+  (gr_line (start 225 60) (end 225 140)
+    (stroke (width 0.1) (type default)) (layer "Edge.Cuts"))
+  (gr_line (start 75 140) (end 75 60)
+    (stroke (width 0.1) (type default)) (layer "Edge.Cuts"))
+  (gr_line (start 85 50) (end 215 50)
+    (stroke (width 0.1) (type default)) (layer "Edge.Cuts"))
+  (gr_arc (start 85 150) (mid 77.928932 147.071068) (end 75 140)
+    (stroke (width 0.1) (type default)) (layer "Edge.Cuts"))
 )

Commit message: Started layout
Parts:
- added C1: 100nF, Capacitor_SMD:C_0402_1005Metric, F.Cu at (378.3, 129.8)
- added C10: 100uF, Capacitor_SMD:CP_Elec_10x10, F.Cu at (455.7, 31.7)
- added C100: 100nF, Capacitor_SMD:C_0402_1005Metric, F.Cu at (446.4, 168.1)
- added C11: 100uF, Capacitor_SMD:CP_Elec_10x10, F.Cu at (455.7, 43.5)
- added C12: 680uF, 0UCIRP-KiCAD-Lib:EEV-FK1V681Q, F.Cu at (480.8, 33.3)
- added C13: 330uF, Capacitor_SMD:CP_Elec_10x12.6, F.Cu at (479.6, 46.7)
- added C14: 4.7uF, Capacitor_SMD:C_0603_1608Metric, F.Cu at (492.3, 58.9)
- added C15: 100nF, Capacitor_SMD:C_0402_1005Metric, F.Cu at (445.2, 32.5)
- added C16: 100nF, Capacitor_SMD:C_0402_1005Metric, F.Cu at (445.2, 34.5)
- added C17: 100nF, Capacitor_SMD:C_0402_1005Metric, F.Cu at (445.2, 36.4)
- added C18: 100nF, Capacitor_SMD:C_0402_1005Metric, F.Cu at (445.2, 38.4)
- added C19: 100nF, Capacitor_SMD:C_0402_1005Metric, F.Cu at (445.2, 40.4)
- added C2: 100nF, Capacitor_SMD:C_0402_1005Metric, F.Cu at (363.3, 130.7)
- added C20: 10uF, Capacitor_SMD:C_0603_1608Metric, F.Cu at (492.3, 61.4)
- added C21: 1uF, Capacitor_SMD:C_0603_1608Metric, F.Cu at (678.2, 39.0)
- added C22: 10uF, Capacitor_SMD:C_0603_1608Metric, F.Cu at (680.0, 39.0)
- added C23: 1uF, Capacitor_SMD:C_0603_1608Metric, F.Cu at (682.8, 38.4)
- added C24: 1uF, Capacitor_SMD:C_0603_1608Metric, F.Cu at (581.1, 35.7)
- added C25: 10uF, Capacitor_SMD:C_0603_1608Metric, F.Cu at (581.1, 38.2)
- added C26: 1uF, Capacitor_SMD:C_0603_1608Metric, F.Cu at (581.1, 40.7)
- added C27: 1uF, Capacitor_SMD:C_0603_1608Metric, F.Cu at (606.4, 63.6)
- added C28: 10uF, Capacitor_SMD:C_0603_1608Metric, F.Cu at (606.4, 66.1)
- added C29: 1uF, Capacitor_SMD:C_0603_1608Metric, F.Cu at (606.4, 68.6)
- added C3: 100nF, Capacitor_SMD:C_0402_1005Metric, F.Cu at (374.6, 131.3)
- added C30: 1uF, Capacitor_SMD:C_0603_1608Metric, F.Cu at (580.3, 63.6)
- added C31: 10uF, Capacitor_SMD:C_0603_1608Metric, F.Cu at (580.3, 66.1)
- added C32: 1uF, Capacitor_SMD:C_0603_1608Metric, F.Cu at (580.3, 68.6)
- added C33: 1uF, Capacitor_SMD:C_0603_1608Metric, F.Cu at (554.2, 88.9)
- added C34: 10uF, Capacitor_SMD:C_0603_1608Metric, F.Cu at (554.2, 91.4)
- added C35: 1uF, Capacitor_SMD:C_0603_1608Metric, F.Cu at (554.2, 93.9)
- added C36: 1uF, Capacitor_SMD:C_0603_1608Metric, F.Cu at (554.2, 63.6)
- added C37: 10uF, Capacitor_SMD:C_0603_1608Metric, F.Cu at (554.2, 66.1)
- added C38: 1uF, Capacitor_SMD:C_0603_1608Metric, F.Cu at (554.2, 68.6)
- added C39: 100nF, Capacitor_SMD:C_0402_1005Metric, F.Cu at (422.5, 142.4)
- added C4: 100nF, Capacitor_SMD:C_0402_1005Metric, F.Cu at (365.1, 132.3)
- added C40: 100nF, Capacitor_SMD:C_0402_1005Metric, F.Cu at (399.4, 198.0)
- added C41: 10nF, Capacitor_SMD:C_0402_1005Metric, F.Cu at (448.5, 193.1)
- added C42: 100nF, Capacitor_SMD:C_0402_1005Metric, F.Cu at (446.5, 193.1)
- added C43: 100nF, Capacitor_SMD:C_0402_1005Metric, F.Cu at (373.3, 198.4)
- added C44: 1uF, Capacitor_SMD:C_0603_1608Metric, F.Cu at (435.7, 149.0)
- added C45: 0.1uF, Capacitor_SMD:C_0603_1608Metric, F.Cu at (450.1, 148.8)
- added C46: 1uF, Capacitor_SMD:C_0603_1608Metric, F.Cu at (460.7, 148.7)
- added C47: 0.1uF, Capacitor_SMD:C_0603_1608Metric, F.Cu at (475.0, 148.7)
- added C48: 100nF, Capacitor_SMD:C_0402_1005Metric, F.Cu at (402.7, 183.2)
- added C49: 100nF, Capacitor_SMD:C_0402_1005Metric, F.Cu at (374.1, 181.9)
- added C5: 100nF, Capacitor_SMD:C_0402_1005Metric, F.Cu at (369.5, 132.2)
- added C50: 100nF, Capacitor_SMD:C_0402_1005Metric, F.Cu at (422.6, 128.0)
- added C51: 100nF, Capacitor_SMD:C_0402_1005Metric, F.Cu at (396.3, 128.5)
- added C52: 100nF, Capacitor_SMD:C_0402_1005Metric, F.Cu at (409.8, 128.1)
- added C53: 4.7uF, Capacitor_SMD:C_0603_1608Metric, F.Cu at (374.8, 26.4)
- added C54: 100nF, Capacitor_SMD:C_0402_1005Metric, F.Cu at (371.3, 20.0)
- added C55: 100nF, Capacitor_SMD:C_0402_1005Metric, F.Cu at (371.3, 22.0)
- added C56: 100nF, Capacitor_SMD:C_0402_1005Metric, F.Cu at (371.3, 24.0)
- added C57: 100nF, Capacitor_SMD:C_0402_1005Metric, F.Cu at (371.3, 25.9)
- added C58: 100nF, Capacitor_SMD:C_0402_1005Metric, F.Cu at (371.3, 27.9)
- added C59: 100nF, Capacitor_SMD:C_0402_1005Metric, F.Cu at (305.5, 30.0)
- added C6: 10uF, Capacitor_SMD:C_0603_1608Metric, F.Cu at (479.2, 178.8)
- added C60: 100nF, Capacitor_SMD:C_0402_1005Metric, F.Cu at (305.5, 31.9)
- added C61: 100nF, Capacitor_SMD:C_0402_1005Metric, F.Cu at (305.5, 33.9)
- added C62: 100nF, Capacitor_SMD:C_0402_1005Metric, F.Cu at (305.5, 35.9)
- added C63: 100nF, Capacitor_SMD:C_0402_1005Metric, F.Cu at (305.5, 37.9)
- added C64: 100nF, Capacitor_SMD:C_0402_1005Metric, F.Cu at (305.5, 39.8)
- added C65: 100nF, Capacitor_SMD:C_0402_1005Metric, F.Cu at (305.5, 41.8)
- added C66: 100nF, Capacitor_SMD:C_0402_1005Metric, F.Cu at (308.4, 30.0)
- added C67: 100nF, Capacitor_SMD:C_0402_1005Metric, F.Cu at (308.4, 31.9)
- added C68: 100nF, Capacitor_SMD:C_0402_1005Metric, F.Cu at (308.4, 33.9)
- added C69: 2.2uF, Capacitor_SMD:C_0603_1608Metric, F.Cu at (334.5, 1.83)
- added C7: 4.7uF, Capacitor_SMD:C_0603_1608Metric, F.Cu at (492.3, 53.9)
- added C70: 100nF, Capacitor_SMD:C_0402_1005Metric, F.Cu at (308.4, 35.9)
- added C71: 100nF, Capacitor_SMD:C_0402_1005Metric, F.Cu at (308.4, 37.9)
- added C72: 100nF, Capacitor_SMD:C_0402_1005Metric, F.Cu at (308.4, 39.8)
- added C73: 2.2uF, Capacitor_SMD:C_0603_1608Metric, F.Cu at (334.5, 4.34)
- added C74: 100nF, Capacitor_SMD:C_0402_1005Metric, F.Cu at (308.4, 41.8)
- added C75: 100nF, Capacitor_SMD:C_0402_1005Metric, F.Cu at (311.3, 30.0)
- added C76: 10uF, Capacitor_SMD:C_0603_1608Metric, F.Cu at (334.5, 6.85)
- added C77: 100nF, Capacitor_SMD:C_0402_1005Metric, F.Cu at (311.3, 31.9)
- added C78: 100nF, Capacitor_SMD:C_0402_1005Metric, F.Cu at (311.3, 33.9)
- added C79: 100nF, Capacitor_SMD:C_0402_1005Metric, F.Cu at (311.3, 35.9)
- added C8: 0.1uF, Capacitor_SMD:C_0603_1608Metric, F.Cu at (492.3, 56.4)
- added C80: 100nF, Capacitor_SMD:C_0402_1005Metric, F.Cu at (311.3, 37.9)
- added C81: 100nF, Capacitor_SMD:C_0402_1005Metric, F.Cu at (311.3, 39.8)
- added C82: 100nF, Capacitor_SMD:C_0402_1005Metric, F.Cu at (311.3, 41.8)
- added C83: 100nF, Capacitor_SMD:C_0402_1005Metric, F.Cu at (314.1, 30.0)
- added C84: 100nF, Capacitor_SMD:C_0402_1005Metric, F.Cu at (314.1, 31.9)
- added C85: 1uF, Capacitor_SMD:C_0603_1608Metric, F.Cu at (334.5, 9.36)
- added C86: 4.7uF, Capacitor_SMD:C_0603_1608Metric, F.Cu at (334.5, 11.9)
- added C87: 1uF, Capacitor_SMD:C_0603_1608Metric, F.Cu at (334.5, 14.4)
- added C88: 100nF, Capacitor_SMD:C_0402_1005Metric, F.Cu at (314.1, 33.9)
- added C89: 100nF, Capacitor_SMD:C_0402_1005Metric, F.Cu at (314.1, 35.9)
- added C9: 100nF, Capacitor_SMD:C_0402_1005Metric, F.Cu at (445.2, 30.5)
- added C90: 2.2uF, Capacitor_SMD:C_0603_1608Metric, F.Cu at (334.5, 16.9)
- added C91: 100nF, Capacitor_SMD:C_0402_1005Metric, F.Cu at (409.2, 142.6)
- added C92: 100nF, Capacitor_SMD:C_0402_1005Metric, F.Cu at (383.9, 142.9)
- added C93: 10uF, Capacitor_SMD:C_0603_1608Metric, F.Cu at (330.0, 154.6)
- added C94: 10uF, Capacitor_SMD:C_0603_1608Metric, F.Cu at (329.5, 189.5)
- added C95: 10uF, Capacitor_SMD:C_0603_1608Metric, F.Cu at (329.8, 172.2)
- added C96: 100nF, Capacitor_SMD:C_0402_1005Metric, F.Cu at (360.8, 143.1)
- added C97: 100nF, Capacitor_SMD:C_0402_1005Metric, F.Cu at (360.8, 150.5)
- added C98: 100nF, Capacitor_SMD:C_0402_1005Metric, F.Cu at (395.9, 142.9)
- added C99: 10nF, Capacitor_SMD:C_0402_1005Metric, F.Cu at (448.5, 168.1)
- added D1: LED, LED_SMD:LED_0603_1608Metric_Pad1.05x0.95mm_HandSolder, F.Cu at (435.8, 30.8)
- added D10: LED, LED_SMD:LED_0603_1608Metric_Pad1.05x0.95mm_HandSolder, F.Cu at (435.8, 38.6)
- added D11: 30V 2A, Diode_SMD:Nexperia_DSN1608-2_1.6x0.8mm, F.Cu at (495.9, 60.9)
- added D12: LED, LED_SMD:LED_0603_1608Metric_Pad1.05x0.95mm_HandSolder, F.Cu at (435.8, 41.2)
- added D13: LED, LED_SMD:LED_0603_1608Metric_Pad1.05x0.95mm_HandSolder, F.Cu at (435.8, 43.8)
- added D14: LED, LED_SMD:LED_0603_1608Metric_Pad1.05x0.95mm_HandSolder, F.Cu at (435.8, 46.4)
- added D15: LED, LED_SMD:LED_0603_1608Metric_Pad1.05x0.95mm_HandSolder, F.Cu at (435.8, 49.0)
- added D16: LED, LED_SMD:LED_0603_1608Metric_Pad1.05x0.95mm_HandSolder, F.Cu at (685.3, 42.9)
- added D17: LED, LED_SMD:LED_0603_1608Metric_Pad1.05x0.95mm_HandSolder, F.Cu at (594.8, 35.7)
- added D18: LED, LED_SMD:LED_0603_1608Metric_Pad1.05x0.95mm_HandSolder, F.Cu at (620.1, 63.6)
- added D19: LED, LED_SMD:LED_0603_1608Metric_Pad1.05x0.95mm_HandSolder, F.Cu at (594.0, 63.6)
- added D2: 30V 2A, Diode_SMD:Nexperia_DSN1608-2_1.6x0.8mm, F.Cu at (495.9, 53.8)
- added D20: LED, LED_SMD:LED_0603_1608Metric_Pad1.05x0.95mm_HandSolder, F.Cu at (567.9, 88.9)
- added D21: LED, LED_SMD:LED_0603_1608Metric_Pad1.05x0.95mm_HandSolder, F.Cu at (567.9, 63.6)
- added D22: BZV55-B5V1, Diode_SMD:D_MiniMELF, F.Cu at (420.9, 146.6)
- added D23: SDT8A100P5-7, Diode_SMD:D_PowerDI-5, F.Cu at (390.7, 191.5)
- added D24: MMSZ4684T1G, Diode_SMD:D_SOD-123, F.Cu at (395.7, 197.5)
- added D25: SDT8A100P5-7, Diode_SMD:D_PowerDI-5, F.Cu at (364.6, 191.9)
- added D26: MMSZ4684T1G, Diode_SMD:D_SOD-123, F.Cu at (369.6, 197.9)
- added D27: SDT8A100P5-7, Diode_SMD:D_PowerDI-5, F.Cu at (394.1, 176.8)
- added D28: MMSZ4684T1G, Diode_SMD:D_SOD-123, F.Cu at (399.0, 182.7)
- added D29: SDT8A100P5-7, Diode_SMD:D_PowerDI-5, F.Cu at (365.5, 175.4)
- added D3: 30V 5A, Diode_SMD:D_SOD-128, F.Cu at (476.0, 61.2)
- added D30: MMSZ4684T1G, Diode_SMD:D_SOD-123, F.Cu at (370.5, 181.4)
- added D31: BZV55-B5V1, Diode_SMD:D_MiniMELF, F.Cu at (421.0, 132.2)
- added D32: BZV55-B5V1, Diode_SMD:D_MiniMELF, F.Cu at (394.8, 132.7)
- added D33: BZV55-B5V1, Diode_SMD:D_MiniMELF, F.Cu at (408.3, 132.3)
- added D34: ESD321, Diode_SMD:D_0402_1005Metric, F.Cu at (334.2, 19.1)
- added D35: ESD321, Diode_SMD:D_0402_1005Metric, F.Cu at (334.2, 21.1)
- added D36: LED, LED_SMD:LED_0603_1608Metric_Pad1.05x0.95mm_HandSolder, F.Cu at (336.7, 38.7)
- added D37: BZV55-B5V1, Diode_SMD:D_MiniMELF, F.Cu at (407.7, 146.8)
- added D38: BZV55-B5V1, Diode_SMD:D_MiniMELF, F.Cu at (382.3, 147.1)
- added D39: BZV55-B5V1, Diode_SMD:D_MiniMELF, F.Cu at (394.4, 147.1)
- added D4: 30V 2A, Diode_SMD:Nexperia_DSN1608-2_1.6x0.8mm, F.Cu at (495.9, 56.2)
- added D5: 700mV 5A, Diode_SMD:D_SMC, F.Cu at (453.9, 53.3)
- added D6: 700mV 5A, Diode_SMD:D_SMC, F.Cu at (453.9, 61.1)
- added D7: 30V 2A, Diode_SMD:Nexperia_DSN1608-2_1.6x0.8mm, F.Cu at (495.9, 58.5)
- added D8: LED, LED_SMD:LED_0603_1608Metric_Pad1.05x0.95mm_HandSolder, F.Cu at (435.8, 33.4)
- added D9: LED, LED_SMD:LED_0603_1608Metric_Pad1.05x0.95mm_HandSolder, F.Cu at (435.8, 36.0)
- added FB1: BLM18PG471SH1D, Inductor_SMD:L_0603_1608Metric, F.Cu at (447.0, 191.6)
- added FB2: BLM18PG471SH1D, Inductor_SMD:L_0603_1608Metric, F.Cu at (450.3, 192.1)
- added FB3: BLM18PG471SH1D, Inductor_SMD:L_0603_1608Metric, F.Cu at (446.9, 166.6)
- added FB4: BLM18PG471SH1D, Inductor_SMD:L_0603_1608Metric, F.Cu at (450.2, 167.1)
- added J1: ALARM, TerminalBlock:TerminalBlock_bornier-2_P5.08mm, F.Cu at (439.1, 132.5)
- added J10: Solenoid, Connector_PinHeader_2.54mm:PinHeader_1x03_P2.54mm_Vertical, F.Cu at (360.9, 181.2)
- added J11: PT, Connector_PinHeader_2.54mm:PinHeader_1x03_P2.54mm_Vertical, F.Cu at (416.8, 135.4)
- added J12: PT, Connector_PinHeader_2.54mm:PinHeader_1x03_P2.54mm_Vertical, F.Cu at (390.6, 135.9)
- added J13: PT, Connector_PinHeader_2.54mm:PinHeader_1x03_P2.54mm_Vertical, F.Cu at (404.1, 135.4)
- added J14: BMI-S-101, RF_Shielding:Laird_Technologies_BMI-S-101_13.66x12.70mm, F.Cu at (377.4, 11.0)
- added J15: GNSS SMA, Connector_Coaxial:SMA_Molex_73251-2200_Horizontal, F.Cu at (364.9, 20.5)
- added J16: ~, Connector_USB:USB_C_Receptacle_GCT_USB4105-xx-A_16P_TopMnt_Horizontal, F.Cu at (321.4, 34.3)
- added J17: ARM Cortex Debug, Connector_PinHeader_1.27mm:PinHeader_2x05_P1.27mm_Vertical_SMD, F.Cu at (335.0, 33.2)
- added J18: PT, Connector_PinHeader_2.54mm:PinHeader_1x03_P2.54mm_Vertical, F.Cu at (403.5, 150.0)
- added J19: PT, Connector_PinHeader_2.54mm:PinHeader_1x03_P2.54mm_Vertical, F.Cu at (378.1, 150.3)
- added J2: Conn_01x07, Connector_JST:JST_PH_B7B-PH-K_1x07_P2.00mm_Vertical, F.Cu at (475.3, 55.4)
- added J20: SMA, Connector_Coaxial:SMA_Molex_73251-2200_Horizontal, F.Cu at (333.0, 161.8)
- added J21: SMA, Connector_Coaxial:SMA_Molex_73251-2200_Horizontal, F.Cu at (333.0, 196.6)
- added J22: SMA, Connector_Coaxial:SMA_Molex_73251-2200_Horizontal, F.Cu at (333.0, 179.3)
- added J23: PT, Connector_PinHeader_2.54mm:PinHeader_1x03_P2.54mm_Vertical, F.Cu at (390.2, 150.2)
- added J3: ~, Connector_USB:USB_C_Receptacle_GCT_USB4105-xx-A_16P_TopMnt_Horizontal, F.Cu at (492.0, 20.3)
- added J4: SMA, Connector_Coaxial:SMA_Molex_73251-2200_Horizontal, F.Cu at (467.4, 43.3)
- added J5: ARM Cortex Debug, Connector_PinHeader_1.27mm:PinHeader_2x05_P1.27mm_Vertical_SMD, F.Cu at (493.9, 30.0)
- added J6: PT, Connector_PinHeader_2.54mm:PinHeader_1x03_P2.54mm_Vertical, F.Cu at (416.7, 149.7)
- added J7: Solenoid, Connector_PinHeader_2.54mm:PinHeader_1x03_P2.54mm_Vertical, F.Cu at (386.1, 197.4)
- added J8: Solenoid, Connector_PinHeader_2.54mm:PinHeader_1x03_P2.54mm_Vertical, F.Cu at (360.1, 197.7)
- added J9: Solenoid, Connector_PinHeader_2.54mm:PinHeader_1x03_P2.54mm_Vertical, F.Cu at (389.5, 182.6)
- added JP1: Bridge, Jumper:SolderJumper-2_P1.3mm_Open_RoundedPad1.0x1.5mm, F.Cu at (682.8, 43.3)
- added JP2: Bridge, Jumper:SolderJumper-2_P1.3mm_Open_RoundedPad1.0x1.5mm, F.Cu at (585.2, 40.4)
- added JP3: Bridge, Jumper:SolderJumper-2_P1.3mm_Open_RoundedPad1.0x1.5mm, F.Cu at (610.5, 68.3)
- added JP4: Bridge, Jumper:SolderJumper-2_P1.3mm_Open_RoundedPad1.0x1.5mm, F.Cu at (584.4, 68.3)
- added JP5: Bridge, Jumper:SolderJumper-2_P1.3mm_Open_RoundedPad1.0x1.5mm, F.Cu at (558.3, 93.6)
- added JP6: Bridge, Jumper:SolderJumper-2_P1.3mm_Open_RoundedPad1.0x1.5mm, F.Cu at (558.3, 68.3)
- added L1: 33uH, Inductor_SMD:L_12x12mm_H8mm, F.Cu at (441.0, 8.18)
- added L2: 68uH, Inductor_SMD:L_12x12mm_H8mm, F.Cu at (441.0, 22.4)
- added P1: PAD_SMD, TestPoint:TestPoint_Plated_Hole_D4.0mm, F.Cu at (345.3, 4.10)
- added P2: PAD_SMD, TestPoint:TestPoint_Plated_Hole_D4.0mm, F.Cu at (345.3, 11.2)
- added P3: PAD_SMD, TestPoint:TestPoint_Plated_Hole_D4.0mm, F.Cu at (345.3, 18.2)
- added P4: PAD_SMD, TestPoint:TestPoint_Plated_Hole_D4.0mm, F.Cu at (345.3, 25.3)
- added P5: PAD_SMD, TestPoint:TestPoint_Pad_2.0x2.0mm, F.Cu at (435.6, 52.3)
- added P6: PAD_SMD, TestPoint:TestPoint_Pad_2.0x2.0mm, F.Cu at (435.6, 56.3)
- added Q1: DMG3402L, Package_TO_SOT_SMD:SOT-23-3, F.Cu at (448.8, 134.4)
- added Q10: DMG3402L, Package_TO_SOT_SMD:SOT-23-3, F.Cu at (395.0, 193.9)
- added Q11: DMG3402L, Package_TO_SOT_SMD:SOT-23-3, F.Cu at (369.0, 194.3)
- added Q12: DMG3402L, Package_TO_SOT_SMD:SOT-23-3, F.Cu at (398.4, 179.2)
- added Q13: DMG3402L, Package_TO_SOT_SMD:SOT-23-3, F.Cu at (369.8, 177.8)
- added Q2: Q_NMOS_GSD, Package_TO_SOT_SMD:SOT-23-3, F.Cu at (465.0, 50.4)
- added Q3: Q_NMOS_GSD, Package_TO_SOT_SMD:SOT-23-3, F.Cu at (465.0, 55.0)
- added Q4: PMOS, Package_SO:Vishay_PowerPAK_1212-8_Single, F.Cu at (441.1, 31.9)
- added Q5: PMOS, Package_SO:Vishay_PowerPAK_1212-8_Single, F.Cu at (441.1, 36.5)
- added Q6: Q_NMOS_GSD, Package_TO_SOT_SMD:SOT-23-3, F.Cu at (465.0, 59.6)
- added Q7: Q_NMOS_GSD, Package_TO_SOT_SMD:SOT-23-3, F.Cu at (465.0, 64.2)
- added Q8: PMOS, Package_SO:Vishay_PowerPAK_1212-8_Single, F.Cu at (441.1, 41.1)
- added Q9: PMOS, Package_SO:Vishay_PowerPAK_1212-8_Single, F.Cu at (441.1, 45.7)
- added R1: 10K, Resistor_SMD:R_0402_1005Metric, F.Cu at (448.0, 130.6)
- added R10: 10K, Resistor_SMD:R_0402_1005Metric, F.Cu at (487.6, 12.0)
- added R100: 1K, Resistor_SMD:R_0402_1005Metric, F.Cu at (404.8, 132.3)
- added R101: 5K, Resistor_SMD:R_0402_1005Metric, F.Cu at (409.8, 130.4)
- added R102: 10K, Resistor_SMD:R_0402_1005Metric, F.Cu at (409.8, 129.2)
- added R103: 10K, Resistor_SMD:R_0402_1005Metric, F.Cu at (328.7, 30.0)
- added R104: 10K, Resistor_SMD:R_0402_1005Metric, F.Cu at (328.7, 32.0)
- added R105: 5.1K, Resistor_SMD:R_0603_1608Metric_Pad0.98x0.95mm_HandSolder, F.Cu at (332.3, 38.7)
- added R106: 5.1K, Resistor_SMD:R_0603_1608Metric_Pad0.98x0.95mm_HandSolder, F.Cu at (332.3, 41.2)
- added R107: 10K, Resistor_SMD:R_0402_1005Metric, F.Cu at (328.7, 34.0)
- added R108: 10K, Resistor_SMD:R_0402_1005Metric, F.Cu at (328.7, 36.0)
- added R109: 100R, Resistor_SMD:R_0402_1005Metric, F.Cu at (328.7, 37.9)
- added R11: 1K, Resistor_SMD:R_0402_1005Metric, F.Cu at (487.6, 14.0)
- added R110: 1K, Resistor_SMD:R_0402_1005Metric, F.Cu at (404.3, 146.8)
- added R111: 5K, Resistor_SMD:R_0402_1005Metric, F.Cu at (409.2, 144.9)
- added R112: 10K, Resistor_SMD:R_0402_1005Metric, F.Cu at (409.2, 143.8)
- added R113: 1K, Resistor_SMD:R_0402_1005Metric, F.Cu at (378.9, 147.1)
- added R114: 5K, Resistor_SMD:R_0402_1005Metric, F.Cu at (383.9, 145.2)
- added R115: 10K, Resistor_SMD:R_0402_1005Metric, F.Cu at (383.9, 144.1)
- added R116: 100K, Resistor_SMD:R_0402_1005Metric, F.Cu at (309.3, 155.8)
- added R117: 100K, Resistor_SMD:R_0402_1005Metric, F.Cu at (309.2, 190.8)
- added R118: 100K, Resistor_SMD:R_0402_1005Metric, F.Cu at (309.4, 173.2)
- added R119: 100K, Resistor_SMD:R_0402_1005Metric, F.Cu at (360.8, 139.6)
- added R12: 100R, Resistor_SMD:R_0402_1005Metric, F.Cu at (490.6, 2.05)
- added R120: 100K, Resistor_SMD:R_0402_1005Metric, F.Cu at (360.8, 147.1)
- added R121: 1K, Resistor_SMD:R_0402_1005Metric, F.Cu at (391.0, 147.1)
- added R122: 5K, Resistor_SMD:R_0402_1005Metric, F.Cu at (395.9, 145.2)
- added R123: 10K, Resistor_SMD:R_0402_1005Metric, F.Cu at (395.9, 144.0)
- added R124: 100K, Resistor_SMD:R_0402_1005Metric, F.Cu at (446.9, 177.1)
- added R13: 15K, Resistor_SMD:R_0402_1005Metric, F.Cu at (490.6, 4.04)
- added R14: 10K, Resistor_SMD:R_0402_1005Metric, F.Cu at (490.6, 6.03)
- added R15: 100R, Resistor_SMD:R_0402_1005Metric, F.Cu at (490.6, 8.02)
- added R16: 100K, Resistor_SMD:R_0402_1005Metric, F.Cu at (490.6, 10.0)
- added R17: 1.5K, Resistor_SMD:R_0402_1005Metric, F.Cu at (490.6, 12.0)
- added R18: 15K, Resistor_SMD:R_0402_1005Metric, F.Cu at (490.6, 14.0)
- added R19: 1.5K, Resistor_SMD:R_0402_1005Metric, F.Cu at (493.5, 2.05)
- added R2: 100R, Resistor_SMD:R_0402_1005Metric, F.Cu at (448.0, 131.7)
- added R20: 1K, Resistor_SMD:R_0402_1005Metric, F.Cu at (493.5, 4.04)
- added R21: 1K, Resistor_SMD:R_0402_1005Metric, F.Cu at (493.5, 6.03)
- added R22: 100R, Resistor_SMD:R_0402_1005Metric, F.Cu at (493.5, 8.02)
- added R23: 10K, Resistor_SMD:R_0402_1005Metric, F.Cu at (493.5, 10.0)
- added R24: 100R, Resistor_SMD:R_0402_1005Metric, F.Cu at (493.5, 12.0)
- added R25: 100K, Resistor_SMD:R_0402_1005Metric, F.Cu at (493.5, 14.0)
- added R26: 10K, Resistor_SMD:R_0402_1005Metric, F.Cu at (496.4, 2.05)
- added R27: 10K, Resistor_SMD:R_0402_1005Metric, F.Cu at (496.4, 4.04)
- added R28: 1.5K, Resistor_SMD:R_0402_1005Metric, F.Cu at (496.4, 6.03)
- added R29: 1.5K, Resistor_SMD:R_0402_1005Metric, F.Cu at (496.4, 8.02)
- added R3: 4k7, Resistor_SMD:R_0402_1005Metric, F.Cu at (365.1, 128.9)
- added R30: 27K, Resistor_SMD:R_0603_1608Metric, F.Cu at (685.3, 39.1)
- added R31: 375R, Resistor_SMD:R_0402_1005Metric, F.Cu at (679.7, 41.1)
- added R32: 10K, Resistor_SMD:R_0402_1005Metric, F.Cu at (679.7, 42.3)
- added R33: 10K, Resistor_SMD:R_0402_1005Metric, F.Cu at (686.7, 39.6)
- added R34: 10K, Resistor_SMD:R_0402_1005Metric, F.Cu at (687.2, 44.1)
- added R35: 1K, Resistor_SMD:R_0402_1005Metric, F.Cu at (686.7, 42.2)
- added R36: 1.5K, Resistor_SMD:R_0402_1005Metric, F.Cu at (687.8, 42.2)
- added R37: 27K, Resistor_SMD:R_0603_1608Metric, F.Cu at (581.1, 43.2)
- added R38: 375R, Resistor_SMD:R_0402_1005Metric, F.Cu at (577.6, 35.4)
- added R39: 10K, Resistor_SMD:R_0402_1005Metric, F.Cu at (577.6, 37.4)
- added R4: 4k7, Resistor_SMD:R_0402_1005Metric, F.Cu at (366.9, 130.7)
- added R40: 10K, Resistor_SMD:R_0402_1005Metric, F.Cu at (577.6, 39.4)
- added R41: 10K, Resistor_SMD:R_0402_1005Metric, F.Cu at (577.6, 41.4)
- added R42: 1K, Resistor_SMD:R_0402_1005Metric, F.Cu at (577.6, 43.4)
- added R43: 1.5K, Resistor_SMD:R_0402_1005Metric, F.Cu at (577.6, 45.4)
- added R44: 27K, Resistor_SMD:R_0603_1608Metric, F.Cu at (606.4, 71.1)
- added R45: 375R, Resistor_SMD:R_0402_1005Metric, F.Cu at (602.9, 63.3)
- added R46: 10K, Resistor_SMD:R_0402_1005Metric, F.Cu at (602.9, 65.3)
- added R47: 10K, Resistor_SMD:R_0402_1005Metric, F.Cu at (602.9, 67.3)
- added R48: 10K, Resistor_SMD:R_0402_1005Metric, F.Cu at (602.9, 69.3)
- added R49: 1K, Resistor_SMD:R_0402_1005Metric, F.Cu at (602.9, 71.3)
- added R5: 10K, Resistor_SMD:R_0402_1005Metric, F.Cu at (487.6, 2.05)
- added R50: 1.5K, Resistor_SMD:R_0402_1005Metric, F.Cu at (602.9, 73.3)
- added R51: 27K, Resistor_SMD:R_0603_1608Metric, F.Cu at (580.3, 71.1)
- added R52: 375R, Resistor_SMD:R_0402_1005Metric, F.Cu at (576.8, 63.3)
- added R53: 10K, Resistor_SMD:R_0402_1005Metric, F.Cu at (576.8, 65.3)
- added R54: 10K, Resistor_SMD:R_0402_1005Metric, F.Cu at (576.8, 67.3)
- added R55: 10K, Resistor_SMD:R_0402_1005Metric, F.Cu at (576.8, 69.3)
- added R56: 1K, Resistor_SMD:R_0402_1005Metric, F.Cu at (576.8, 71.3)
- added R57: 1.5K, Resistor_SMD:R_0402_1005Metric, F.Cu at (576.8, 73.3)
- added R58: 27K, Resistor_SMD:R_0603_1608Metric, F.Cu at (554.2, 96.4)
- added R59: 375R, Resistor_SMD:R_0402_1005Metric, F.Cu at (550.7, 88.6)
- added R6: 5ohm, Resistor_SMD:R_0402_1005Metric, F.Cu at (487.6, 4.04)
- added R60: 10K, Resistor_SMD:R_0402_1005Metric, F.Cu at (550.7, 90.6)
- added R61: 10K, Resistor_SMD:R_0402_1005Metric, F.Cu at (550.7, 92.6)
- added R62: 10K, Resistor_SMD:R_0402_1005Metric, F.Cu at (550.7, 94.6)
- added R63: 1K, Resistor_SMD:R_0402_1005Metric, F.Cu at (550.7, 96.6)
- added R64: 1.5K, Resistor_SMD:R_0402_1005Metric, F.Cu at (550.7, 98.6)
- added R65: 27K, Resistor_SMD:R_0603_1608Metric, F.Cu at (554.2, 71.1)
- added R66: 375R, Resistor_SMD:R_0402_1005Metric, F.Cu at (550.7, 63.3)
- added R67: 10K, Resistor_SMD:R_0402_1005Metric, F.Cu at (550.7, 65.3)
- added R68: 10K, Resistor_SMD:R_0402_1005Metric, F.Cu at (550.7, 67.3)
- added R69: 10K, Resistor_SMD:R_0402_1005Metric, F.Cu at (550.7, 69.3)
- added R7: 2K, Resistor_SMD:R_0402_1005Metric, F.Cu at (487.6, 6.03)
- added R70: 1K, Resistor_SMD:R_0402_1005Metric, F.Cu at (550.7, 71.3)
- added R71: 1.5K, Resistor_SMD:R_0402_1005Metric, F.Cu at (550.7, 73.3)
- added R72: 1K, Resistor_SMD:R_0402_1005Metric, F.Cu at (417.5, 146.6)
- added R73: 5K, Resistor_SMD:R_0402_1005Metric, F.Cu at (422.5, 144.7)
- added R74: 10K, Resistor_SMD:R_0402_1005Metric, F.Cu at (422.5, 143.5)
- added R75: 10K, Resistor_SMD:R_0402_1005Metric, F.Cu at (400.2, 192.3)
- added R76: 100R, Resistor_SMD:R_0402_1005Metric, F.Cu at (398.1, 192.3)
- added R77: 0.1R, Resistor_SMD:R_2512_6332Metric, F.Cu at (397.2, 189.6)
- added R78: 1K, Resistor_SMD:R_0402_1005Metric, F.Cu at (397.6, 193.9)
- added R79: 100K, Resistor_SMD:R_0402_1005Metric, F.Cu at (447.0, 202.1)
- added R8: 2K, Resistor_SMD:R_0402_1005Metric, F.Cu at (487.6, 8.02)
- added R80: 10K, Resistor_SMD:R_0402_1005Metric, F.Cu at (374.2, 192.7)
- added R81: 100R, Resistor_SMD:R_0402_1005Metric, F.Cu at (372.0, 192.7)
- added R82: 0.1R, Resistor_SMD:R_2512_6332Metric, F.Cu at (371.1, 190.0)
- added R83: 1K, Resistor_SMD:R_0402_1005Metric, F.Cu at (371.5, 194.3)
- added R84: 0, Resistor_SMD:R_1206_3216Metric_Pad1.30x1.75mm_HandSolder, F.Cu at (450.5, 144.7)
- added R85: 0, Resistor_SMD:R_1206_3216Metric_Pad1.30x1.75mm_HandSolder, F.Cu at (475.4, 144.5)
- added R86: 10K, Resistor_SMD:R_0402_1005Metric, F.Cu at (403.6, 177.5)
- added R87: 100R, Resistor_SMD:R_0402_1005Metric, F.Cu at (401.4, 177.5)
- added R88: 0.1R, Resistor_SMD:R_2512_6332Metric, F.Cu at (400.5, 174.8)
- added R89: 1K, Resistor_SMD:R_0402_1005Metric, F.Cu at (400.9, 179.2)
- added R9: 100K, Resistor_SMD:R_0402_1005Metric, F.Cu at (487.6, 10.0)
- added R90: 10K, Resistor_SMD:R_0402_1005Metric, F.Cu at (375.0, 176.1)
- added R91: 100R, Resistor_SMD:R_0402_1005Metric, F.Cu at (372.9, 176.1)
- added R92: 0.1R, Resistor_SMD:R_2512_6332Metric, F.Cu at (372.0, 173.5)
- added R93: 1K, Resistor_SMD:R_0402_1005Metric, F.Cu at (372.4, 177.8)
- added R94: 1K, Resistor_SMD:R_0402_1005Metric, F.Cu at (417.6, 132.2)
- added R95: 5K, Resistor_SMD:R_0402_1005Metric, F.Cu at (422.6, 130.3)
- added R96: 10K, Resistor_SMD:R_0402_1005Metric, F.Cu at (422.6, 129.1)
- added R97: 1K, Resistor_SMD:R_0402_1005Metric, F.Cu at (391.3, 132.7)
- added R98: 5K, Resistor_SMD:R_0402_1005Metric, F.Cu at (396.3, 130.8)
- added R99: 10K, Resistor_SMD:R_0402_1005Metric, F.Cu at (396.3, 129.7)
- added TC1: Thermocouple, 0UCIRP-KiCAD-Lib:AM-K-PCB, F.Cu at (434.6, 195.7)
- added TC2: Thermocouple, 0UCIRP-KiCAD-Lib:AM-K-PCB, F.Cu at (434.6, 170.7)
- added TP1: Cell 1, TestPoint:TestPoint_Pad_2.0x2.0mm, F.Cu at (435.6, 60.4)
- added TP2: Cell 2, TestPoint:TestPoint_Pad_2.0x2.0mm, F.Cu at (439.7, 52.3)
- added TP3: Cell 3, TestPoint:TestPoint_Pad_2.0x2.0mm, F.Cu at (439.7, 56.3)
- added TP4: Cell 4, TestPoint:TestPoint_Pad_2.0x2.0mm, F.Cu at (439.7, 60.4)
- added TP5: Cell 5, TestPoint:TestPoint_Pad_2.0x2.0mm, F.Cu at (443.7, 52.3)
- added TP6: Cell 6, TestPoint:TestPoint_Pad_2.0x2.0mm, F.Cu at (443.7, 56.3)
- added TP7: GND, TestPoint:TestPoint_Pad_2.0x2.0mm, F.Cu at (443.7, 60.4)
- added U1: ~, 0UCIRP-KiCAD-Lib:BMI088, F.Cu at (372.0, 131.2)
- added U10: ~, 0UCIRP-KiCAD-Lib:EC4SAW-xxSxxN, F.Cu at (665.7, 41.1)
- added U11: ~, Package_SON:WSON-8-1EP_2x2mm_P0.5mm_EP0.9x1.6mm, F.Cu at (682.8, 40.6)
- added U12: VOS615A-1, Package_SO:SOP-4_4.4x2.6mm_P1.27mm, F.Cu at (690.0, 41.9)
- added U13: ~, 0UCIRP-KiCAD-Lib:EC4SAW-xxSxxN, F.Cu at (588.7, 28.4)
- added U14: ~, Package_SON:WSON-8-1EP_2x2mm_P0.5mm_EP0.9x1.6mm, F.Cu at (585.3, 44.0)
- added U15: VOS615A-1, Package_SO:SOP-4_4.4x2.6mm_P1.27mm, F.Cu at (587.8, 36.5)
- added U16: ~, 0UCIRP-KiCAD-Lib:EC4SAW-xxSxxN, F.Cu at (614.0, 56.3)
- added U17: ~, Package_SON:WSON-8-1EP_2x2mm_P0.5mm_EP0.9x1.6mm, F.Cu at (610.6, 71.9)
- added U18: VOS615A-1, Package_SO:SOP-4_4.4x2.6mm_P1.27mm, F.Cu at (613.1, 64.4)
- added U19: ~, 0UCIRP-KiCAD-Lib:EC4SAW-xxSxxN, F.Cu at (587.9, 56.3)
- added U2: ~, 0UCIRP-KiCAD-Lib:MS5607-02BA, F.Cu at (381.0, 131.2)
- added U20: ~, Package_SON:WSON-8-1EP_2x2mm_P0.5mm_EP0.9x1.6mm, F.Cu at (584.5, 71.9)
- added U21: VOS615A-1, Package_SO:SOP-4_4.4x2.6mm_P1.27mm, F.Cu at (587.0, 64.4)
- added U22: ~, 0UCIRP-KiCAD-Lib:EC4SAW-xxSxxN, F.Cu at (561.8, 81.6)
- added U23: ~, Package_SON:WSON-8-1EP_2x2mm_P0.5mm_EP0.9x1.6mm, F.Cu at (558.4, 97.2)
- added U24: VOS615A-1, Package_SO:SOP-4_4.4x2.6mm_P1.27mm, F.Cu at (560.9, 89.7)
- added U25: ~, 0UCIRP-KiCAD-Lib:EC4SAW-xxSxxN, F.Cu at (561.8, 56.3)
- added U26: ~, Package_SON:WSON-8-1EP_2x2mm_P0.5mm_EP0.9x1.6mm, F.Cu at (558.4, 71.9)
- added U27: VOS615A-1, Package_SO:SOP-4_4.4x2.6mm_P1.27mm, F.Cu at (560.9, 64.4)
- added U28: ~, Package_TO_SOT_SMD:SOT-23-5, F.Cu at (419.2, 143.5)
- added U29: ~, Package_TO_SOT_SMD:SOT-23-5, F.Cu at (400.0, 195.2)
- added U3: ~, Package_CSP:WLCSP-12_1.56x1.56mm_P0.4mm, F.Cu at (365.1, 130.6)
- added U30: ~, Package_SO:SOIC-8_3.9x4.9mm_P1.27mm, F.Cu at (448.2, 197.5)
- added U31: ~, Package_TO_SOT_SMD:SOT-23-5, F.Cu at (373.9, 195.6)
- added U32: ~, Converter_DCDC:Converter_DCDC_TRACO_TSR-1_THT, F.Cu at (440.5, 148.1)
- added U33: ~, Converter_DCDC:Converter_DCDC_TRACO_TSR-1_THT, F.Cu at (465.5, 148.0)
- added U34: ~, Package_TO_SOT_SMD:SOT-23-5, F.Cu at (403.3, 180.4)
- added U35: ~, Package_TO_SOT_SMD:SOT-23-5, F.Cu at (374.8, 179.1)
- added U36: ~, Package_TO_SOT_SMD:SOT-23-5, F.Cu at (419.3, 129.1)
- added U37: ~, Package_TO_SOT_SMD:SOT-23-5, F.Cu at (393.0, 129.7)
- added U38: ~, Package_TO_SOT_SMD:SOT-23-5, F.Cu at (406.5, 129.2)
- added U39: ~, 0UCIRP-KiCAD-Lib:ZOE-M8Q, F.Cu at (375.8, 22.1)
- added U4: ~, 0UCIRP-KiCAD-Lib:GC-XPORT, F.Cu at (478.2, 169.7)
- added U40: ~, Package_QFP:LQFP-176_24x24mm_P0.5mm, F.Cu at (318.3, 14.8)
- added U41: ~, Package_TO_SOT_SMD:SOT-23-5, F.Cu at (405.9, 143.8)
- added U42: ~, Package_TO_SOT_SMD:SOT-23-5, F.Cu at (380.6, 144.1)
- added U43: ~, 0UCIRP-KiCAD-Lib:RFM95W, F.Cu at (319.2, 154.7)
- added U44: ~, 0UCIRP-KiCAD-Lib:RFM95W, F.Cu at (319.1, 189.7)
- added U45: ~, 0UCIRP-KiCAD-Lib:RFM95W, F.Cu at (319.2, 172.3)
- added U46: ~, Package_SO:SOIC-8W_5.3x5.3mm_P1.27mm, F.Cu at (366.2, 141.6)
- added U47: ~, Package_SO:SOIC-8W_5.3x5.3mm_P1.27mm, F.Cu at (366.2, 149.1)
- added U48: ~, Package_TO_SOT_SMD:SOT-23-5, F.Cu at (392.6, 144.0)
- added U49: ~, Package_SO:SOIC-8_3.9x4.9mm_P1.27mm, F.Cu at (448.2, 172.5)
- added U5: ADS7828, Package_SO:TSSOP-16_4.4x5mm_P0.65mm, F.Cu at (493.9, 37.5)
- added U6: LM2596S-3.3, Package_TO_SOT_SMD:TO-263-5_TabPin3, F.Cu at (459.1, 7.23)
- added U7: LM2596S-5, Package_TO_SOT_SMD:TO-263-5_TabPin3, F.Cu at (459.1, 19.6)
- added U8: ~, Package_QFP:LQFP-48_7x7mm_P0.5mm, F.Cu at (492.6, 46.5)
- added U9: ~, 0UCIRP-KiCAD-Lib:RFM95W, F.Cu at (476.6, 10.6)
- added Y1: 16MHz, Crystal:Crystal_SMD_2520-4Pin_2.5x2.0mm, F.Cu at (481.9, 61.2)
- added Y2: 16MHz, Crystal:Crystal_SMD_2016-4Pin_2.0x1.6mm, F.Cu at (337.6, 20.0)
Routing:
- net +24V: track 0.00 -> 46.3 mm
- net +3.3V: track 0.00 -> 41.1 mm
- net Net-(TC2--): track 0.00 -> 29.5 mm
- net Net-(TC1--): track 0.00 -> 29.5 mm
- net /REDs/Single-Cell-Charger/ISO_GND: track 0.00 -> 22.2 mm
- net +5V: track 0.00 -> 19.0 mm
- net Net-(TC2-+): track 0.00 -> 17.6 mm
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Other:
- copper layers 4 -> 6

Commit message: Started putting it all together
Parts:
- C20, C93, C94, C95, R116, R117, R118, R25, U43, U44, U45, U9: moved to B.Cu
- moved R25 396.3 mm to (102.3, 77.7), turned to 180 degrees
- moved C20 389.1 mm to (103.2, 57.3), turned to 180 degrees
- moved U9 378.0 mm to (103.0, 67.8), turned to 90 degrees
- moved J4 371.6 mm to (96.0, 54.0)
- moved J14 293.1 mm to (90.9, 73.1), turned to 90 degrees
- moved J15 290.9 mm to (78.9, 73.7), turned to 90 degrees
- moved U39 289.4 mm to (90.9, 73.1), turned to 90 degrees
- moved C53 286.3 mm to (91.6, 69.1), turned to 180 degrees
- moved C55 284.9 mm to (91.7, 76.8), turned to -90 degrees
- moved C56 283.4 mm to (92.9, 76.8), turned to -90 degrees
- moved C54 282.2 mm to (94.7, 75.7)
- moved C57 280.9 mm to (94.7, 74.5)
- moved C58 280.0 mm to (94.4, 69.1)
- moved J20 262.5 mm to (78.8, 96.3), turned to 90 degrees
- moved J21 262.5 mm to (78.8, 131.1), turned to 90 degrees
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Routing:
- net /REDs/Single-Cell-Charger3/ISO_5V: track 0.00 -> 45.8 mm
- net /REDs/Single-Cell-Charger4/ISO_5V: track 0.00 -> 45.8 mm
- net /REDs/Single-Cell-Charger1/ISO_5V: track 0.00 -> 45.8 mm
- net /REDs/Single-Cell-Charger2/ISO_5V: track 0.00 -> 45.8 mm
- net /REDs/Single-Cell-Charger5/ISO_5V: track 0.00 -> 45.8 mm
- net /REDs/Single-Cell-Charger/ISO_5V: track 14.2 -> 45.8 mm
- net +3V3: track 0.00 -> 30.7 mm
- net /REDs/Single-Cell-Charger2/ISO_GND: track 0.00 -> 23.8 mm
- net /REDs/Single-Cell-Charger4/ISO_GND: track 0.00 -> 23.8 mm
- net /REDs/Single-Cell-Charger3/ISO_GND: track 0.00 -> 23.8 mm
- net /REDs/Single-Cell-Charger1/ISO_GND: track 0.00 -> 23.8 mm
- net GND: track 4.68 -> 26.9 mm
- net Net-(D6-K): track 0.00 -> 20.0 mm
- net Net-(U7-FB): track 0.00 -> 18.2 mm
- net +3.3V: track 41.1 -> 58.1 mm
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
Commit message: More layout updates
Parts:
- moved U27 363.8 mm to (188.6, 121.7), turned to -90 degrees
- moved U24 362.6 mm to (188.6, 111.3), turned to -90 degrees
- moved U21 361.9 mm to (188.6, 100.8), turned to -90 degrees
- moved FB2 361.8 mm to (94.9, 123.8), turned to 180 degrees
- moved U18 360.9 mm to (188.6, 90.4), turned to -90 degrees
- moved U15 359.7 mm to (188.6, 80.0), turned to -90 degrees
- moved R71 359.7 mm to (190.8, 121.4), turned to -90 degrees
- moved R69 359.4 mm to (191.4, 119.5), turned to 180 degrees
- moved C41 359.0 mm to (96.0, 125.6), turned to 90 degrees
- moved U12 358.6 mm to (188.6, 69.6), turned to -90 degrees
- moved R64 358.5 mm to (190.8, 111.0), turned to -90 degrees
- moved FB1 358.4 mm to (94.4, 127.1), turned to 90 degrees
- moved R62 358.1 mm to (191.4, 109.1), turned to 180 degrees
- moved R57 357.8 mm to (190.8, 100.6), turned to -90 degrees
- moved R70 357.5 mm to (191.9, 121.4), turned to -90 degrees
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Routing:
- net GND: track 26.9 -> 37.1 mm, vias 0 -> 33
- net Net-(J15-In): track 0.00 -> 10.0 mm, vias 0 -> 1
- added copper zone on F.Cu, net GND
- added copper zone on In1.Cu, net GND
- added copper zone on In4.Cu, net GND
