File: rocket2-ecu.kicad_pcb (KiCad board)
At the start: 6 copper layers, 150 x 100 mm, 381 parts, among them J1 ALARM, J10 Solenoid, J11 PT, J12 PT, J13 PT, J14 BMI-S-101, J15 GNSS SMA, J17 ARM Cortex Debug, J18 PT, J19 PT, J2 Conn_01x07, J20 SMA, J21 SMA, J22 SMA, J23 PT, J4 SMA, J5 ARM Cortex Debug, J6 PT, J7 Solenoid, J8 Solenoid, J9 Solenoid, P1 PAD_SMD, P2 PAD_SMD, P3 PAD_SMD, P4 PAD_SMD, P5 PAD_SMD, P6 PAD_SMD, Q1 DMG3402L, Q10 DMG3402L, Q11 DMG3402L, Q12 DMG3402L, Q13 DMG3402L, Q2 Q_NMOS_GSD, Q3 Q_NMOS_GSD, Q4 PMOS, Q5 PMOS, Q6 Q_NMOS_GSD, Q7 Q_NMOS_GSD, Q8 PMOS, Q9 PMOS, U12 VOS615A-1, U15 VOS615A-1, U18 VOS615A-1, U21 VOS615A-1, U24 VOS615A-1, U27 VOS615A-1, U5 ADS7828, U6 LM2596S-3.3, U7 LM2596S-5, Y1 16MHz, Y2 16MHz

Commit message: Replaced Regs
Parts:
- removed C44, C46: 1uF, Capacitor_SMD:C_0603_1608Metric
- removed C45, C47: 0.1uF, Capacitor_SMD:C_0603_1608Metric
- removed D9: LED, LED_SMD:LED_0603_1608Metric_Pad1.05x0.95mm_HandSolder
- removed REF** (x4): MountingHole_4.3mm_M4_Pad_Via, MountingHole:MountingHole_4.3mm_M4_Pad_Via
- removed TP1: Cell 1, TestPoint:TestPoint_Pad_2.0x2.0mm
- removed TP2: Cell 2, TestPoint:TestPoint_Pad_2.0x2.0mm
- removed TP3: Cell 3, TestPoint:TestPoint_Pad_2.0x2.0mm
- removed TP4: Cell 4, TestPoint:TestPoint_Pad_2.0x2.0mm
- removed TP5: Cell 5, TestPoint:TestPoint_Pad_2.0x2.0mm
- removed TP6: Cell 6, TestPoint:TestPoint_Pad_2.0x2.0mm
- removed TP7: GND, TestPoint:TestPoint_Pad_2.0x2.0mm
- removed U32, U33: ~, Converter_DCDC:Converter_DCDC_TRACO_TSR-1_THT
- added C101: 10uF, Capacitor_SMD:C_1206_3216Metric, F.Cu at (531.9, 88.5)
- added C102: 10uF, Capacitor_SMD:C_1210_3225Metric, F.Cu at (526.2, 76.2)
- added C103: 10uF, Capacitor_SMD:C_1210_3225Metric, F.Cu at (526.2, 80.4)
- added C104: 10uF, Capacitor_SMD:C_1210_3225Metric, F.Cu at (526.2, 84.7)
- added C105: 10uF, Capacitor_SMD:C_1210_3225Metric, F.Cu at (531.8, 67.7)
- added C106: 10uF, Capacitor_SMD:C_1210_3225Metric, F.Cu at (531.8, 71.9)
- added C107: 10uF, Capacitor_SMD:C_1210_3225Metric, F.Cu at (531.8, 76.2)
- added C108: 10uF, Capacitor_SMD:C_1206_3216Metric, F.Cu at (531.9, 91.8)
- added C109: 10uF, Capacitor_SMD:C_1210_3225Metric, F.Cu at (526.2, 43.6)
- added C110: 10uF, Capacitor_SMD:C_1210_3225Metric, F.Cu at (526.2, 47.9)
- added C111: 10uF, Capacitor_SMD:C_1206_3216Metric, F.Cu at (531.9, 55.9)
- added C112: 10uF, Capacitor_SMD:C_1210_3225Metric, F.Cu at (526.2, 52.1)
- added C113: 10uF, Capacitor_SMD:C_1210_3225Metric, F.Cu at (531.8, 35.1)
- added C114: 10uF, Capacitor_SMD:C_1210_3225Metric, F.Cu at (531.8, 39.4)
- added C115: 10uF, Capacitor_SMD:C_1210_3225Metric, F.Cu at (531.8, 43.6)
- added C116: 10uF, Capacitor_SMD:C_1206_3216Metric, F.Cu at (531.9, 59.3)
- added D40: LED, LED_SMD:LED_0603_1608Metric_Pad1.05x0.95mm_HandSolder, F.Cu at (536.9, 69.4)
- added L3: 2.2uH 3A, Inductor_SMD:L_Vishay_IHLP-1212, F.Cu at (526.2, 93.8)
- added L4: 2.2uH 3A, Inductor_SMD:L_Vishay_IHLP-1212, F.Cu at (526.2, 61.2)
- added R125: 1.5K, Resistor_SMD:R_0402_1005Metric, F.Cu at (536.1, 73.7)
- added R126: 1.5K, Resistor_SMD:R_0402_1005Metric, F.Cu at (536.1, 41.2)
- added U50: 24V->3.3V 3A, Converter_DCDC:Converter_DCDC_RECOM_RPMx.x-x.0, F.Cu at (515.7, 88.4)
- added U51: 24V->5V 3A, Converter_DCDC:Converter_DCDC_RECOM_RPMx.x-x.0, F.Cu at (515.7, 55.9)
- C10, C11: value 100uF -> 10uF; footprint Capacitor_SMD:CP_Elec_10x10 -> Capacitor_SMD:C_1210_3225Metric
- C12: value 680uF -> 10uF; footprint 0UCIRP-KiCAD-Lib:EEV-FK1V681Q -> Capacitor_SMD:C_1210_3225Metric
- C13: value 330uF -> 10uF; footprint Capacitor_SMD:CP_Elec_10x12.6 -> Capacitor_SMD:C_1210_3225Metric
- D5, D6: value 700mV 5A -> LED; footprint Diode_SMD:D_SMC -> LED_SMD:LED_0603_1608Metric_Pad1.05x0.95mm_HandSolder
- L1: value 33uH -> 2.2uH 3A; footprint Inductor_SMD:L_12x12mm_H8mm -> Inductor_SMD:L_Vishay_IHLP-1212
- L2: value 68uH -> 2.2uH 3A; footprint Inductor_SMD:L_12x12mm_H8mm -> Inductor_SMD:L_Vishay_IHLP-1212
- U6: value LM2596S-3.3 -> 24V->5V 3A; footprint Package_TO_SOT_SMD:TO-263-5_TabPin3 -> Converter_DCDC:Converter_DCDC_RECOM_RPMx.x-x.0
- U7: value LM2596S-5 -> 24V->3.3V 3A; footprint Package_TO_SOT_SMD:TO-263-5_TabPin3 -> Converter_DCDC:Converter_DCDC_RECOM_RPMx.x-x.0
- moved C85 263.2 mm to (90.1, 107.3), turned to -90 degrees
- moved C87 263.0 mm to (88.5, 107.3), turned to -90 degrees
- moved Y2 261.3 mm to (90.0, 103.4), turned to -90 degrees
- moved R103 252.9 mm to (86.8, 103.9), turned to -90 degrees
- moved C86 250.7 mm to (95.1, 86.2)
- moved C73 246.6 mm to (114.4, 115.6), turned to 180 degrees
- moved C88 238.8 mm to (87.1, 107.8), turned to -90 degrees
- moved R104 236.6 mm to (98.4, 86.1), turned to 90 degrees
- moved D8 235.0 mm to (536.9, 36.9), turned to 0 degrees
- moved R17 234.4 mm to (536.1, 39.2), turned to 0 degrees
- moved C89 233.5 mm to (90.0, 101.5), turned to 180 degrees
- moved C75 232.2 mm to (90.0, 100.4)
- moved C84 231.8 mm to (90.5, 93.2), turned to 90 degrees
- moved D6 230.8 mm to (536.9, 34.3), turned to 0 degrees
- moved C90 230.5 mm to (121.0, 103.7), turned to -90 degrees
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Connections:
- C10 pad 1: Net-(D2-K) -> Net-(D3-K)
- C11 pad 1: Net-(D3-K) -> +24V
- C12 pad 1: +3V3 -> Net-(D3-K)
- C13 pad 1: Net-(U7-FB) -> +24V
- D5 pad 1: Net-(D5-K) -> GND
- D5 pad 2: GND -> Net-(D5-A)
- D6 pad 1: Net-(D6-K) -> GND
- D6 pad 2: GND -> Net-(D6-A)
- J3 pad A4: Net-(U7-FB) -> Net-(U6-Sense)
- J3 pad A9: Net-(U7-FB) -> Net-(U6-Sense)
- J3 pad B4: Net-(U7-FB) -> Net-(U6-Sense)
- J3 pad B9: Net-(U7-FB) -> Net-(U6-Sense)
- L1 pad 1: Net-(D5-K) -> Net-(D3-K)
- L1 pad 2: +3V3 -> Net-(C107-Pad1)
- L2 pad 1: Net-(D6-K) -> +24V
- L2 pad 2: Net-(U7-FB) -> Net-(C110-Pad1)
- R17 pad 1: Net-(U7-FB) -> Net-(U7-PGood)
- R17 pad 2: Net-(D8-A) -> Net-(D6-A)
- R19 pad 1: +3V3 -> Net-(U6-PGood)
- R19 pad 2: Net-(D9-A) -> Net-(D5-A)
Routing:
- net +3.3V: track 58.1 -> 104.2 mm
- net Net-(D6-K): track 20.0 -> 0.00 mm
- net Net-(U7-FB): track 18.2 -> 0.00 mm
- net +3V3: track 30.7 -> 13.0 mm
- net Net-(D5-K): track 14.7 -> 0.00 mm
- net Net-(D3-K): track 10.9 -> 0.00 mm
- net +24V: track 46.3 -> 35.4 mm
- net Net-(D2-K): track 10.1 -> 0.00 mm
- net MCU_nRST: track 0.00 -> 7.16 mm
- net +5V: track 19.0 -> 12.4 mm
- net Net-(U40F-VCAPDSI): track 0.00 -> 5.49 mm
- net Net-(U40A-VCAP2): track 0.00 -> 3.52 mm
- net Net-(U40E-PH0): track 0.00 -> 3.14 mm
- net Net-(U8-PD0): track 0.00 -> 2.34 mm
- net Net-(U40A-VCAP1): track 0.00 -> 1.98 mm
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- added copper zone on In2.Cu, net +3.3V

Commit message: made reg circuits
Parts:
- moved J3 330.7 mm to (661.8, 138.2)
- moved D3 250.6 mm to (676.0, 141.1)
- moved C10 170.5 mm to (690.7, 112.7)
- moved C108 170.5 mm to (696.4, 136.9)
- moved C12 170.5 mm to (690.7, 117.0)
- moved D5 170.5 mm to (701.3, 111.9)
- moved C106 170.5 mm to (696.3, 117.0)
- moved C107 170.5 mm to (696.3, 121.2)
- moved L1 170.5 mm to (690.7, 134.2)
- moved R19 170.5 mm to (700.6, 116.8)
- moved U6 170.5 mm to (680.2, 118.2)
- moved D4 134.2 mm to (497.7, 49.3), turned to 180 degrees
- moved D2 130.8 mm to (497.7, 50.9), turned to 180 degrees
- moved L4 66.1 mm to (510.2, -2.92), turned to 90 degrees
- moved C111 64.2 mm to (563.6, 0.13), turned to -90 degrees
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Routing:
- net +24V: track 35.4 -> 67.2 mm
- net Net-(C110-Pad1): track 0.00 -> 27.4 mm
- net Net-(D2-K): track 0.00 -> 24.7 mm
- net Net-(C115-Pad1): track 0.00 -> 22.6 mm
- net Net-(C105-Pad1): track 0.00 -> 16.2 mm
- net +5V: track 12.4 -> 21.2 mm
- net +3.3V: track 104.2 -> 113.1 mm
- net +3V3: track 13.0 -> 21.8 mm
- net Net-(U50-PGood): track 0.00 -> 6.36 mm
- net Net-(U51-PGood): track 0.00 -> 6.22 mm
- net Net-(U7-PGood): track 0.00 -> 6.14 mm
- net Net-(D40-A): track 0.00 -> 1.88 mm
- net Net-(D6-A): track 0.00 -> 1.88 mm
- net Net-(D8-A): track 0.00 -> 1.80 mm
- added copper zone on F.Cu, net +3.3V
- added copper zone on F.Cu, net +3V3
- added copper zone on F.Cu, net +5V
