File: rocket2-ecu.kicad_pcb (KiCad board)
At the start: 6 copper layers, 150 x 100 mm, 1 part

Commit message: idk what I changed tbh
Parts:
- added C1: 100nF, Capacitor_SMD:C_0402_1005Metric, F.Cu at (16.0, 21.4)
- added C10: 10uF, Capacitor_SMD:C_1210_3225Metric, F.Cu at (-66.8, 7.47)
- added C100: 100nF, Capacitor_SMD:C_0402_1005Metric, F.Cu at (-99.1, 64.2)
- added C101: 10uF, Capacitor_SMD:C_1206_3216Metric, F.Cu at (-41.6, 0.28)
- added C102: 10uF, Capacitor_SMD:C_1210_3225Metric, F.Cu at (-66.8, 16.0)
- added C103: 10uF, Capacitor_SMD:C_1210_3225Metric, F.Cu at (-66.8, 20.2)
- added C104: 10uF, Capacitor_SMD:C_1210_3225Metric, F.Cu at (-66.8, 24.5)
- added C105: 10uF, Capacitor_SMD:C_1210_3225Metric, F.Cu at (-61.2, 7.47)
- added C106: 10uF, Capacitor_SMD:C_1210_3225Metric, F.Cu at (-61.2, 11.7)
- added C107: 10uF, Capacitor_SMD:C_1210_3225Metric, F.Cu at (-61.2, 16.0)
- added C108: 10uF, Capacitor_SMD:C_1206_3216Metric, F.Cu at (-41.6, 3.62)
- added C109: 10uF, Capacitor_SMD:C_1210_3225Metric, F.Cu at (-66.8, 95.3)
- added C11: 10uF, Capacitor_SMD:C_1210_3225Metric, F.Cu at (-66.8, 86.8)
- added C110: 10uF, Capacitor_SMD:C_1210_3225Metric, F.Cu at (-66.8, 99.5)
- added C111: 10uF, Capacitor_SMD:C_1206_3216Metric, F.Cu at (-55.5, 86.3)
- added C112: 10uF, Capacitor_SMD:C_1210_3225Metric, F.Cu at (-66.8, 103.8)
- added C113: 10uF, Capacitor_SMD:C_1210_3225Metric, F.Cu at (-61.2, 86.8)
- added C114: 10uF, Capacitor_SMD:C_1210_3225Metric, F.Cu at (-61.2, 91.0)
- added C115: 10uF, Capacitor_SMD:C_1210_3225Metric, F.Cu at (-61.2, 95.3)
- added C116: 10uF, Capacitor_SMD:C_1206_3216Metric, F.Cu at (-55.5, 89.7)
- added C117: 2.2uF, Capacitor_SMD:C_0402_1005Metric, F.Cu at (16.0, 31.2)
- added C12: 10uF, Capacitor_SMD:C_1210_3225Metric, F.Cu at (-66.8, 11.7)
- added C13: 10uF, Capacitor_SMD:C_1210_3225Metric, F.Cu at (-66.8, 91.0)
- added C14: 4.7uF, Capacitor_SMD:C_0603_1608Metric, F.Cu at (-34.9, 6.61)
- added C15: 100nF, Capacitor_SMD:C_0402_1005Metric, F.Cu at (-68.2, 29.6)
- added C16: 100nF, Capacitor_SMD:C_0402_1005Metric, F.Cu at (-68.2, 31.5)
- added C17: 100nF, Capacitor_SMD:C_0402_1005Metric, F.Cu at (-68.2, 33.5)
- added C18: 100nF, Capacitor_SMD:C_0402_1005Metric, F.Cu at (-68.2, 35.5)
- added C19: 100nF, Capacitor_SMD:C_0402_1005Metric, F.Cu at (-68.2, 37.4)
- added C2: 100nF, Capacitor_SMD:C_0402_1005Metric, F.Cu at (16.0, 23.3)
- added C20: 10uF, Capacitor_SMD:C_0603_1608Metric, F.Cu at (-34.9, 9.12)
- added C21: 1uF, Capacitor_SMD:C_0603_1608Metric, F.Cu at (-11.5, 53.1)
- added C22: 10uF, Capacitor_SMD:C_0603_1608Metric, F.Cu at (-11.5, 55.6)
- added C23: 1uF, Capacitor_SMD:C_0603_1608Metric, F.Cu at (-11.5, 58.1)
- added C24: 1uF, Capacitor_SMD:C_0603_1608Metric, F.Cu at (-37.6, 53.1)
- added C25: 10uF, Capacitor_SMD:C_0603_1608Metric, F.Cu at (-37.6, 55.6)
- added C26: 1uF, Capacitor_SMD:C_0603_1608Metric, F.Cu at (-37.6, 58.1)
- added C27: 1uF, Capacitor_SMD:C_0603_1608Metric, F.Cu at (-11.5, 107.7)
- added C28: 10uF, Capacitor_SMD:C_0603_1608Metric, F.Cu at (-11.5, 110.2)
- added C29: 1uF, Capacitor_SMD:C_0603_1608Metric, F.Cu at (-11.5, 112.7)
- added C3: 100nF, Capacitor_SMD:C_0402_1005Metric, F.Cu at (16.0, 25.3)
- added C30: 1uF, Capacitor_SMD:C_0603_1608Metric, F.Cu at (-37.6, 107.7)
- added C31: 10uF, Capacitor_SMD:C_0603_1608Metric, F.Cu at (-37.6, 110.2)
- added C32: 1uF, Capacitor_SMD:C_0603_1608Metric, F.Cu at (-37.6, 112.7)
- added C33: 1uF, Capacitor_SMD:C_0603_1608Metric, F.Cu at (-11.5, 80.4)
- added C34: 10uF, Capacitor_SMD:C_0603_1608Metric, F.Cu at (-11.5, 82.9)
- added C35: 1uF, Capacitor_SMD:C_0603_1608Metric, F.Cu at (-11.5, 85.4)
- added C36: 1uF, Capacitor_SMD:C_0603_1608Metric, F.Cu at (-37.6, 80.4)
- added C37: 10uF, Capacitor_SMD:C_0603_1608Metric, F.Cu at (-37.6, 82.9)
- added C38: 1uF, Capacitor_SMD:C_0603_1608Metric, F.Cu at (-37.6, 85.4)
- added C39: 100nF, Capacitor_SMD:C_0402_1005Metric, F.Cu at (-61.5, 124.2)
- added C4: 100nF, Capacitor_SMD:C_0402_1005Metric, F.Cu at (16.0, 27.3)
- added C40: 100nF, Capacitor_SMD:C_0402_1005Metric, F.Cu at (-111.4, 86.5)
- added C41: 10nF, Capacitor_SMD:C_0402_1005Metric, F.Cu at (-122.7, 62.2)
- added C42: 100nF, Capacitor_SMD:C_0402_1005Metric, F.Cu at (-122.7, 64.2)
- added C43: 100nF, Capacitor_SMD:C_0402_1005Metric, F.Cu at (-108.8, 131.8)
- added C48: 100nF, Capacitor_SMD:C_0402_1005Metric, F.Cu at (-129.3, 131.8)
- added C49: 100nF, Capacitor_SMD:C_0402_1005Metric, F.Cu at (-108.8, 110.7)
- added C5: 100nF, Capacitor_SMD:C_0402_1005Metric, F.Cu at (16.0, 29.3)
- added C50: 100nF, Capacitor_SMD:C_0402_1005Metric, F.Cu at (-11.3, 129.4)
- added C51: 100nF, Capacitor_SMD:C_0402_1005Metric, F.Cu at (-37.4, 129.4)
- added C52: 100nF, Capacitor_SMD:C_0402_1005Metric, F.Cu at (14.8, 102.0)
- added C53: 4.7uF, Capacitor_SMD:C_0603_1608Metric, F.Cu at (-124.7, 87.0)
- added C54: 100nF, Capacitor_SMD:C_0402_1005Metric, F.Cu at (-125.3, 70.8)
- added C55: 100nF, Capacitor_SMD:C_0402_1005Metric, F.Cu at (-125.3, 72.8)
- added C56: 100nF, Capacitor_SMD:C_0402_1005Metric, F.Cu at (-125.3, 74.8)
- added C57: 100nF, Capacitor_SMD:C_0402_1005Metric, F.Cu at (-125.3, 76.7)
- added C58: 100nF, Capacitor_SMD:C_0402_1005Metric, F.Cu at (-125.3, 78.7)
- added C59: 100nF, Capacitor_SMD:C_0402_1005Metric, F.Cu at (-83.5, 69.9)
- added C6: 10uF, Capacitor_SMD:C_0603_1608Metric, F.Cu at (-5.67, 32.4)
- added C60: 100nF, Capacitor_SMD:C_0402_1005Metric, F.Cu at (-83.5, 71.8)
- added C61: 100nF, Capacitor_SMD:C_0402_1005Metric, F.Cu at (-83.5, 73.8)
- added C62: 100nF, Capacitor_SMD:C_0402_1005Metric, F.Cu at (-83.5, 75.8)
- added C63: 100nF, Capacitor_SMD:C_0402_1005Metric, F.Cu at (-83.5, 77.7)
- added C64: 100nF, Capacitor_SMD:C_0402_1005Metric, F.Cu at (-83.5, 79.7)
- added C65: 100nF, Capacitor_SMD:C_0402_1005Metric, F.Cu at (-83.5, 81.7)
- added C66: 100nF, Capacitor_SMD:C_0402_1005Metric, F.Cu at (-80.6, 69.9)
- added C67: 100nF, Capacitor_SMD:C_0402_1005Metric, F.Cu at (-80.6, 71.8)
- added C68: 100nF, Capacitor_SMD:C_0402_1005Metric, F.Cu at (-80.6, 73.8)
- added C69: 2.2uF, Capacitor_SMD:C_0603_1608Metric, F.Cu at (-54.5, 41.7)
- added C7: 100nF, Capacitor_SMD:C_0402_1005Metric, F.Cu at (-75.1, 124.2)
- added C70: 100nF, Capacitor_SMD:C_0402_1005Metric, F.Cu at (-80.6, 75.8)
- added C71: 100nF, Capacitor_SMD:C_0402_1005Metric, F.Cu at (-80.6, 77.7)
- added C72: 100nF, Capacitor_SMD:C_0402_1005Metric, F.Cu at (-80.6, 79.7)
- added C73: 2.2uF, Capacitor_SMD:C_0603_1608Metric, F.Cu at (-54.5, 44.2)
- added C74: 100nF, Capacitor_SMD:C_0402_1005Metric, F.Cu at (-80.6, 81.7)
- added C75: 100nF, Capacitor_SMD:C_0402_1005Metric, F.Cu at (-77.7, 69.9)
- added C76: 10uF, Capacitor_SMD:C_0603_1608Metric, F.Cu at (-54.5, 46.7)
- added C77: 100nF, Capacitor_SMD:C_0402_1005Metric, F.Cu at (-77.7, 71.8)
- added C78: 100nF, Capacitor_SMD:C_0402_1005Metric, F.Cu at (-77.7, 73.8)
- added C79: 100nF, Capacitor_SMD:C_0402_1005Metric, F.Cu at (-77.7, 75.8)
- added C8: 100nF, Capacitor_SMD:C_0402_1005Metric, F.Cu at (-129.3, 110.7)
- added C80: 100nF, Capacitor_SMD:C_0402_1005Metric, F.Cu at (-77.7, 77.7)
- added C81: 100nF, Capacitor_SMD:C_0402_1005Metric, F.Cu at (-77.7, 79.7)
- added C82: 100nF, Capacitor_SMD:C_0402_1005Metric, F.Cu at (-77.7, 81.7)
- added C83: 100nF, Capacitor_SMD:C_0402_1005Metric, F.Cu at (-74.9, 69.9)
- added C84: 100nF, Capacitor_SMD:C_0402_1005Metric, F.Cu at (-74.9, 71.8)
- added C85: 1uF, Capacitor_SMD:C_0603_1608Metric, F.Cu at (-54.5, 49.3)
- added C86: 4.7uF, Capacitor_SMD:C_0603_1608Metric, F.Cu at (-54.5, 51.8)
- added C87: 1uF, Capacitor_SMD:C_0603_1608Metric, F.Cu at (-54.5, 54.3)
- added C88: 100nF, Capacitor_SMD:C_0402_1005Metric, F.Cu at (-74.9, 73.8)
- added C89: 100nF, Capacitor_SMD:C_0402_1005Metric, F.Cu at (-74.9, 75.8)
- added C9: 100nF, Capacitor_SMD:C_0402_1005Metric, F.Cu at (-68.2, 27.6)
- added C90: 2.2uF, Capacitor_SMD:C_0603_1608Metric, F.Cu at (-54.5, 56.8)
- added C91: 100nF, Capacitor_SMD:C_0402_1005Metric, F.Cu at (15.8, 129.4)
- added C92: 100nF, Capacitor_SMD:C_0402_1005Metric, F.Cu at (14.8, 47.4)
- added C93: 10uF, Capacitor_SMD:C_0603_1608Metric, F.Cu at (-114.4, 10.7)
- added C94: 10uF, Capacitor_SMD:C_0603_1608Metric, F.Cu at (-114.4, 13.2)
- added C95: 10uF, Capacitor_SMD:C_0603_1608Metric, F.Cu at (-114.4, 15.7)
- added C96: 100nF, Capacitor_SMD:C_0402_1005Metric, F.Cu at (16.5, 72.7)
- added C97: 100nF, Capacitor_SMD:C_0402_1005Metric, F.Cu at (16.5, 74.7)
- added C98: 100nF, Capacitor_SMD:C_0402_1005Metric, F.Cu at (2.29, 129.4)
- added C99: 10nF, Capacitor_SMD:C_0402_1005Metric, F.Cu at (-99.1, 62.2)
- added D1: 30V 2A, 0UCIRP-KiCAD-Lib:NSR20F30NXT5G, F.Cu at (-31.1, -11.5)
- added D10: LED, LED_SMD:LED_0603_1608Metric_Pad1.05x0.95mm_HandSolder, F.Cu at (-82.7, 24.2)
- added D11: 5.1V, Diode_SMD:D_MiniMELF, F.Cu at (-81.7, 127.2)
- added D12: LED, LED_SMD:LED_0603_1608Metric_Pad1.05x0.95mm_HandSolder, F.Cu at (-82.7, 26.8)
- added D13: LED, LED_SMD:LED_0603_1608Metric_Pad1.05x0.95mm_HandSolder, F.Cu at (-82.7, 29.4)
- added D14: LED, LED_SMD:LED_0603_1608Metric_Pad1.05x0.95mm_HandSolder, F.Cu at (-82.7, 32.0)
- added D15: LED, LED_SMD:LED_0603_1608Metric_Pad1.05x0.95mm_HandSolder, F.Cu at (-82.7, 34.6)
- added D16: LED, LED_SMD:LED_0603_1608Metric_Pad1.05x0.95mm_HandSolder, F.Cu at (-7.30, 57.3)
- added D17: LED, LED_SMD:LED_0603_1608Metric_Pad1.05x0.95mm_HandSolder, F.Cu at (-33.4, 57.3)
- added D18: LED, LED_SMD:LED_0603_1608Metric_Pad1.05x0.95mm_HandSolder, F.Cu at (-7.30, 111.9)
- added D19: LED, LED_SMD:LED_0603_1608Metric_Pad1.05x0.95mm_HandSolder, F.Cu at (-33.4, 111.9)
- added D2: 30V 2A, 0UCIRP-KiCAD-Lib:NSR20F30NXT5G, F.Cu at (-31.1, -9.04)
- added D20: LED, LED_SMD:LED_0603_1608Metric_Pad1.05x0.95mm_HandSolder, F.Cu at (-7.30, 84.6)
- added D21: LED, LED_SMD:LED_0603_1608Metric_Pad1.05x0.95mm_HandSolder, F.Cu at (-33.4, 84.6)
- added D22: 5.1V, Diode_SMD:D_MiniMELF, F.Cu at (-68.1, 127.2)
- added D23: 100V 8A, Diode_SMD:D_PowerDI-5, F.Cu at (-105.5, 83.4)
- added D24: 3.3V, Diode_SMD:D_SOD-123, F.Cu at (-115.7, 87.2)
- added D25: 100V 8A, Diode_SMD:D_PowerDI-5, F.Cu at (-102.9, 128.7)
- added D26: 3.3V, Diode_SMD:D_SOD-123, F.Cu at (-113.1, 132.5)
- added D27: 100V 8A, Diode_SMD:D_PowerDI-5, F.Cu at (-123.5, 128.7)
- added D28: 3.3V, Diode_SMD:D_SOD-123, F.Cu at (-133.6, 132.5)
- added D29: 100V 8A, Diode_SMD:D_PowerDI-5, F.Cu at (-102.9, 107.6)
- added D3: 30V 5A, Diode_SMD:D_SOD-128, F.Cu at (-35.0, 0.62)
- added D30: 3.3V, Diode_SMD:D_SOD-123, F.Cu at (-113.1, 111.4)
- added D31: 5.1V, Diode_SMD:D_MiniMELF, F.Cu at (-17.9, 132.4)
- added D32: 5.1V, Diode_SMD:D_MiniMELF, F.Cu at (-44.0, 132.4)
- added D33: 5.1V, Diode_SMD:D_MiniMELF, F.Cu at (8.23, 105.1)
- added D34: 6.8V, Diode_SMD:D_0402_1005Metric, F.Cu at (-54.8, 59.0)
- added D35: 6.8V, Diode_SMD:D_0402_1005Metric, F.Cu at (-54.8, 61.0)
- added D36: LED, LED_SMD:LED_0603_1608Metric_Pad1.05x0.95mm_HandSolder, F.Cu at (-52.2, 78.6)
- added D37: 5.1V, Diode_SMD:D_MiniMELF, F.Cu at (9.21, 132.4)
- added D38: 5.1V, Diode_SMD:D_MiniMELF, F.Cu at (8.23, 50.4)
- added D39: 5.1V, Diode_SMD:D_MiniMELF, F.Cu at (-4.33, 132.4)
- added D4: 30V 2A, 0UCIRP-KiCAD-Lib:NSR20F30NXT5G, F.Cu at (-31.1, -6.57)
- added D40: LED, LED_SMD:LED_0603_1608Metric_Pad1.05x0.95mm_HandSolder, F.Cu at (-82.7, 37.2)
- added D41: 100V 8A, Diode_SMD:D_PowerDI-5, F.Cu at (-123.5, 107.6)
- added D42: 3.3V, Diode_SMD:D_SOD-123, F.Cu at (-133.6, 111.4)
- added D5: LED, LED_SMD:LED_0603_1608Metric_Pad1.05x0.95mm_HandSolder, F.Cu at (-82.7, 19.0)
- added D6: LED, LED_SMD:LED_0603_1608Metric_Pad1.05x0.95mm_HandSolder, F.Cu at (-56.1, 92.7)
- added D7: 30V 2A, 0UCIRP-KiCAD-Lib:NSR20F30NXT5G, F.Cu at (-31.1, -4.09)
- added D8: LED, LED_SMD:LED_0603_1608Metric_Pad1.05x0.95mm_HandSolder, F.Cu at (-56.1, 95.3)
- added D9: LED, LED_SMD:LED_0603_1608Metric_Pad1.05x0.95mm_HandSolder, F.Cu at (-82.7, 21.6)
- added FB1: 470ohm @100MHz, Inductor_SMD:L_0603_1608Metric, F.Cu at (-126.1, 62.5)
- added FB2: 470ohm @100MHz, Inductor_SMD:L_0603_1608Metric, F.Cu at (-126.1, 65.0)
- added FB3: 470ohm @100MHz, Inductor_SMD:L_0603_1608Metric, F.Cu at (-102.5, 62.5)
- added FB4: 470ohm @100MHz, Inductor_SMD:L_0603_1608Metric, F.Cu at (-102.5, 65.0)
- added H1: MountingHole_Pad, MountingHole:MountingHole_4.3mm_M4_Pad_Via, F.Cu at (-22.1, -7.67)
- added H2: MountingHole_Pad, MountingHole:MountingHole_4.3mm_M4_Pad_Via, F.Cu at (-22.1, 2.48)
- added H3: MountingHole_Pad, MountingHole:MountingHole_4.3mm_M4_Pad_Via, F.Cu at (-22.1, 12.6)
- added H4: MountingHole_Pad, MountingHole:MountingHole_4.3mm_M4_Pad_Via, F.Cu at (-22.1, 22.8)
- added J1: ALARM, Buzzer_Beeper:Buzzer_TDK_PS1240P02BT_D12.2mm_H6.5mm, F.Cu at (5.20, 27.3)
- added J10: Solenoid, 0UCIRP-KiCAD-Lib:GX-16 3 pin, F.Cu at (-110.7, 94.8)
- added J11: PT, 0UCIRP-KiCAD-Lib:GX-12 3 pin, F.Cu at (-16.9, 123.2)
- added J12: PT, 0UCIRP-KiCAD-Lib:GX-12 3 pin, F.Cu at (-43.0, 123.2)
- added J13: PT, 0UCIRP-KiCAD-Lib:GX-12 3 pin, F.Cu at (9.21, 95.8)
- added J14: PT, 0UCIRP-KiCAD-Lib:GX-12 3 pin, F.Cu at (-80.7, 118.0)
- added J15: GNSS SMA, Connector_Coaxial:SMA_Molex_73251-2200_Horizontal, F.Cu at (-131.6, 87.4)
- added J16: USB-C, Connector_USB:USB_C_Receptacle_GCT_USB4105-xx-A_16P_TopMnt_Horizontal, F.Cu at (-67.6, 74.2)
- added J17: ARM Cortex Debug, Connector_PinHeader_1.27mm:PinHeader_2x05_P1.27mm_Vertical_SMD, F.Cu at (-54.0, 73.1)
- added J18: PT, 0UCIRP-KiCAD-Lib:GX-12 3 pin, F.Cu at (10.2, 123.2)
- added J19: PT, 0UCIRP-KiCAD-Lib:GX-12 3 pin, F.Cu at (9.21, 41.2)
- added J2: Conn_01x07, Connector_JST:JST_PH_B7B-PH-K_1x07_P2.00mm_Vertical, F.Cu at (-45.5, 22.0)
- added J20: SMA, Connector_Coaxial:SMA_Molex_73251-2200_Horizontal, F.Cu at (-111.5, 4.78)
- added J21: SMA, Connector_Coaxial:SMA_Molex_73251-2200_Horizontal, F.Cu at (-101.7, 4.78)
- added J22: SMA, Connector_Coaxial:SMA_Molex_73251-2200_Horizontal, F.Cu at (-91.8, 4.78)
- added J23: PT, 0UCIRP-KiCAD-Lib:GX-12 3 pin, F.Cu at (-3.35, 123.2)
- added J24: XT60, Connector_AMASS:AMASS_XT60PW-M_1x02_P7.20mm_Horizontal, F.Cu at (-11.8, 23.7)
- added J25: Solenoid, 0UCIRP-KiCAD-Lib:GX-16 3 pin, F.Cu at (-131.3, 94.8)
- added J3: USB-C, Connector_USB:USB_C_Receptacle_GCT_USB4105-xx-A_16P_TopMnt_Horizontal, F.Cu at (-42.7, 31.1)
- added J4: SMA, Connector_Coaxial:SMA_Molex_73251-2200_Horizontal, F.Cu at (-53.4, 22.9)
- added J5: ARM Cortex Debug, Connector_PinHeader_1.27mm:PinHeader_2x05_P1.27mm_Vertical_SMD, F.Cu at (-53.5, 31.8)
- added J6: PT, 0UCIRP-KiCAD-Lib:GX-12 3 pin, F.Cu at (-67.2, 118.0)
- added J7: Solenoid, 0UCIRP-KiCAD-Lib:GX-16 3 pin, F.Cu at (-113.3, 70.6)
- added J8: Solenoid, 0UCIRP-KiCAD-Lib:GX-16 3 pin, F.Cu at (-110.7, 115.8)
- added J9: Solenoid, 0UCIRP-KiCAD-Lib:GX-16 3 pin, F.Cu at (-131.3, 115.8)
- added L1: 2.2uH 3A, Inductor_SMD:L_Vishay_IHLP-1212, F.Cu at (-33.9, 28.2)
- added L2: 2.2uH 3A, Inductor_SMD:L_Vishay_IHLP-1212, F.Cu at (-60.8, 108.2)
- added L3: 2.2uH 3A, Inductor_SMD:L_Vishay_IHLP-1212, F.Cu at (-33.9, 32.8)
- added L4: 2.2uH 3A, Inductor_SMD:L_Vishay_IHLP-1212, F.Cu at (-60.8, 112.9)
- added P3: PAD_SMD, TestPoint:TestPoint_Plated_Hole_D4.0mm, F.Cu at (4.09, 9.81)
- added P4: PAD_SMD, TestPoint:TestPoint_Plated_Hole_D4.0mm, F.Cu at (4.09, 16.9)
- added Q1: DMG3402L, Package_TO_SOT_SMD:SOT-23-3, F.Cu at (-5.11, 29.0)
- added Q10: DMG3402L, Package_TO_SOT_SMD:SOT-23-3, F.Cu at (-102.6, 72.1)
- added Q11: DMG3402L, Package_TO_SOT_SMD:SOT-23-3, F.Cu at (-100.0, 117.3)
- added Q12: DMG3402L, Package_TO_SOT_SMD:SOT-23-3, F.Cu at (-120.6, 117.3)
- added Q13: DMG3402L, Package_TO_SOT_SMD:SOT-23-3, F.Cu at (-100.0, 96.3)
- added Q14: DMG3402L, Package_TO_SOT_SMD:SOT-23-3, F.Cu at (-120.6, 96.3)
- added Q2: Q_NMOS_GSD, Package_TO_SOT_SMD:SOT-23-3, F.Cu at (-47.0, -10.5)
- added Q3: Q_NMOS_GSD, Package_TO_SOT_SMD:SOT-23-3, F.Cu at (-47.0, -6.08)
- added Q4: PMOS, Package_SO:Vishay_PowerPAK_1212-8_Single, F.Cu at (-77.6, 20.2)
- added Q5: PMOS, Package_SO:Vishay_PowerPAK_1212-8_Single, F.Cu at (-77.6, 24.9)
- added Q6: Q_NMOS_GSD, Package_TO_SOT_SMD:SOT-23-3, F.Cu at (-47.0, -1.62)
- added Q7: Q_NMOS_GSD, Package_TO_SOT_SMD:SOT-23-3, F.Cu at (-47.0, 2.83)
- added Q8: PMOS, Package_SO:Vishay_PowerPAK_1212-8_Single, F.Cu at (-77.6, 29.6)
- added Q9: PMOS, Package_SO:Vishay_PowerPAK_1212-8_Single, F.Cu at (-77.6, 34.3)
- added R1: 10K, Resistor_SMD:R_0402_1005Metric, F.Cu at (13.7, 7.29)
- added R10: 10K, Resistor_SMD:R_0402_1005Metric, F.Cu at (-47.0, 10.3)
- added R100: 1K, Resistor_SMD:R_0402_1005Metric, F.Cu at (14.9, 96.1)
- added R101: 5K, Resistor_SMD:R_0402_1005Metric, F.Cu at (14.9, 98.1)
- added R102: 10K, Resistor_SMD:R_0402_1005Metric, F.Cu at (14.9, 100.1)
- added R103: 10K, Resistor_SMD:R_0402_1005Metric, F.Cu at (-60.3, 69.9)
- added R104: 10K, Resistor_SMD:R_0402_1005Metric, F.Cu at (-60.3, 71.9)
- added R105: 5.1K, Resistor_SMD:R_0603_1608Metric_Pad0.98x0.95mm_HandSolder, F.Cu at (-56.6, 78.5)
- added R106: 5.1K, Resistor_SMD:R_0603_1608Metric_Pad0.98x0.95mm_HandSolder, F.Cu at (-56.6, 81.1)
- added R107: 10K, Resistor_SMD:R_0402_1005Metric, F.Cu at (-60.3, 73.9)
- added R108: 10K, Resistor_SMD:R_0402_1005Metric, F.Cu at (-60.3, 75.8)
- added R109: 100, Resistor_SMD:R_0402_1005Metric, F.Cu at (-60.3, 77.8)
- added R11: 1K, Resistor_SMD:R_0402_1005Metric, F.Cu at (-47.0, 12.3)
- added R110: 1K, Resistor_SMD:R_0402_1005Metric, F.Cu at (15.8, 123.4)
- added R111: 5K, Resistor_SMD:R_0402_1005Metric, F.Cu at (15.8, 125.4)
- added R112: 10K, Resistor_SMD:R_0402_1005Metric, F.Cu at (15.8, 127.4)
- added R113: 1K, Resistor_SMD:R_0402_1005Metric, F.Cu at (14.9, 41.5)
- added R114: 5K, Resistor_SMD:R_0402_1005Metric, F.Cu at (14.9, 43.5)
- added R115: 10K, Resistor_SMD:R_0402_1005Metric, F.Cu at (14.9, 45.4)
- added R116: 100K, Resistor_SMD:R_0402_1005Metric, F.Cu at (-115.0, 18.0)
- added R117: 100K, Resistor_SMD:R_0402_1005Metric, F.Cu at (-115.0, 20.0)
- added R118: 100K, Resistor_SMD:R_0402_1005Metric, F.Cu at (-115.0, 22.0)
- added R119: 100K, Resistor_SMD:R_0402_1005Metric, F.Cu at (16.5, 68.8)
- added R12: 100, Resistor_SMD:R_0402_1005Metric, F.Cu at (-47.0, 14.3)
- added R120: 100K, Resistor_SMD:R_0402_1005Metric, F.Cu at (16.5, 70.8)
- added R121: 1K, Resistor_SMD:R_0402_1005Metric, F.Cu at (2.31, 123.4)
- added R122: 5K, Resistor_SMD:R_0402_1005Metric, F.Cu at (2.31, 125.4)
- added R123: 10K, Resistor_SMD:R_0402_1005Metric, F.Cu at (2.31, 127.4)
- added R124: 100K, Resistor_SMD:R_0402_1005Metric, F.Cu at (-96.2, 62.2)
- added R125: 1.5K, Resistor_SMD:R_0402_1005Metric, F.Cu at (-38.3, 6.34)
- added R126: 1.5K, Resistor_SMD:R_0402_1005Metric, F.Cu at (-56.9, 99.5)
- added R127: 15K, Resistor_SMD:R_0402_1005Metric, F.Cu at (-38.3, 8.34)
- added R128: 100K, Resistor_SMD:R_0402_1005Metric, F.Cu at (-38.3, 10.3)
- added R129: 15K, Resistor_SMD:R_0402_1005Metric, F.Cu at (-38.3, 12.3)
- added R13: 15K, Resistor_SMD:R_0402_1005Metric, F.Cu at (-47.0, 16.3)
- added R130: 1K, Resistor_SMD:R_0402_1005Metric, F.Cu at (-38.3, 14.3)
- added R131: 10K, Resistor_SMD:R_0402_1005Metric, F.Cu at (-124.6, 95.0)
- added R132: 100, Resistor_SMD:R_0402_1005Metric, F.Cu at (-124.6, 97.0)
- added R133: 0.1, Resistor_SMD:R_2512_6332Metric, F.Cu at (-132.2, 107.3)
- added R134: 1K, Resistor_SMD:R_0402_1005Metric, F.Cu at (-124.6, 99.0)
- added R14: 10K, Resistor_SMD:R_0402_1005Metric, F.Cu at (-47.0, 18.3)
- added R15: 100, Resistor_SMD:R_0402_1005Metric, F.Cu at (-44.1, 6.34)
- added R16: 100K, Resistor_SMD:R_0402_1005Metric, F.Cu at (-44.1, 8.34)
- added R17: 1.5K, Resistor_SMD:R_0402_1005Metric, F.Cu at (-56.9, 97.5)
- added R18: 15K, Resistor_SMD:R_0402_1005Metric, F.Cu at (-44.1, 10.3)
- added R19: 1.5K, Resistor_SMD:R_0402_1005Metric, F.Cu at (-44.1, 12.3)
- added R2: 100, Resistor_SMD:R_0402_1005Metric, F.Cu at (13.7, 9.28)
- added R20: 1K, Resistor_SMD:R_0402_1005Metric, F.Cu at (-44.1, 14.3)
- added R21: 1K, Resistor_SMD:R_0402_1005Metric, F.Cu at (-44.1, 16.3)
- added R22: 100, Resistor_SMD:R_0402_1005Metric, F.Cu at (-44.1, 18.3)
- added R23: 10K, Resistor_SMD:R_0402_1005Metric, F.Cu at (-41.2, 6.34)
- added R24: 100, Resistor_SMD:R_0402_1005Metric, F.Cu at (-41.2, 8.34)
- added R25: 100K, Resistor_SMD:R_0402_1005Metric, F.Cu at (-41.2, 10.3)
- added R26: 10K, Resistor_SMD:R_0402_1005Metric, F.Cu at (-41.2, 12.3)
- added R27: 10K, Resistor_SMD:R_0402_1005Metric, F.Cu at (-41.2, 14.3)
- added R28: 1.5K, Resistor_SMD:R_0402_1005Metric, F.Cu at (-41.2, 16.3)
- added R29: 1.5K, Resistor_SMD:R_0402_1005Metric, F.Cu at (-41.2, 18.3)
- added R3: 4k7, Resistor_SMD:R_0402_1005Metric, F.Cu at (13.7, 11.3)
- added R30: 27K, Resistor_SMD:R_0603_1608Metric, F.Cu at (-11.5, 60.6)
- added R31: 375, Resistor_SMD:R_0402_1005Metric, F.Cu at (-15.0, 52.8)
- added R32: 10K, Resistor_SMD:R_0402_1005Metric, F.Cu at (-15.0, 54.8)
- added R33: 10K, Resistor_SMD:R_0402_1005Metric, F.Cu at (-15.0, 56.8)
- added R34: 10K, Resistor_SMD:R_0402_1005Metric, F.Cu at (-15.0, 58.8)
- added R35: 1K, Resistor_SMD:R_0402_1005Metric, F.Cu at (-15.0, 60.8)
- added R36: 1.5K, Resistor_SMD:R_0402_1005Metric, F.Cu at (-15.0, 62.8)
- added R37: 27K, Resistor_SMD:R_0603_1608Metric, F.Cu at (-37.6, 60.6)
- added R38: 375, Resistor_SMD:R_0402_1005Metric, F.Cu at (-41.1, 52.8)
- added R39: 10K, Resistor_SMD:R_0402_1005Metric, F.Cu at (-41.1, 54.8)
- added R4: 4k7, Resistor_SMD:R_0402_1005Metric, F.Cu at (13.7, 13.3)
- added R40: 10K, Resistor_SMD:R_0402_1005Metric, F.Cu at (-41.1, 56.8)
- added R41: 10K, Resistor_SMD:R_0402_1005Metric, F.Cu at (-41.1, 58.8)
- added R42: 1K, Resistor_SMD:R_0402_1005Metric, F.Cu at (-41.1, 60.8)
- added R43: 1.5K, Resistor_SMD:R_0402_1005Metric, F.Cu at (-41.1, 62.8)
- added R44: 27K, Resistor_SMD:R_0603_1608Metric, F.Cu at (-11.5, 115.2)
- added R45: 375, Resistor_SMD:R_0402_1005Metric, F.Cu at (-15.0, 107.4)
- added R46: 10K, Resistor_SMD:R_0402_1005Metric, F.Cu at (-15.0, 109.4)
- added R47: 10K, Resistor_SMD:R_0402_1005Metric, F.Cu at (-15.0, 111.4)
- added R48: 10K, Resistor_SMD:R_0402_1005Metric, F.Cu at (-15.0, 113.4)
- added R49: 1K, Resistor_SMD:R_0402_1005Metric, F.Cu at (-15.0, 115.4)
- added R5: 100K, Resistor_SMD:R_0402_1005Metric, F.Cu at (-47.0, 6.34)
- added R50: 1.5K, Resistor_SMD:R_0402_1005Metric, F.Cu at (-15.0, 117.4)
- added R51: 27K, Resistor_SMD:R_0603_1608Metric, F.Cu at (-37.6, 115.2)
- added R52: 375, Resistor_SMD:R_0402_1005Metric, F.Cu at (-41.1, 107.4)
- added R53: 10K, Resistor_SMD:R_0402_1005Metric, F.Cu at (-41.1, 109.4)
- added R54: 10K, Resistor_SMD:R_0402_1005Metric, F.Cu at (-41.1, 111.4)
- added R55: 10K, Resistor_SMD:R_0402_1005Metric, F.Cu at (-41.1, 113.4)
- added R56: 1K, Resistor_SMD:R_0402_1005Metric, F.Cu at (-41.1, 115.4)
- added R57: 1.5K, Resistor_SMD:R_0402_1005Metric, F.Cu at (-41.1, 117.4)
- added R58: 27K, Resistor_SMD:R_0603_1608Metric, F.Cu at (-11.5, 87.9)
- added R59: 375, Resistor_SMD:R_0402_1005Metric, F.Cu at (-15.0, 80.1)
- added R6: 1K, Resistor_SMD:R_0402_1005Metric, F.Cu at (-75.0, 118.2)
- added R60: 10K, Resistor_SMD:R_0402_1005Metric, F.Cu at (-15.0, 82.1)
- added R61: 10K, Resistor_SMD:R_0402_1005Metric, F.Cu at (-15.0, 84.1)
- added R62: 10K, Resistor_SMD:R_0402_1005Metric, F.Cu at (-15.0, 86.1)
- added R63: 1K, Resistor_SMD:R_0402_1005Metric, F.Cu at (-15.0, 88.1)
- added R64: 1.5K, Resistor_SMD:R_0402_1005Metric, F.Cu at (-15.0, 90.1)
- added R65: 27K, Resistor_SMD:R_0603_1608Metric, F.Cu at (-37.6, 87.9)
- added R66: 375, Resistor_SMD:R_0402_1005Metric, F.Cu at (-41.1, 80.1)
- added R67: 10K, Resistor_SMD:R_0402_1005Metric, F.Cu at (-41.1, 82.1)
- added R68: 10K, Resistor_SMD:R_0402_1005Metric, F.Cu at (-41.1, 84.1)
- added R69: 10K, Resistor_SMD:R_0402_1005Metric, F.Cu at (-41.1, 86.1)
- added R7: 5K, Resistor_SMD:R_0402_1005Metric, F.Cu at (-75.0, 120.2)
- added R70: 1K, Resistor_SMD:R_0402_1005Metric, F.Cu at (-41.1, 88.1)
- added R71: 1.5K, Resistor_SMD:R_0402_1005Metric, F.Cu at (-41.1, 90.1)
- added R72: 1K, Resistor_SMD:R_0402_1005Metric, F.Cu at (-61.5, 118.2)
- added R73: 5K, Resistor_SMD:R_0402_1005Metric, F.Cu at (-61.5, 120.2)
- added R74: 10K, Resistor_SMD:R_0402_1005Metric, F.Cu at (-61.5, 122.2)
- added R75: 10K, Resistor_SMD:R_0402_1005Metric, F.Cu at (-106.6, 70.8)
- added R76: 100, Resistor_SMD:R_0402_1005Metric, F.Cu at (-106.6, 72.8)
- added R77: 0.1, Resistor_SMD:R_2512_6332Metric, F.Cu at (-114.2, 83.1)
- added R78: 1K, Resistor_SMD:R_0402_1005Metric, F.Cu at (-106.6, 74.8)
- added R79: 100K, Resistor_SMD:R_0402_1005Metric, F.Cu at (-119.8, 62.2)
- added R8: 10K, Resistor_SMD:R_0402_1005Metric, F.Cu at (-75.0, 122.2)
- added R80: 10K, Resistor_SMD:R_0402_1005Metric, F.Cu at (-104.0, 116.1)
- added R81: 100, Resistor_SMD:R_0402_1005Metric, F.Cu at (-104.0, 118.1)
- added R82: 0.1, Resistor_SMD:R_2512_6332Metric, F.Cu at (-111.6, 128.4)
- added R83: 1K, Resistor_SMD:R_0402_1005Metric, F.Cu at (-104.0, 120.1)
- added R84: 0, Resistor_SMD:R_1206_3216Metric_Pad1.30x1.75mm_HandSolder, F.Cu at (-66.7, 107.6)
- added R85: 0, Resistor_SMD:R_1206_3216Metric_Pad1.30x1.75mm_HandSolder, F.Cu at (-66.7, 110.9)
- added R86: 10K, Resistor_SMD:R_0402_1005Metric, F.Cu at (-124.6, 116.1)
- added R87: 100, Resistor_SMD:R_0402_1005Metric, F.Cu at (-124.6, 118.1)
- added R88: 0.1, Resistor_SMD:R_2512_6332Metric, F.Cu at (-132.2, 128.4)
- added R89: 1K, Resistor_SMD:R_0402_1005Metric, F.Cu at (-124.6, 120.1)
- added R9: 100K, Resistor_SMD:R_0402_1005Metric, F.Cu at (-47.0, 8.34)
- added R90: 10K, Resistor_SMD:R_0402_1005Metric, F.Cu at (-104.0, 95.0)
- added R91: 100, Resistor_SMD:R_0402_1005Metric, F.Cu at (-104.0, 97.0)
- added R92: 0.1, Resistor_SMD:R_2512_6332Metric, F.Cu at (-111.6, 107.3)
- added R93: 1K, Resistor_SMD:R_0402_1005Metric, F.Cu at (-104.0, 99.0)
- added R94: 1K, Resistor_SMD:R_0402_1005Metric, F.Cu at (-11.2, 123.4)
- added R95: 5K, Resistor_SMD:R_0402_1005Metric, F.Cu at (-11.2, 125.4)
- added R96: 10K, Resistor_SMD:R_0402_1005Metric, F.Cu at (-11.2, 127.4)
- added R97: 1K, Resistor_SMD:R_0402_1005Metric, F.Cu at (-37.3, 123.4)
- added R98: 5K, Resistor_SMD:R_0402_1005Metric, F.Cu at (-37.3, 125.4)
- added R99: 10K, Resistor_SMD:R_0402_1005Metric, F.Cu at (-37.3, 127.4)
- added TC1: Thermocouple, 0UCIRP-KiCAD-Lib:AM-K-PCB, F.Cu at (-125.8, 52.4)
- added TC2: Thermocouple, 0UCIRP-KiCAD-Lib:AM-K-PCB, F.Cu at (-102.2, 52.4)
- added TP1: ISO_5V, TestPoint:TestPoint_Plated_Hole_D2.0mm, F.Cu at (-18.8, 54.2)
- added TP10: BAT+, TestPoint:TestPoint_Plated_Hole_D2.0mm, F.Cu at (-44.9, 113.4)
- added TP11: BAT+, TestPoint:TestPoint_Plated_Hole_D2.0mm, F.Cu at (-18.8, 86.1)
- added TP12: BAT+, TestPoint:TestPoint_Plated_Hole_D2.0mm, F.Cu at (-44.9, 86.1)
- added TP13: BAT-, TestPoint:TestPoint_Plated_Hole_D2.0mm, F.Cu at (-18.8, 63.5)
- added TP14: BAT-, TestPoint:TestPoint_Plated_Hole_D2.0mm, F.Cu at (-44.9, 63.5)
- added TP15: BAT-, TestPoint:TestPoint_Plated_Hole_D2.0mm, F.Cu at (-18.8, 118.1)
- added TP16: BAT-, TestPoint:TestPoint_Plated_Hole_D2.0mm, F.Cu at (-44.9, 118.1)
- added TP17: BAT-, TestPoint:TestPoint_Plated_Hole_D2.0mm, F.Cu at (-18.8, 90.8)
- added TP18: BAT-, TestPoint:TestPoint_Plated_Hole_D2.0mm, F.Cu at (-44.9, 90.8)
- added TP19: Battery, TestPoint:TestPoint_Plated_Hole_D2.0mm, F.Cu at (9.95, 8.62)
- added TP2: ISO_5V, TestPoint:TestPoint_Plated_Hole_D2.0mm, F.Cu at (-44.9, 54.2)
- added TP20: Ground_Power, TestPoint:TestPoint_Plated_Hole_D2.0mm, F.Cu at (9.95, 13.3)
- added TP21: 3V3_REDS, TestPoint:TestPoint_Plated_Hole_D2.0mm, F.Cu at (-72.6, 20.1)
- added TP22: 5V0_REDS, TestPoint:TestPoint_Plated_Hole_D2.0mm, F.Cu at (-72.6, 24.7)
- added TP23: MAIN_OUT+, TestPoint:TestPoint_Plated_Hole_D2.0mm, F.Cu at (-72.6, 29.4)
- added TP24: GND, TestPoint:TestPoint_Plated_Hole_D2.0mm, F.Cu at (-72.6, 34.0)
- added TP3: ISO_5V, TestPoint:TestPoint_Plated_Hole_D2.0mm, F.Cu at (-18.8, 108.8)
- added TP4: ISO_5V, TestPoint:TestPoint_Plated_Hole_D2.0mm, F.Cu at (-44.9, 108.8)
- added TP5: ISO_5V, TestPoint:TestPoint_Plated_Hole_D2.0mm, F.Cu at (-18.8, 81.5)
- added TP6: ISO_5V, TestPoint:TestPoint_Plated_Hole_D2.0mm, F.Cu at (-44.9, 81.5)
- added TP7: BAT+, TestPoint:TestPoint_Plated_Hole_D2.0mm, F.Cu at (-18.8, 58.8)
- added TP8: BAT+, TestPoint:TestPoint_Plated_Hole_D2.0mm, F.Cu at (-44.9, 58.8)
- added TP9: BAT+, TestPoint:TestPoint_Plated_Hole_D2.0mm, F.Cu at (-18.8, 113.4)
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
Commit message: Component placement halfway done
Parts:
- removed REF**: UCIRP_Logo_3, 0UCIRP-KiCAD-Lib:UCIRP_Logo_3
- removed TP13, TP14, TP15, TP16, TP17, TP18: BAT-, TestPoint:TestPoint_Plated_Hole_D2.0mm
- added D43: LED, LED_SMD:LED_0603_1608Metric_Pad1.05x0.95mm_HandSolder, F.Cu at (33.2, 52.9)
- added D44: LED, LED_SMD:LED_0603_1608Metric_Pad1.05x0.95mm_HandSolder, F.Cu at (33.2, 63.9)
- added D45: LED, LED_SMD:LED_0603_1608Metric_Pad1.05x0.95mm_HandSolder, F.Cu at (33.2, 74.9)
- added D46: LED, LED_SMD:LED_0603_1608Metric_Pad1.05x0.95mm_HandSolder, F.Cu at (33.2, 85.9)
- added D47: LED, LED_SMD:LED_0603_1608Metric_Pad1.05x0.95mm_HandSolder, F.Cu at (33.2, 96.9)
- added D48: LED, LED_SMD:LED_0603_1608Metric_Pad1.05x0.95mm_HandSolder, F.Cu at (33.2, 107.9)
- added TP25: 5V, TestPoint:TestPoint_Plated_Hole_D2.0mm, F.Cu at (-117.5, 254.7)
- added TP26: 3.3V, TestPoint:TestPoint_Plated_Hole_D2.0mm, F.Cu at (-95.1, 122.5)
- C21, C22, C23, C24, C25, C26, C27, C28, C29, C30, C31, C32, C33, C34, C35, C36, C37, C38, C39, C40, C43, C48, C49, C50, C51, C52, C7, C8, C91, C92, C98, D11, D22, D23, D24, D25, D26, D27, D28, D29, D30, D31, D32, D33, D37, D38, D39, D41, D42, Q10, Q11, Q12, Q13, Q14, R100, R101, R102, R110, R111, R112, R113, R114, R115, R121, R122, R123, R131, R132, R133, R134, R6, R7, R72, R73, R74, R75, R76, R77, R78, R8, R80, R81, R82, R83, R86, R87, R88, R89, R90, R91, R92, R93, R94, R95, R96, R97, R98, R99, U11, U14, U17, U20, U23, U26, U28, U29, U31, U34, U35, U36, U37, U38, U40, U41, U42, U48, U5, U52: moved to B.Cu
- D1, D7: value 30V 2A -> 100V 8A; footprint 0UCIRP-KiCAD-Lib:NSR20F30NXT5G -> Diode_SMD:D_PowerDI-5
- D2, D4: value 30V 2A -> 150V 3A; footprint 0UCIRP-KiCAD-Lib:NSR20F30NXT5G -> Diode_SMD:D_SMF
- moved D28 307.3 mm to (171.0, 91.8)
- moved R88 303.6 mm to (169.5, 95.2), turned to 180 degrees
- moved J9 296.6 mm to (165.1, 105.0), turned to 90 degrees
- moved R89 293.1 mm to (167.1, 92.3)
- moved C48 292.7 mm to (160.7, 92.6), turned to -90 degrees
- moved D26 291.0 mm to (171.0, 69.2)
- moved D42 289.8 mm to (151.0, 56.8)
- moved D24 289.5 mm to (171.0, 46.8)
- moved R86 288.3 mm to (163.0, 95.5), turned to -90 degrees
- moved R87 287.0 mm to (161.5, 95.5), turned to -90 degrees
- moved R82 286.6 mm to (169.5, 72.8), turned to 180 degrees
- moved R77 285.7 mm to (169.6, 50.2), turned to 180 degrees
- moved R133 285.6 mm to (149.5, 60.2), turned to 180 degrees
- moved U34 285.5 mm to (163.4, 92.0), turned to 180 degrees
- moved D27 284.5 mm to (160.0, 105.0), turned to 90 degrees
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Connections:
- R33 pad 1: Net-(U11-~{PG}) -> Net-(D43-A)
- R40 pad 1: Net-(U14-~{PG}) -> Net-(D44-A)
- R47 pad 1: Net-(U17-~{PG}) -> Net-(D45-A)
- R54 pad 1: Net-(U20-~{PG}) -> Net-(D46-A)
- R61 pad 1: Net-(U23-~{PG}) -> Net-(D47-A)
- R68 pad 1: Net-(U26-~{PG}) -> Net-(D48-A)
- U11 pad 6: Net-(U11-~{PG}) -> Net-(D43-K)
- U14 pad 6: Net-(U14-~{PG}) -> Net-(D44-K)
- U17 pad 6: Net-(U17-~{PG}) -> Net-(D45-K)
- U20 pad 6: Net-(U20-~{PG}) -> Net-(D46-K)
- U23 pad 6: Net-(U23-~{PG}) -> Net-(D47-K)
- U26 pad 6: Net-(U26-~{PG}) -> Net-(D48-K)
Routing:
- net /REDs/Single-Cell-Charger2/ISO_5V: track 0.00 -> 125.6 mm, vias 0 -> 2
- net /REDs/Single-Cell-Charger4/ISO_5V: track 0.00 -> 125.6 mm, vias 0 -> 2
- net /REDs/Single-Cell-Charger3/ISO_5V: track 0.00 -> 125.6 mm, vias 0 -> 2
- net /REDs/Single-Cell-Charger5/ISO_5V: track 0.00 -> 125.6 mm, vias 0 -> 2
- net GND: track 0.00 -> 101.1 mm, vias 0 -> 54
- net /REDs/Single-Cell-Charger5/stat: track 0.00 -> 100.5 mm, vias 0 -> 4
- net /REDs/Single-Cell-Charger4/stat: track 0.00 -> 100.5 mm, vias 0 -> 4
- net /REDs/Single-Cell-Charger3/stat: track 0.00 -> 100.5 mm, vias 0 -> 4
- net /REDs/Single-Cell-Charger2/stat: track 0.00 -> 100.5 mm, vias 0 -> 4
- net /REDs/Single-Cell-Charger4/ISO_GND: track 0.00 -> 68.6 mm, vias 0 -> 2
- net /REDs/Single-Cell-Charger3/ISO_GND: track 0.00 -> 68.6 mm, vias 0 -> 2
- net /REDs/Single-Cell-Charger2/ISO_GND: track 0.00 -> 68.6 mm, vias 0 -> 2
- net /REDs/Single-Cell-Charger/ISO_5V: track 0.00 -> 62.8 mm, vias 0 -> 1
- net /REDs/Single-Cell-Charger1/ISO_5V: track 0.00 -> 62.8 mm, vias 0 -> 1
- net /REDs/Single-Cell-Charger1/stat: track 0.00 -> 50.3 mm, vias 0 -> 2
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Other:
- outline, holes or cut-outs redrawn

Commit message: Placed radios
Parts:
- removed H4: MountingHole_Pad, MountingHole:MountingHole_4.3mm_M4_Pad_Via
- R35, R36, R42, R43, R49, R50, R56, R57, R63, R64, R70, R71, U12, U15, U18, U21, U24, U27: moved to B.Cu
- moved C109 519.8 mm to (334.6, 176.3)
- moved C11 519.8 mm to (334.6, 167.8)
- moved C110 519.8 mm to (334.6, 180.6)
- moved C13 519.8 mm to (334.6, 172.1)
- moved R17 519.8 mm to (430.2, 208.6)
- moved R85 519.8 mm to (415.9, 199.4)
- moved C111 519.8 mm to (340.3, 182.6)
- moved D6 519.8 mm to (430.5, 203.7)
- moved L2 519.8 mm to (425.8, 210.0)
- moved TP26 519.8 mm to (417.6, 208.1)
- moved U7 301.8 mm to (366.2, 199.2)
- moved U50 282.7 mm to (-182.1, 172.7)
- moved U6 282.7 mm to (-182.2, 157.6)
- moved U45 197.1 mm to (159.6, 89.7)
- moved U44 177.3 mm to (159.6, 71.6)
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Routing:
- net /REDs/Single-Cell-Charger4/ISO_5V: track 125.6 -> 39.8 mm, vias 2 -> 1
- net /REDs/Single-Cell-Charger3/ISO_5V: track 125.6 -> 39.8 mm, vias 2 -> 1
- net /REDs/Single-Cell-Charger2/ISO_5V: track 125.6 -> 39.8 mm, vias 2 -> 1
- net /REDs/Single-Cell-Charger5/ISO_5V: track 125.6 -> 39.8 mm, vias 2 -> 1
- net /REDs/Single-Cell-Charger5/stat: track 100.5 -> 40.4 mm, vias 4 -> 1
- net /REDs/Single-Cell-Charger4/stat: track 100.5 -> 40.4 mm, vias 4 -> 1
- net /REDs/Single-Cell-Charger3/stat: track 100.5 -> 40.4 mm, vias 4 -> 1
- net /REDs/Single-Cell-Charger2/stat: track 100.5 -> 40.4 mm, vias 4 -> 1
- net /REDs/Single-Cell-Charger4/ISO_GND: track 68.6 -> 32.9 mm, vias 2 -> 1
- net /REDs/Single-Cell-Charger3/ISO_GND: track 68.6 -> 32.9 mm, vias 2 -> 1
- net /REDs/Single-Cell-Charger2/ISO_GND: track 68.6 -> 32.9 mm, vias 2 -> 1
- net GND: track 101.1 -> 76.9 mm, vias 54 -> 53
- net /REDs/Single-Cell-Charger/ISO_5V: track 62.8 -> 39.8 mm
- net /REDs/Single-Cell-Charger1/ISO_5V: track 62.8 -> 39.8 mm
- net /REDs/Single-Cell-Charger1/stat: track 50.3 -> 40.4 mm, vias 2 -> 1
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
Commit message: 3/4 DC-DC converters done
Parts:
- removed C7, C98: 100nF, Capacitor_SMD:C_0402_1005Metric
- removed C94: 10uF, Capacitor_SMD:C_0603_1608Metric
- removed D11, D39: 5.1V, Diode_SMD:D_MiniMELF
- removed J14, J23: PT, 0UCIRP-KiCAD-Lib:GX-12 3 pin
- removed J21: SMA, Connector_Coaxial:SMA_Molex_73251-2200_Horizontal
- removed R117: 100K, Resistor_SMD:R_0402_1005Metric
- removed R121, R6: 1K, Resistor_SMD:R_0402_1005Metric
- removed R122, R7: 5K, Resistor_SMD:R_0402_1005Metric
- removed R123, R8: 10K, Resistor_SMD:R_0402_1005Metric
- removed U44: ~, 0UCIRP-KiCAD-Lib:RFM95W
- removed U48, U5: ~, Package_TO_SOT_SMD:SOT-23-5
- added H4: MountingHole_Pad, MountingHole:MountingHole_4.3mm_M4_Pad_Via, F.Cu at (169.6, 120.2)
- C100, C6, C99, FB3, FB4, R124, U49: moved to B.Cu
- moved L2 383.9 mm to (70.5, 64.8), turned to 90 degrees
- moved TP26 382.9 mm to (71.0, 45.1)
- moved R17 380.5 mm to (78.5, 63.5)
- moved D6 376.8 mm to (80.3, 64.7), turned to -90 degrees
- moved R85 374.0 mm to (75.8, 44.0)
- moved U7 325.0 mm to (75.0, 55.0), turned to 90 degrees
- moved C111 297.6 mm to (75.7, 46.5)
- moved U6 297.5 mm to (115.0, 170.7)
- moved TP25 287.5 mm to (73.2, 39.5), turned to -90 degrees
- moved C116 286.9 mm to (70.1, 33.2), turned to 90 degrees
- moved C109 285.0 mm to (70.3, 69.7), turned to -90 degrees
- moved C110 284.7 mm to (74.9, 64.0)
- moved C115 281.4 mm to (52.6, 37.8), turned to -90 degrees
- moved C13 280.2 mm to (73.8, 69.7), turned to -90 degrees
- moved C11 275.5 mm to (77.2, 69.7), turned to -90 degrees
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Routing:
- net Net-(U7-Sense): track 0.00 -> 24.9 mm
- net Net-(U51-Sense): track 0.00 -> 23.4 mm
- net +24V: track 46.3 -> 65.7 mm
- net Net-(D2-K): track 0.00 -> 17.3 mm
- net Net-(U51-PGood): track 0.00 -> 15.4 mm
- net Net-(C115-Pad1): track 0.00 -> 14.1 mm
- net Net-(C110-Pad1): track 0.00 -> 9.35 mm
- net GND: track 76.9 -> 85.0 mm, vias 53 -> 58
- net Net-(U49-T-): track 0.00 -> 5.94 mm
- net Net-(U49-T+): track 0.00 -> 5.80 mm
- net Net-(U50-PGood): track 0.00 -> 5.76 mm
- net Net-(U5--): track 4.93 -> 0.00 mm
- net Net-(U48--): track 4.93 -> 0.00 mm
- net Net-(U7-PGood): track 0.00 -> 4.14 mm
- net +5V: track 20.2 -> 16.2 mm, vias 8 -> 6
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
Commit message: power connectors done
Parts:
- removed P3, P4: PAD_SMD, TestPoint:TestPoint_Plated_Hole_D4.0mm
- removed TP19: Battery, TestPoint:TestPoint_Plated_Hole_D2.0mm
- removed TP20: Ground_Power, TestPoint:TestPoint_Plated_Hole_D2.0mm
- removed U1: BMI088, 0UCIRP-KiCAD-Lib:BMI088
- removed U2: MS560702BA03-50, 0UCIRP-KiCAD-Lib:MS5607-02BA
- removed U3: BMM350, 0UCIRP-KiCAD-Lib:BMM350
- removed U39: ~, 0UCIRP-KiCAD-Lib:ZOE-M8Q
- added J14: Barrel_Jack_Switch, Connector_BarrelJack:BarrelJack_Horizontal, F.Cu at (64.2, 119.4)
- moved Q9 215.0 mm to (93.7, 111.6)
- moved D13 214.0 mm to (80.5, 123.6), turned to -90 degrees
- moved Q8 211.5 mm to (88.1, 111.6), turned to 180 degrees
- moved Q3 201.8 mm to (77.6, 125.8), turned to 90 degrees
- moved Q2 201.2 mm to (73.0, 125.8), turned to 90 degrees
- moved Q5 196.7 mm to (68.3, 114.9)
- moved Q4 194.3 mm to (63.2, 114.9), turned to 180 degrees
- moved D7 193.0 mm to (96.4, 106.6), turned to 180 degrees
- moved Q7 192.2 mm to (82.9, 111.6), turned to 90 degrees
- moved Q6 190.9 mm to (78.1, 111.8), turned to 90 degrees
- moved R27 187.7 mm to (80.5, 127.0), turned to 90 degrees
- moved R15 187.6 mm to (75.2, 122.1), turned to 90 degrees
- moved R12 186.2 mm to (71.5, 128.8)
- moved R11 185.2 mm to (70.2, 126.8), turned to -90 degrees
- moved R23 184.9 mm to (84.5, 108.1), turned to -90 degrees
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Routing:
- net /BATT: track 0.00 -> 23.4 mm
- net Net-(D1-A): track 0.00 -> 23.1 mm
- net Net-(Q8-G): track 0.00 -> 20.7 mm
- net Net-(Q4-G): track 0.00 -> 17.4 mm
- net Net-(D7-A): track 0.00 -> 16.5 mm
- net Net-(D3-K): track 0.00 -> 14.0 mm
- net Net-(C107-Pad1): track 0.00 -> 12.1 mm
- net GND: track 85.0 -> 95.2 mm, vias 58 -> 68
- net Net-(Q2-D): track 0.00 -> 9.49 mm
- net /GSE: track 0.00 -> 9.15 mm
- net Net-(Q6-D): track 0.00 -> 9.11 mm
- net Net-(Q6-G): track 0.00 -> 8.58 mm
- net Net-(Q2-G): track 0.00 -> 7.28 mm
- net REDs_MOSFET2: track 0.00 -> 5.50 mm
- net Net-(U6-Sense): track 0.00 -> 4.75 mm
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- added copper zone on F.Cu, net /BATT
- added copper zone on F.Cu, net /GSE
Other:
- board text added: "TP5"
- board text added: "TP6"
- board text added: "U25"

Commit message: ALMOST DONE WITH PLACEMENT
Parts:
- added U1: BMI088, 0UCIRP-KiCAD-Lib:BMI088, B.Cu at (118.2, 93.2)
- added U2: MS560702BA03-50, 0UCIRP-KiCAD-Lib:MS5607-02BA, B.Cu at (124.5, 67.8)
- added U3: BMM350, 0UCIRP-KiCAD-Lib:BMM350, B.Cu at (122.1, 87.4)
- added U39: ~, 0UCIRP-KiCAD-Lib:ZOE-M8Q, B.Cu at (167.8, 69.3)
- C1, C117, C14, C15, C16, C17, C18, C19, C2, C3, C4, C41, C42, C5, C53, C54, C55, C56, C57, C58, C59, C60, C61, C62, C63, C64, C65, C66, C67, C68, C70, C71, C74, C75, C77, C78, C79, C80, C83, C84, C86, C89, C9, C90, C93, C96, C97, FB1, FB2, J17, J5, R10, R105, R106, R107, R108, R119, R120, R127, R128, R129, R3, R4, R5, R79, U30, U46, U47, U53, U54, U8, Y1, Y2: moved to B.Cu
- moved C78 249.6 mm to (214.1, 92.7), turned to 180 degrees
- moved C79 249.6 mm to (214.1, 94.7), turned to 180 degrees
- moved C80 249.6 mm to (214.1, 96.6), turned to 180 degrees
- moved C81 236.1 mm to (204.7, 136.7)
- moved C82 236.1 mm to (204.7, 138.6)
- moved C87 236.1 mm to (195.5, 139.6)
- moved C88 236.1 mm to (207.6, 130.7)
- moved C20 234.2 mm to (171.3, 88.9)
- moved C85 232.1 mm to (189.9, 114.1)
- moved Q1 213.5 mm to (143.9, 70.0), turned to 90 degrees
- moved R2 208.7 mm to (143.6, 72.7), turned to 180 degrees
- moved R1 207.5 mm to (143.6, 73.9), turned to 180 degrees
- moved C93 206.1 mm to (165.0, 53.7), turned to -90 degrees
- moved C95 203.9 mm to (169.8, 72.1), turned to -90 degrees
- moved J1 202.6 mm to (132.8, 68.7)
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Routing:
- net GND: track 95.2 -> 198.7 mm, vias 68 -> 155
- net +3.3V: track 14.7 -> 97.3 mm, vias 0 -> 27
- net USB_VBUS: track 0.00 -> 39.1 mm, vias 0 -> 1
- net ALARM: track 0.00 -> 28.0 mm, vias 0 -> 1
- net ETH_TX: track 0.00 -> 19.2 mm
- net ETH_RX: track 0.00 -> 16.7 mm
- net +3V3_REDS: track 0.00 -> 15.6 mm, vias 0 -> 4
- net Net-(U30-T-): track 0.00 -> 6.85 mm
- net /BATT: track 23.4 -> 29.8 mm
- net Net-(J1-Pin_2): track 0.00 -> 6.17 mm
- net /GSE: track 9.15 -> 15.2 mm
- net Net-(U30-T+): track 0.00 -> 5.80 mm
- net Net-(U40F-VCAPDSI): track 0.00 -> 5.55 mm
- net Net-(J15-In): track 0.00 -> 5.22 mm
- net REDs_nRST: track 0.00 -> 4.52 mm
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