File: eve_gps.kicad_sch (KiCad schematic)
At the start: 9 parts, among them J14 BMI-S-101, J15 GNSS SMA

Commit message: new BOM
Parts:
- C53: Part # Generic 0603 4.7uF 6.3V X7R MLCC -> Generic CAP CER 4.7UF 6.3V X7R 0603
- C54, C55, C56, C57, C58: Part # Generic 100nF 6.3V X7R 0402 MLCC -> Generic CAP CER 0.1UF 6.3V X7R 0402
- J15: Part # 732512200 -> 0732512200
Changed lines of the file:
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@@
 			)
 		)
-		(property "Datasheet" " ~"
+		(property "Datasheet" "https://www.molex.com/en-us/products/part-detail/732512200?display=pdf"
 			(at 194.31 86.36 0)
 			(effects
@@
 			)
 		)
-		(property "Part #" "732512200"
+		(property "Part #" "0732512200"
 			(at 194.31 86.36 0)
 			(effects
@@
 			)
 		)
-		(property "Part #" "Generic 100nF 6.3V X7R 0402 MLCC"
+		(property "Part #" "Generic CAP CER 0.1UF 6.3V X7R 0402"
 			(at 147.32 60.96 0)
 			(effects
@@
 			)
 		)
-		(property "Part #" "Generic 0603 4.7uF 6.3V X7R MLCC"
+		(property "Part #" "Generic CAP CER 4.7UF 6.3V X7R 0603"
 			(at 90.17 60.96 0)
 			(effects
@@
 			)
 		)
-		(property "Part #" "Generic 100nF 6.3V X7R 0402 MLCC"
+		(property "Part #" "Generic CAP CER 0.1UF 6.3V X7R 0402"
 			(at 113.03 60.96 0)
 			(effects
@@
 			)
 		)
-		(property "Part #" "Generic 100nF 6.3V X7R 0402 MLCC"
+		(property "Part #" "Generic CAP CER 0.1UF 6.3V X7R 0402"
 			(at 101.6 60.96 0)
 			(effects
@@
 			)
 		)
-		(property "Part #" "Generic 100nF 6.3V X7R 0402 MLCC"
+		(property "Part #" "Generic CAP CER 0.1UF 6.3V X7R 0402"
 			(at 135.89 60.96 0)
 			(effects
@@
 			)
 		)
-		(property "Datasheet" "~"
+		(property "Datasheet" "https://www.laird.com/sites/default/files/bmi-s-101-sales.pdf"
 			(at 168.91 137.16 0)
 			(effects
@@
 			)
 		)
-		(property "Part #" "Generic 100nF 6.3V X7R 0402 MLCC"
+		(property "Part #" "Generic CAP CER 0.1UF 6.3V X7R 0402"
 			(at 124.46 60.96 0)
 			(effects
