File: eve_gps.kicad_sch (KiCad schematic)
At the start: 9 parts, among them J14 BMI-S-101, J15 GNSS SMA

Commit message: notes
Other:
- note added: "MURK SHIELD AND MOVE CIRCUIT COSER"
Changed lines of the file:
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@@
+		)
+	)
+	(text "MURK SHIELD AND  MOVE CIRCUIT COSER"
+		(exclude_from_sim no)
+		(at 185.674 117.602 0)
+		(effects
+			(font
+				(size 1.27 1.27)
+				(color 255 0 21 1)
+			)
 		)
 	)
