File: solenoid.kicad_sch (KiCad schematic)
At the start: 10 parts, among them J6 Solenoid, Q10 DMG3402L

Commit message: Lots of cleanup and updates; Waiting on PR approval for GPS filter
Parts:
- renumbered C39 to C47, D20 to D22, D21 to D23, J6 to J11, U23 to U26

Commit message: 8.02 Update; Also changed VRMs and added some notes
Parts:
- renumbered C47 to C40, D22 to D17, D23 to D18, J11 to J7, R55 to R71, R56 to R72, R57 to R73, R58 to R74, U26 to U30

Commit message: ECU essentially reviewable
Parts:
- renumbered D17 to D24, D18 to D25, R71 to R75, R72 to R76, R73 to R77, R74 to R78, U30 to U29

Commit message: addressed PR comments
Parts:
- renumbered D24 to D23, D25 to D24

Commit message: Updated schematic with IOC
Parts:
- J7: footprint TerminalBlock:TerminalBlock_bornier-3_P5.08mm -> Connector_PinHeader_2.54mm:PinHeader_1x03_P2.54mm_Vertical
- R77: value 1R -> 0.1R; Part # Generic 1R 2W 1% 2512 Resistor -> Generic 0.1R 2W 1% 2512 Resistor
Changed lines of the file:
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@@
 			)
 		)
-		(property "Value" "1R"
+		(property "Value" "0.1R"
 			(at 142.24 107.95 0)
 			(effects
@@
 			)
 		)
-		(property "Part #" "Generic 1R 2W 1% 2512 Resistor"
+		(property "Part #" "Generic 0.1R 2W 1% 2512 Resistor"
 			(at 139.7 106.68 0)
 			(effects
@@
 			)
 		)
-		(property "Footprint" "TerminalBlock:TerminalBlock_bornier-3_P5.08mm"
+		(property "Footprint" "Connector_PinHeader_2.54mm:PinHeader_1x03_P2.54mm_Vertical"
 			(at 121.92 81.28 0)
 			(effects

Commit message: new BOM
Parts:
- C40: Part # Generic 100nF 6.3V X7R 0402 MLCC -> Generic CAP CER 0.1UF 6.3V X7R 0402
- D23: value SDT8A100P5-7 -> 100V 8A; Manufacturer Diodes -> Diodes Incorporated
- D24: value MMSZ4684T1G -> 3.3V
- Q10: Manufacturer Diodes -> Diodes Incorporated
- R75: Part # Generic 10K 1% 0402 Resistor -> Generic RES SMD 10K OHM 1% 1/4W 0402
- R76: value 100R -> 100; Part # Generic 100R 1% 0402 Resistor -> Generic RES SMD 100 OHM 1% 1/4W 0402
- R77: value 0.1R -> 0.1; Part # Generic 0.1R 2W 1% 2512 Resistor -> Generic RES SMD 0.1 OHM 0.1% 2W 2512
- R78: Part # Generic 1K 1% 0402 Resistor -> Generic RES SMD 1K OHM 1% 1/16W 0402
Changed lines of the file:
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@@
 			)
 		)
-		(property "Value" "0.1R"
+		(property "Value" "0.1"
 			(at 142.24 107.95 0)
 			(effects
@@
 			)
 		)
-		(property "Part #" "Generic 0.1R 2W 1% 2512 Resistor"
+		(property "Part #" "Generic RES SMD 0.1 OHM 0.1% 2W 2512"
 			(at 139.7 106.68 0)
 			(effects
@@
 			)
 		)
-		(property "Manufacturer" "Diodes"
+		(property "Manufacturer" "Diodes Incorporated"
 			(at 137.16 93.98 0)
 			(effects
@@
 			)
 		)
-		(property "Value" "MMSZ4684T1G"
+		(property "Value" "3.3V"
 			(at 168.91 107.95 90)
 			(effects
@@
 			)
 		)
-		(property "Datasheet" "~"
+		(property "Datasheet" "https://www.onsemi.com/pdf/datasheet/mmsz4678t1-d.pdf"
 			(at 166.37 106.68 90)
 			(effects
@@
 			)
 		)
-		(property "Part #" "Generic 100nF 6.3V X7R 0402 MLCC"
+		(property "Part #" "Generic CAP CER 0.1UF 6.3V X7R 0402"
 			(at 181.61 90.17 0)
 			(effects
@@
 			)
 		)
-		(property "Manufacturer" "~"
+		(property "Manufacturer" ""
 			(at 121.92 81.28 0)
 			(effects
@@
 			)
 		)
-		(property "Part #" "~"
+		(property "Part #" ""
 			(at 121.92 81.28 0)
 			(effects
@@
 			)
 		)
-		(property "Part #" "Generic 10K 1% 0402 Resistor"
+		(property "Part #" "Generic RES SMD 10K OHM 1% 1/4W 0402"
 			(at 124.46 99.06 0)
 			(effects
@@
 			)
 		)
-		(property "Value" "SDT8A100P5-7"
+		(property "Value" "100V 8A"
 			(at 151.13 78.74 0)
 			(effects
@@
 			)
 		)
-		(property "Manufacturer" "Diodes"
+		(property "Manufacturer" "Diodes Incorporated"
 			(at 151.13 81.28 0)
 			(effects
@@
 			)
 		)
-		(property "Part #" "Generic 1K 1% 0402 Resistor"
+		(property "Part #" "Generic RES SMD 1K OHM 1% 1/16W 0402"
 			(at 161.29 101.6 0)
 			(effects
@@
 			)
 		)
-		(property "Value" "100R"
+		(property "Value" "100"
 			(at 129.54 91.44 90)
 			(effects
@@
 			)
 		)
-		(property "Part #" "Generic 100R 1% 0402 Resistor"
+		(property "Part #" "Generic RES SMD 100 OHM 1% 1/4W 0402"
 			(at 129.54 93.98 0)
 			(effects
