File: solenoid.kicad_sch (KiCad schematic)
At the start: 10 parts, among them J7 Solenoid, Q10 DMG3402L

Commit message: notes
Other:
- note added: "find part"
Changed lines of the file:
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@@
+		)
+	)
+	(text "find part"
+		(exclude_from_sim no)
+		(at 147.32 110.998 0)
+		(effects
+			(font
+				(size 1.27 1.27)
+				(color 255 32 32 1)
+			)
 		)
 	)
@@
 			)
 		)
-		(property "Description" ""
+		(property "Description" "FIND SPEWfUAF"
 			(at 139.7 106.68 0)
 			(effects
