File: tc.kicad_sch (KiCad schematic)
At the start: 6 parts

Commit message: Lots of cleanup and updates; Waiting on PR approval for GPS filter
Parts:
- renumbered C40 to C48, C41 to C49, U24 to U27
Changed lines of the file:
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@@
   (symbol (lib_id "UCIRP-KiCAD-Lib:MAX31855") (at 152.4 101.6 0) (mirror x) (unit 1)
     (in_bom yes) (on_board yes) (dnp no)
-    (property "Reference" "U24" (at 152.4 88.9 0)
+    (property "Reference" "U27" (at 152.4 88.9 0)
       (effects (font (size 1.27 1.27)))
     )
@@
       (project "rocket2-ecu"
         (path "/02606b2c-b376-4ffb-9781-f9cea3f70994/224b2102-9471-4db4-a51e-6702830844ba"
+          (reference "U27") (unit 1)
+        )
+      )
+      (project "rocket2-gse"
+        (path "/94c3ca0c-6aa1-4bff-ab47-a0279d059895/c7d5fc99-8b63-4a42-996c-97b63a613c71"
+          (reference "U21") (unit 1)
+        )
+        (path "/94c3ca0c-6aa1-4bff-ab47-a0279d059895/339cdff9-22b3-471e-94e8-a08c3a88ebe1"
+          (reference "U22") (unit 1)
+        )
+        (path "/94c3ca0c-6aa1-4bff-ab47-a0279d059895/e37acb46-d41c-43ff-890c-4e9139fb294b"
+          (reference "U19") (unit 1)
+        )
+        (path "/94c3ca0c-6aa1-4bff-ab47-a0279d059895/d496d162-84e0-4206-8055-60227dc94527"
           (reference "U24") (unit 1)
         )
-      )
-      (project "rocket2-gse"
-        (path "/94c3ca0c-6aa1-4bff-ab47-a0279d059895/c7d5fc99-8b63-4a42-996c-97b63a613c71"
-          (reference "U21") (unit 1)
-        )
-        (path "/94c3ca0c-6aa1-4bff-ab47-a0279d059895/339cdff9-22b3-471e-94e8-a08c3a88ebe1"
-          (reference "U22") (unit 1)
-        )
-        (path "/94c3ca0c-6aa1-4bff-ab47-a0279d059895/e37acb46-d41c-43ff-890c-4e9139fb294b"
-          (reference "U19") (unit 1)
-        )
-        (path "/94c3ca0c-6aa1-4bff-ab47-a0279d059895/d496d162-84e0-4206-8055-60227dc94527"
-          (reference "U24") (unit 1)
-        )
         (path "/94c3ca0c-6aa1-4bff-ab47-a0279d059895/64b31f2e-4849-43cf-bb2a-fe1c71693eda"
           (reference "U20") (unit 1)
@@
   (symbol (lib_id "power:+3.3V") (at 152.4 74.93 0) (unit 1)
     (in_bom yes) (on_board yes) (dnp no)
-    (property "Reference" "#PWR0106" (at 152.4 78.74 0)
+    (property "Reference" "#PWR0135" (at 152.4 78.74 0)
       (effects (font (size 1.27 1.27)) hide)
     )
@@
       (project "rocket2-ecu"
         (path "/02606b2c-b376-4ffb-9781-f9cea3f70994/224b2102-9471-4db4-a51e-6702830844ba"
-          (reference "#PWR0106") (unit 1)
+          (reference "#PWR0135") (unit 1)
         )
       )
@@
   (symbol (lib_id "power:GND") (at 142.24 105.41 270) (unit 1)
     (in_bom yes) (on_board yes) (dnp no) (fields_autoplaced)
-    (property "Reference" "#PWR0105" (at 135.89 105.41 0)
+    (property "Reference" "#PWR0134" (at 135.89 105.41 0)
       (effects (font (size 1.27 1.27)) hide)
     )
@@
       (project "rocket2-ecu"
         (path "/02606b2c-b376-4ffb-9781-f9cea3f70994/224b2102-9471-4db4-a51e-6702830844ba"
-          (reference "#PWR0105") (unit 1)
+          (reference "#PWR0134") (unit 1)
         )
       )
@@
   (symbol (lib_id "Device:C_Small") (at 152.4 77.47 0) (unit 1)
     (in_bom yes) (on_board yes) (dnp no)
-    (property "Reference" "C41" (at 154.94 76.2 0)
+    (property "Reference" "C49" (at 154.94 76.2 0)
       (effects (font (size 1.27 1.27)) (justify left))
     )
@@
       (project "rocket2-ecu"
         (path "/02606b2c-b376-4ffb-9781-f9cea3f70994/224b2102-9471-4db4-a51e-6702830844ba"
-          (reference "C41") (unit 1)
+          (reference "C49") (unit 1)
         )
       )
@@
   (symbol (lib_id "power:+3.3V") (at 142.24 97.79 90) (unit 1)
     (in_bom yes) (on_board yes) (dnp no) (fields_autoplaced)
-    (property "Reference" "#PWR0104" (at 146.05 97.79 0)
+    (property "Reference" "#PWR0133" (at 146.05 97.79 0)
       (effects (font (size 1.27 1.27)) hide)
     )
@@
       (project "rocket2-ecu"
         (path "/02606b2c-b376-4ffb-9781-f9cea3f70994/224b2102-9471-4db4-a51e-6702830844ba"
-          (reference "#PWR0104") (unit 1)
+          (reference "#PWR0133") (unit 1)
         )
       )
@@
   (symbol (lib_id "Device:C_Small") (at 120.65 101.6 0) (unit 1)
     (in_bom yes) (on_board yes) (dnp no)
-    (property "Reference" "C40" (at 123.19 100.33 0)
+    (property "Reference" "C48" (at 123.19 100.33 0)
       (effects (font (size 1.27 1.27)) (justify left))
     )
@@
       (project "rocket2-ecu"
         (path "/02606b2c-b376-4ffb-9781-f9cea3f70994/224b2102-9471-4db4-a51e-6702830844ba"
-          (reference "C40") (unit 1)
+          (reference "C48") (unit 1)
         )
       )
@@
   (symbol (lib_id "power:GND") (at 152.4 80.01 0) (unit 1)
     (in_bom yes) (on_board yes) (dnp no)
-    (property "Reference" "#PWR0107" (at 152.4 86.36 0)
+    (property "Reference" "#PWR0136" (at 152.4 86.36 0)
       (effects (font (size 1.27 1.27)) hide)
     )
@@
       (project "rocket2-ecu"
         (path "/02606b2c-b376-4ffb-9781-f9cea3f70994/224b2102-9471-4db4-a51e-6702830844ba"
-          (reference "#PWR0107") (unit 1)
-        )
-      )
+          (reference "#PWR0136") (unit 1)
+        )
+      )

Commit message: 8.02 Update; Also changed VRMs and added some notes
Parts:
- renumbered C48 to C41, C49 to C42, U27 to U31
Changed lines of the file:
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@@
 		(on_board yes)
 		(dnp no)
-		(property "Reference" "U27"
+		(property "Reference" "U31"
 			(at 152.4 88.9 0)
 			(effects
@@
 			(project "rocket2-ecu"
 				(path "/02606b2c-b376-4ffb-9781-f9cea3f70994/224b2102-9471-4db4-a51e-6702830844ba"
-					(reference "U27")
+					(reference "U31")
 					(unit 1)
 				)
@@
 		(on_board yes)
 		(dnp no)
-		(property "Reference" "#PWR0135"
+		(property "Reference" "#PWR0121"
 			(at 152.4 78.74 0)
 			(effects
@@
 			(project "rocket2-ecu"
 				(path "/02606b2c-b376-4ffb-9781-f9cea3f70994/224b2102-9471-4db4-a51e-6702830844ba"
-					(reference "#PWR0135")
+					(reference "#PWR0121")
 					(unit 1)
 				)
@@
 		(dnp no)
 		(fields_autoplaced yes)
-		(property "Reference" "#PWR0134"
+		(property "Reference" "#PWR0120"
 			(at 135.89 105.41 0)
 			(effects
@@
 			(project "rocket2-ecu"
 				(path "/02606b2c-b376-4ffb-9781-f9cea3f70994/224b2102-9471-4db4-a51e-6702830844ba"
-					(reference "#PWR0134")
+					(reference "#PWR0120")
 					(unit 1)
 				)
@@
 		(on_board yes)
 		(dnp no)
-		(property "Reference" "C49"
+		(property "Reference" "C42"
 			(at 154.94 76.2 0)
 			(effects
@@
 			(project "rocket2-ecu"
 				(path "/02606b2c-b376-4ffb-9781-f9cea3f70994/224b2102-9471-4db4-a51e-6702830844ba"
-					(reference "C49")
+					(reference "C42")
 					(unit 1)
 				)
@@
 		(dnp no)
 		(fields_autoplaced yes)
-		(property "Reference" "#PWR0133"
+		(property "Reference" "#PWR0119"
 			(at 146.05 97.79 0)
 			(effects
@@
 			(project "rocket2-ecu"
 				(path "/02606b2c-b376-4ffb-9781-f9cea3f70994/224b2102-9471-4db4-a51e-6702830844ba"
-					(reference "#PWR0133")
+					(reference "#PWR0119")
 					(unit 1)
 				)
@@
 		(on_board yes)
 		(dnp no)
-		(property "Reference" "C48"
+		(property "Reference" "C41"
 			(at 123.19 100.33 0)
 			(effects
@@
 			(project "rocket2-ecu"
 				(path "/02606b2c-b376-4ffb-9781-f9cea3f70994/224b2102-9471-4db4-a51e-6702830844ba"
-					(reference "C48")
+					(reference "C41")
 					(unit 1)
 				)
@@
 		(on_board yes)
 		(dnp no)
-		(property "Reference" "#PWR0136"
+		(property "Reference" "#PWR0122"
 			(at 152.4 86.36 0)
 			(effects
@@
 			(project "rocket2-ecu"
 				(path "/02606b2c-b376-4ffb-9781-f9cea3f70994/224b2102-9471-4db4-a51e-6702830844ba"
-					(reference "#PWR0136")
-					(unit 1)
-				)
+					(reference "#PWR0122")
+					(unit 1)
+				)

Commit message: ECU essentially reviewable
Parts:
- added R79: 100k, kicad-egglib:0402_1005M, symbol Device:R_Small_US
- renumbered U31 to U30
Connections:
- net +3.3V: now also R79.1
- net ~{CS}: now also R79.2
Changed lines of the file:
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@@
 		(color 0 0 0 0)
 	)
+	(junction
+		(at 172.72 100.33)
+		(diameter 0)
+		(color 0 0 0 0)
+	)
 	(wire
 		(pts
@@
 	(wire
 		(pts
+			(xy 172.72 100.33) (xy 162.56 100.33)
+		)
+		(stroke
+			(width 0)
+			(type default)
+		)
+	)
+	(wire
+		(pts
 			(xy 100.33 104.14) (xy 102.87 104.14)
 		)
@@
 	(wire
 		(pts
+			(xy 172.72 97.79) (xy 172.72 100.33)
+		)
+		(stroke
+			(width 0)
+			(type default)
+		)
+	)
+	(wire
+		(pts
 			(xy 142.24 100.33) (xy 130.81 100.33)
 		)
@@
 		(pts
 			(xy 130.81 96.52) (xy 120.65 96.52)
+		)
+		(stroke
+			(width 0)
+			(type default)
+		)
+	)
+	(wire
+		(pts
+			(xy 176.53 100.33) (xy 172.72 100.33)
 		)
 		(stroke
@@
 	(hierarchical_label "~{CS}"
 		(shape input)
-		(at 162.56 100.33 0)
+		(at 176.53 100.33 0)
 		(fields_autoplaced yes)
 		(effects
@@
 		(on_board yes)
 		(dnp no)
-		(property "Reference" "U31"
+		(property "Reference" "U30"
 			(at 152.4 88.9 0)
 			(effects
@@
 			(project "rocket2-ecu"
 				(path "/02606b2c-b376-4ffb-9781-f9cea3f70994/224b2102-9471-4db4-a51e-6702830844ba"
-					(reference "U31")
+					(reference "U30")
 					(unit 1)
 				)
@@
 		(on_board yes)
 		(dnp no)
-		(property "Reference" "#PWR0121"
+		(property "Reference" "#PWR0118"
 			(at 152.4 78.74 0)
 			(effects
@@
 			(project "rocket2-ecu"
 				(path "/02606b2c-b376-4ffb-9781-f9cea3f70994/224b2102-9471-4db4-a51e-6702830844ba"
-					(reference "#PWR0121")
+					(reference "#PWR0118")
 					(unit 1)
 				)
@@
 				(path "/94c3ca0c-6aa1-4bff-ab47-a0279d059895/3a0ce878-a305-4d14-89b9-2463ba92207c"
 					(reference "#PWR0163")
+					(unit 1)
+				)
+			)
+		)
+	)
+	(symbol
+		(lib_id "power:+3.3V")
+		(at 172.72 92.71 0)
+		(unit 1)
+		(exclude_from_sim no)
+		(in_bom yes)
+		(on_board yes)
+		(dnp no)
+		(property "Reference" "#PWR0120"
+			(at 172.72 96.52 0)
+			(effects
+				(font
+					(size 1.27 1.27)
+				)
+				(hide yes)
+			)
+		)
+		(property "Value" "+3.3V"
+			(at 172.72 87.63 0)
+			(effects
+				(font
+					(size 1.27 1.27)
+				)
+			)
+		)
+		(property "Footprint" ""
+			(at 172.72 92.71 0)
+			(effects
+				(font
+					(size 1.27 1.27)
+				)
+				(hide yes)
+			)
+		)
+		(property "Datasheet" ""
+			(at 172.72 92.71 0)
+			(effects
+				(font
+					(size 1.27 1.27)
+				)
+				(hide yes)
+			)
+		)
+		(property "Description" "Power symbol creates a global label with name \"+3.3V\""
+			(at 172.72 92.71 0)
+			(effects
+				(font
+					(size 1.27 1.27)
+				)
+				(hide yes)
+			)
+		)
+		(pin "1"
+		)
+		(instances
+			(project "rocket2-ecu"
+				(path "/02606b2c-b376-4ffb-9781-f9cea3f70994/224b2102-9471-4db4-a51e-6702830844ba"
+					(reference "#PWR0120")
 					(unit 1)
 				)
@@
 		(dnp no)
 		(fields_autoplaced yes)
-		(property "Reference" "#PWR0120"
+		(property "Reference" "#PWR0117"
 			(at 135.89 105.41 0)
 			(effects
@@
 			(project "rocket2-ecu"
 				(path "/02606b2c-b376-4ffb-9781-f9cea3f70994/224b2102-9471-4db4-a51e-6702830844ba"
-					(reference "#PWR0120")
+					(reference "#PWR0117")
 					(unit 1)
 				)
@@
 		(dnp no)
 		(fields_autoplaced yes)
-		(property "Reference" "#PWR0119"
+		(property "Reference" "#PWR0116"
 			(at 146.05 97.79 0)
 			(effects
@@
 			(project "rocket2-ecu"
 				(path "/02606b2c-b376-4ffb-9781-f9cea3f70994/224b2102-9471-4db4-a51e-6702830844ba"
-					(reference "#PWR0119")
+					(reference "#PWR0116")
 					(unit 1)
 				)
@@
 				(path "/94c3ca0c-6aa1-4bff-ab47-a0279d059895/9b4ffa27-b22d-4c40-bf79-fb37f5b9ee9d"
 					(reference "#PWR0223")
+					(unit 1)
+				)
+			)
+		)
+	)
+	(symbol
+		(lib_id "Device:R_Small_US")
+		(at 172.72 95.25 0)
+		(unit 1)
+		(exclude_from_sim no)
+		(in_bom yes)
+		(on_board yes)
+		(dnp no)
+		(property "Reference" "R79"
+			(at 175.26 93.98 0)
+			(effects
+				(font
+					(size 1.27 1.27)
+				)
+				(justify left)
+			)
+		)
+		(property "Value" "100k"
+			(at 175.26 96.52 0)
+			(effects
+				(font
+					(size 1.27 1.27)
+				)
+				(justify left)
+			)
+		)
+		(property "Footprint" "kicad-egglib:0402_1005M"
+			(at 172.72 95.25 0)
+			(effects
+				(font
+					(size 1.27 1.27)
+				)
+				(hide yes)
+			)
+		)
+		(property "Datasheet" "~"
+			(at 172.72 95.25 0)
+			(effects
+				(font
+					(size 1.27 1.27)
+				)
+				(hide yes)
+			)
+		)
+		(property "Description" ""
+			(at 172.72 95.25 0)
+			(effects
+				(font
+					(size 1.27 1.27)
+				)
+				(hide yes)
+			)
+		)
+		(property "Manufacturer" "Generic"
+			(at 172.72 95.25 0)
+			(effects
+				(font
+					(size 1.27 1.27)
+				)
+				(hide yes)
+			)
+		)
+		(property "Part #" "Generic 100k 1% 0402 Chip Resistor"
+			(at 172.72 95.25 0)
+			(effects
+				(font
+					(size 1.27 1.27)
+				)
+				(hide yes)
+			)
+		)
+		(pin "2"
+		)
+		(pin "1"
+		)
+		(instances
+			(project "rocket2-ecu"
+				(path "/02606b2c-b376-4ffb-9781-f9cea3f70994/224b2102-9471-4db4-a51e-6702830844ba"
+					(reference "R79")
 					(unit 1)
 				)
@@
 		(on_board yes)
 		(dnp no)
-		(property "Reference" "#PWR0122"
+		(property "Reference" "#PWR0119"
 			(at 152.4 86.36 0)
 			(effects
@@
 			(project "rocket2-ecu"
 				(path "/02606b2c-b376-4ffb-9781-f9cea3f70994/224b2102-9471-4db4-a51e-6702830844ba"
-					(reference "#PWR0122")
-					(unit 1)
-				)
+					(reference "#PWR0119")
+					(unit 1)
+				)

Commit message: Assigned almost all footprints
Parts:
- R79: value 100k -> 100K; footprint kicad-egglib:0402_1005M -> Resistor_SMD:R_0402_1005Metric; Part # Generic 100k 1% 0402 Chip Resistor -> Generic 100K 5% 0402 Resistor
- TC1: footprint UCIRP-KiCAD-Lib:AM-K-PCB -> 0UCIRP-KiCAD-Lib:AM-K-PCB
Changed lines of the file:
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@@
 				)
 				(path "/02606b2c-b376-4ffb-9781-f9cea3f70994/d5dcb60d-501b-41cc-98ca-6e0288432cc2"
-					(reference "U50")
+					(reference "U49")
 					(unit 1)
 				)
@@
 				)
 				(path "/02606b2c-b376-4ffb-9781-f9cea3f70994/d5dcb60d-501b-41cc-98ca-6e0288432cc2"
-					(reference "#PWR0336")
+					(reference "#PWR0330")
 					(unit 1)
 				)
@@
 				)
 				(path "/02606b2c-b376-4ffb-9781-f9cea3f70994/d5dcb60d-501b-41cc-98ca-6e0288432cc2"
-					(reference "#PWR0338")
+					(reference "#PWR0332")
 					(unit 1)
 				)
@@
 				)
 				(path "/02606b2c-b376-4ffb-9781-f9cea3f70994/d5dcb60d-501b-41cc-98ca-6e0288432cc2"
-					(reference "#PWR0335")
+					(reference "#PWR0329")
 					(unit 1)
 				)
@@
 			)
 		)
-		(property "Footprint" "UCIRP-KiCAD-Lib:AM-K-PCB"
+		(property "Footprint" "0UCIRP-KiCAD-Lib:AM-K-PCB"
 			(at 83.185 100.33 0)
 			(effects
@@
 				)
 				(path "/02606b2c-b376-4ffb-9781-f9cea3f70994/d5dcb60d-501b-41cc-98ca-6e0288432cc2"
-					(reference "C101")
+					(reference "C100")
 					(unit 1)
 				)
@@
 				)
 				(path "/02606b2c-b376-4ffb-9781-f9cea3f70994/d5dcb60d-501b-41cc-98ca-6e0288432cc2"
-					(reference "#PWR0334")
+					(reference "#PWR0328")
 					(unit 1)
 				)
@@
 			)
 		)
-		(property "Value" "100k"
+		(property "Value" "100K"
 			(at 175.26 96.52 0)
 			(effects
@@
 			)
 		)
-		(property "Footprint" "kicad-egglib:0402_1005M"
+		(property "Footprint" "Resistor_SMD:R_0402_1005Metric"
 			(at 172.72 95.25 0)
 			(effects
@@
 			)
 		)
-		(property "Part #" "Generic 100k 1% 0402 Chip Resistor"
+		(property "Part #" "Generic 100K 5% 0402 Resistor"
 			(at 172.72 95.25 0)
 			(effects
@@
 				)
 				(path "/02606b2c-b376-4ffb-9781-f9cea3f70994/d5dcb60d-501b-41cc-98ca-6e0288432cc2"
-					(reference "R125")
+					(reference "R124")
 					(unit 1)
 				)
@@
 				)
 				(path "/02606b2c-b376-4ffb-9781-f9cea3f70994/d5dcb60d-501b-41cc-98ca-6e0288432cc2"
-					(reference "C100")
+					(reference "C99")
 					(unit 1)
 				)
@@
 				)
 				(path "/02606b2c-b376-4ffb-9781-f9cea3f70994/d5dcb60d-501b-41cc-98ca-6e0288432cc2"
-					(reference "#PWR0337")
-					(unit 1)
-				)
+					(reference "#PWR0331")
+					(unit 1)
+				)

Commit message: new BOM
Parts:
- C41: Part # Generic 10nF 6.3V X7R 0402 MLCC -> Generic CAP CER 10NF 6.3V X7R 0402
- C42: Part # Generic 100nF 6.3V X7R 0402 MLCC -> Generic CAP CER 0.1UF 6.3V X7R 0402
- FB1, FB2: value BLM18PG471SH1D -> 470ohm @100MHz
- R79: Part # Generic 100K 5% 0402 Resistor -> Generic RES SMD 100K OHM 1% 1/16W 0402
- U30: Part # MAX31855 -> MAX31855JASA+
Changed lines of the file:
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@@
 			)
 		)
-		(property "Value" "BLM18PG471SH1D"
+		(property "Value" "470ohm @100MHz"
 			(at 110.49 92.71 90)
 			(effects
@@
 			)
 		)
-		(property "Value" "BLM18PG471SH1D"
+		(property "Value" "470ohm @100MHz"
 			(at 110.49 110.49 90)
 			(effects
@@
 			)
 		)
-		(property "Part #" "MAX31855"
+		(property "Part #" "MAX31855JASA+"
 			(at 152.4 93.98 0)
 			(effects
@@
 			)
 		)
-		(property "Datasheet" "~"
+		(property "Datasheet" "https://www.farnell.com/datasheets/4071246.pdf"
 			(at 83.185 100.33 0)
 			(effects
@@
 			)
 		)
-		(property "Part #" "Generic 100nF 6.3V X7R 0402 MLCC"
+		(property "Part #" "Generic CAP CER 0.1UF 6.3V X7R 0402"
 			(at 152.4 77.47 0)
 			(effects
@@
 			)
 		)
-		(property "Part #" "Generic 100K 5% 0402 Resistor"
+		(property "Part #" "Generic RES SMD 100K OHM 1% 1/16W 0402"
 			(at 172.72 95.25 0)
 			(effects
@@
 			)
 		)
-		(property "Part #" "Generic 10nF 6.3V X7R 0402 MLCC"
+		(property "Part #" "Generic CAP CER 10NF 6.3V X7R 0402"
 			(at 120.65 101.6 0)
 			(effects
