File: rocket2-battery.kicad_sch (KiCad schematic)
At the start: 78 parts, among them J2 Conn_01x07, J4 SMA, J5 ARM Cortex Debug, P5 PAD_SMD, P6 PAD_SMD, Q2 Q_NMOS_GSD, Q3 Q_NMOS_GSD, Q4 PMOS, Q5 PMOS, Q6 Q_NMOS_GSD, Q7 Q_NMOS_GSD, Q8 PMOS, Q9 PMOS, U5 ADS7828, U50 24V->3.3V 3A, U6 24V->5V 3A, Y1 16MHz

Commit message: Finished layout
Connections:
- net REDs_RADIO_DIO2: no longer names the net of U8.19 (PB1)
- no-connect marks 45 -> 46
Changed lines of the file:
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@@
 	)
 	(no_connect
+		(at 205.74 44.45)
+	)
+	(no_connect
 		(at 58.42 241.3)
 	)
@@
 			(effects
 				(font
-					(size 1.27 1.27)
-				)
-				(justify left)
-				(hide yes)
-			)
-		)
-	)
-	(global_label "REDs_RADIO_DIO2"
-		(shape input)
-		(at 205.74 44.45 0)
-		(fields_autoplaced yes)
-		(effects
-			(font
-				(size 1.27 1.27)
-			)
-			(justify left)
-		)
-		(property "Intersheetrefs" "${INTERSHEET_REFS}"
-			(at 225.2768 44.45 0)
-			(effects
-				(font

Commit message: notes
Other:
- note added: "MURK MOUNTING HOLE AND MOVE antenanan"
Changed lines of the file:
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@@
+		)
+	)
+	(text "MURK MOUNTING HOLE AND MOVE antenanan "
+		(exclude_from_sim no)
+		(at 282.702 50.8 0)
+		(effects
+			(font
+				(size 1.27 1.27)
+				(color 255 22 24 1)
+			)
 		)
 	)
