File: ECU_Memory.kicad_sch (KiCad schematic)
At the start: 6 parts

Commit message: addressed PR comments
Parts:
- renumbered C94 to C97, C95 to C98, R115 to R120, R116 to R121, U44 to U47, U45 to U48
Changed lines of the file:
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@@
 		(on_board yes)
 		(dnp no)
-		(property "Reference" "U44"
+		(property "Reference" "U47"
 			(at 120.65 103.505 0)
 			(effects
@@
 			(project "rocket2-ecu"
 				(path "/02606b2c-b376-4ffb-9781-f9cea3f70994/fc637a4d-3fde-405d-ae60-ec7da7a8a72d"
-					(reference "U44")
+					(reference "U47")
 					(unit 1)
 				)
@@
 		(on_board yes)
 		(dnp no)
-		(property "Reference" "#PWR0300"
+		(property "Reference" "#PWR0321"
 			(at 187.96 87.63 0)
 			(effects
@@
 			(project "rocket2-ecu"
 				(path "/02606b2c-b376-4ffb-9781-f9cea3f70994/fc637a4d-3fde-405d-ae60-ec7da7a8a72d"
-					(reference "#PWR0300")
+					(reference "#PWR0321")
 					(unit 1)
 				)
@@
 		(on_board yes)
 		(dnp no)
-		(property "Reference" "#PWR0295"
+		(property "Reference" "#PWR0316"
 			(at 105.41 99.06 0)
 			(effects
@@
 			(project "rocket2-ecu"
 				(path "/02606b2c-b376-4ffb-9781-f9cea3f70994/fc637a4d-3fde-405d-ae60-ec7da7a8a72d"
-					(reference "#PWR0295")
+					(reference "#PWR0316")
 					(unit 1)
 				)
@@
 		(on_board yes)
 		(dnp no)
-		(property "Reference" "#PWR0292"
+		(property "Reference" "#PWR0313"
 			(at 87.63 102.87 0)
 			(effects
@@
 			(project "rocket2-ecu"
 				(path "/02606b2c-b376-4ffb-9781-f9cea3f70994/fc637a4d-3fde-405d-ae60-ec7da7a8a72d"
-					(reference "#PWR0292")
+					(reference "#PWR0313")
 					(unit 1)
 				)
@@
 		(dnp no)
 		(fields_autoplaced yes)
-		(property "Reference" "C95"
+		(property "Reference" "C98"
 			(at 168.91 93.9863 0)
 			(effects
@@
 			(project "rocket2-ecu"
 				(path "/02606b2c-b376-4ffb-9781-f9cea3f70994/fc637a4d-3fde-405d-ae60-ec7da7a8a72d"
-					(reference "C95")
+					(reference "C98")
 					(unit 1)
 				)
@@
 		(on_board yes)
 		(dnp no)
-		(property "Reference" "#PWR0303"
+		(property "Reference" "#PWR0324"
 			(at 205.74 93.98 0)
 			(effects
@@
 			(project "rocket2-ecu"
 				(path "/02606b2c-b376-4ffb-9781-f9cea3f70994/fc637a4d-3fde-405d-ae60-ec7da7a8a72d"
-					(reference "#PWR0303")
+					(reference "#PWR0324")
 					(unit 1)
 				)
@@
 		(on_board yes)
 		(dnp no)
-		(property "Reference" "#PWR0291"
+		(property "Reference" "#PWR0312"
 			(at 87.63 95.25 0)
 			(effects
@@
 			(project "rocket2-ecu"
 				(path "/02606b2c-b376-4ffb-9781-f9cea3f70994/fc637a4d-3fde-405d-ae60-ec7da7a8a72d"
-					(reference "#PWR0291")
+					(reference "#PWR0312")
 					(unit 1)
 				)
@@
 		(on_board yes)
 		(dnp no)
-		(property "Reference" "#PWR0293"
+		(property "Reference" "#PWR0314"
 			(at 107.95 87.63 0)
 			(effects
@@
 			(project "rocket2-ecu"
 				(path "/02606b2c-b376-4ffb-9781-f9cea3f70994/fc637a4d-3fde-405d-ae60-ec7da7a8a72d"
-					(reference "#PWR0293")
+					(reference "#PWR0314")
 					(unit 1)
 				)
@@
 		(on_board yes)
 		(dnp no)
-		(property "Reference" "#PWR0297"
+		(property "Reference" "#PWR0318"
 			(at 130.81 93.98 0)
 			(effects
@@
 			(project "rocket2-ecu"
 				(path "/02606b2c-b376-4ffb-9781-f9cea3f70994/fc637a4d-3fde-405d-ae60-ec7da7a8a72d"
-					(reference "#PWR0297")
+					(reference "#PWR0318")
 					(unit 1)
 				)
@@
 		(on_board yes)
 		(dnp no)
-		(property "Reference" "U45"
+		(property "Reference" "U48"
 			(at 200.66 103.505 0)
 			(effects
@@
 			(project "rocket2-ecu"
 				(path "/02606b2c-b376-4ffb-9781-f9cea3f70994/fc637a4d-3fde-405d-ae60-ec7da7a8a72d"
-					(reference "U45")
+					(reference "U48")
 					(unit 1)
 				)
@@
 		(dnp no)
 		(fields_autoplaced yes)
-		(property "Reference" "C94"
+		(property "Reference" "C97"
 			(at 90.17 92.7163 0)
 			(effects
@@
 			(project "rocket2-ecu"
 				(path "/02606b2c-b376-4ffb-9781-f9cea3f70994/fc637a4d-3fde-405d-ae60-ec7da7a8a72d"
-					(reference "C94")
+					(reference "C97")
 					(unit 1)
 				)
@@
 		(on_board yes)
 		(dnp no)
-		(property "Reference" "#PWR0301"
+		(property "Reference" "#PWR0322"
 			(at 195.58 96.52 0)
 			(effects
@@
 			(project "rocket2-ecu"
 				(path "/02606b2c-b376-4ffb-9781-f9cea3f70994/fc637a4d-3fde-405d-ae60-ec7da7a8a72d"
-					(reference "#PWR0301")
+					(reference "#PWR0322")
 					(unit 1)
 				)
@@
 		(on_board yes)
 		(dnp no)
-		(property "Reference" "#PWR0298"
+		(property "Reference" "#PWR0319"
 			(at 166.37 96.52 0)
 			(effects
@@
 			(project "rocket2-ecu"
 				(path "/02606b2c-b376-4ffb-9781-f9cea3f70994/fc637a4d-3fde-405d-ae60-ec7da7a8a72d"
-					(reference "#PWR0298")
+					(reference "#PWR0319")
 					(unit 1)
 				)
@@
 		(on_board yes)
 		(dnp no)
-		(property "Reference" "R115"
+		(property "Reference" "R120"
 			(at 101.346 84.328 0)
 			(effects
@@
 			(project "rocket2-ecu"
 				(path "/02606b2c-b376-4ffb-9781-f9cea3f70994/fc637a4d-3fde-405d-ae60-ec7da7a8a72d"
-					(reference "R115")
+					(reference "R120")
 					(unit 1)
 				)
@@
 		(on_board yes)
 		(dnp no)
-		(property "Reference" "#PWR0294"
+		(property "Reference" "#PWR0315"
 			(at 115.57 96.52 0)
 			(effects
@@
 			(project "rocket2-ecu"
 				(path "/02606b2c-b376-4ffb-9781-f9cea3f70994/fc637a4d-3fde-405d-ae60-ec7da7a8a72d"
-					(reference "#PWR0294")
+					(reference "#PWR0315")
 					(unit 1)
 				)
@@
 		(on_board yes)
 		(dnp no)
-		(property "Reference" "#PWR0302"
+		(property "Reference" "#PWR0323"
 			(at 185.42 99.06 0)
 			(effects
@@
 			(project "rocket2-ecu"
 				(path "/02606b2c-b376-4ffb-9781-f9cea3f70994/fc637a4d-3fde-405d-ae60-ec7da7a8a72d"
-					(reference "#PWR0302")
+					(reference "#PWR0323")
 					(unit 1)
 				)
@@
 		(on_board yes)
 		(dnp no)
-		(property "Reference" "R116"
+		(property "Reference" "R121"
 			(at 181.356 84.328 0)
 			(effects
@@
 			(project "rocket2-ecu"
 				(path "/02606b2c-b376-4ffb-9781-f9cea3f70994/fc637a4d-3fde-405d-ae60-ec7da7a8a72d"
-					(reference "R116")
+					(reference "R121")
 					(unit 1)
 				)
@@
 		(on_board yes)
 		(dnp no)
-		(property "Reference" "#PWR0304"
+		(property "Reference" "#PWR0325"
 			(at 210.82 93.98 0)
 			(effects
@@
 			(project "rocket2-ecu"
 				(path "/02606b2c-b376-4ffb-9781-f9cea3f70994/fc637a4d-3fde-405d-ae60-ec7da7a8a72d"
-					(reference "#PWR0304")
+					(reference "#PWR0325")
 					(unit 1)
 				)
@@
 		(on_board yes)
 		(dnp no)
-		(property "Reference" "#PWR0299"
+		(property "Reference" "#PWR0320"
 			(at 166.37 104.14 0)
 			(effects
@@
 			(project "rocket2-ecu"
 				(path "/02606b2c-b376-4ffb-9781-f9cea3f70994/fc637a4d-3fde-405d-ae60-ec7da7a8a72d"
-					(reference "#PWR0299")
+					(reference "#PWR0320")
 					(unit 1)
 				)
@@
 		(on_board yes)
 		(dnp no)
-		(property "Reference" "#PWR0296"
+		(property "Reference" "#PWR0317"
 			(at 125.73 93.98 0)
 			(effects
@@
 			(project "rocket2-ecu"
 				(path "/02606b2c-b376-4ffb-9781-f9cea3f70994/fc637a4d-3fde-405d-ae60-ec7da7a8a72d"
-					(reference "#PWR0296")
-					(unit 1)
-				)
+					(reference "#PWR0317")
+					(unit 1)
+				)

Commit message: Assigned almost all footprints
Parts:
- C96: renamed from C97; footprint Capacitor_SMD:C_0603_1608Metric -> Capacitor_SMD:C_0402_1005Metric; Part # (none) -> Generic 100nF 6.3V X7R 0402 MLCC
- C97: renamed from C98; footprint Capacitor_SMD:C_0603_1608Metric -> Capacitor_SMD:C_0402_1005Metric; Part # (none) -> Generic 100nF 6.3V X7R 0402 MLCC
- R119: renamed from R120; value 100k -> 100K; footprint Resistor_SMD:R_0603_1608Metric_Pad0.98x0.95mm_HandSolder -> Resistor_SMD:R_0402_1005Metric; Part # Generic 100k 1% 0402 Chip Resistor -> Generic 100K 5% 0402 Resistor
- R120: renamed from R121; value 100k -> 100K; footprint Resistor_SMD:R_0603_1608Metric_Pad0.98x0.95mm_HandSolder -> Resistor_SMD:R_0402_1005Metric; Part # Generic 100k 1% 0402 Chip Resistor -> Generic 100K 5% 0402 Resistor
- renumbered U47 to U46, U48 to U47
Changed lines of the file:
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@@
 		(on_board yes)
 		(dnp no)
-		(property "Reference" "U47"
+		(property "Reference" "U46"
 			(at 120.65 103.505 0)
 			(effects
@@
 			(project "rocket2-ecu"
 				(path "/02606b2c-b376-4ffb-9781-f9cea3f70994/fc637a4d-3fde-405d-ae60-ec7da7a8a72d"
-					(reference "U47")
+					(reference "U46")
 					(unit 1)
 				)
@@
 		(on_board yes)
 		(dnp no)
-		(property "Reference" "#PWR0321"
+		(property "Reference" "#PWR0315"
 			(at 187.96 87.63 0)
 			(effects
@@
 			(project "rocket2-ecu"
 				(path "/02606b2c-b376-4ffb-9781-f9cea3f70994/fc637a4d-3fde-405d-ae60-ec7da7a8a72d"
-					(reference "#PWR0321")
+					(reference "#PWR0315")
 					(unit 1)
 				)
@@
 		(on_board yes)
 		(dnp no)
-		(property "Reference" "#PWR0316"
+		(property "Reference" "#PWR0310"
 			(at 105.41 99.06 0)
 			(effects
@@
 			(project "rocket2-ecu"
 				(path "/02606b2c-b376-4ffb-9781-f9cea3f70994/fc637a4d-3fde-405d-ae60-ec7da7a8a72d"
-					(reference "#PWR0316")
+					(reference "#PWR0310")
 					(unit 1)
 				)
@@
 		(on_board yes)
 		(dnp no)
-		(property "Reference" "#PWR0313"
+		(property "Reference" "#PWR0307"
 			(at 87.63 102.87 0)
 			(effects
@@
 			(project "rocket2-ecu"
 				(path "/02606b2c-b376-4ffb-9781-f9cea3f70994/fc637a4d-3fde-405d-ae60-ec7da7a8a72d"
-					(reference "#PWR0313")
+					(reference "#PWR0307")
 					(unit 1)
 				)
@@
 		(dnp no)
 		(fields_autoplaced yes)
-		(property "Reference" "C98"
+		(property "Reference" "C97"
 			(at 168.91 93.9863 0)
 			(effects
@@
 			)
 		)
-		(property "Footprint" "Capacitor_SMD:C_0603_1608Metric"
+		(property "Footprint" "Capacitor_SMD:C_0402_1005Metric"
 			(at 166.37 95.25 0)
 			(effects
@@
 			)
 		)
+		(property "Part #" "Generic 100nF 6.3V X7R 0402 MLCC"
+			(at 166.37 95.25 0)
+			(effects
+				(font
+					(size 1.27 1.27)
+				)
+				(hide yes)
+			)
+		)
 		(pin "1"
 		)
@@
 			(project "rocket2-ecu"
 				(path "/02606b2c-b376-4ffb-9781-f9cea3f70994/fc637a4d-3fde-405d-ae60-ec7da7a8a72d"
-					(reference "C98")
+					(reference "C97")
 					(unit 1)
 				)
@@
 		(on_board yes)
 		(dnp no)
-		(property "Reference" "#PWR0324"
+		(property "Reference" "#PWR0318"
 			(at 205.74 93.98 0)
 			(effects
@@
 			(project "rocket2-ecu"
 				(path "/02606b2c-b376-4ffb-9781-f9cea3f70994/fc637a4d-3fde-405d-ae60-ec7da7a8a72d"
-					(reference "#PWR0324")
+					(reference "#PWR0318")
 					(unit 1)
 				)
@@
 		(on_board yes)
 		(dnp no)
-		(property "Reference" "#PWR0312"
+		(property "Reference" "#PWR0306"
 			(at 87.63 95.25 0)
 			(effects
@@
 			(project "rocket2-ecu"
 				(path "/02606b2c-b376-4ffb-9781-f9cea3f70994/fc637a4d-3fde-405d-ae60-ec7da7a8a72d"
-					(reference "#PWR0312")
+					(reference "#PWR0306")
 					(unit 1)
 				)
@@
 		(on_board yes)
 		(dnp no)
-		(property "Reference" "#PWR0314"
+		(property "Reference" "#PWR0308"
 			(at 107.95 87.63 0)
 			(effects
@@
 			(project "rocket2-ecu"
 				(path "/02606b2c-b376-4ffb-9781-f9cea3f70994/fc637a4d-3fde-405d-ae60-ec7da7a8a72d"
-					(reference "#PWR0314")
+					(reference "#PWR0308")
 					(unit 1)
 				)
@@
 		(on_board yes)
 		(dnp no)
-		(property "Reference" "#PWR0318"
+		(property "Reference" "#PWR0312"
 			(at 130.81 93.98 0)
 			(effects
@@
 			(project "rocket2-ecu"
 				(path "/02606b2c-b376-4ffb-9781-f9cea3f70994/fc637a4d-3fde-405d-ae60-ec7da7a8a72d"
-					(reference "#PWR0318")
+					(reference "#PWR0312")
 					(unit 1)
 				)
@@
 		(on_board yes)
 		(dnp no)
-		(property "Reference" "U48"
+		(property "Reference" "U47"
 			(at 200.66 103.505 0)
 			(effects
@@
 			(project "rocket2-ecu"
 				(path "/02606b2c-b376-4ffb-9781-f9cea3f70994/fc637a4d-3fde-405d-ae60-ec7da7a8a72d"
-					(reference "U48")
+					(reference "U47")
 					(unit 1)
 				)
@@
 		(dnp no)
 		(fields_autoplaced yes)
-		(property "Reference" "C97"
+		(property "Reference" "C96"
 			(at 90.17 92.7163 0)
 			(effects
@@
 			)
 		)
-		(property "Footprint" "Capacitor_SMD:C_0603_1608Metric"
+		(property "Footprint" "Capacitor_SMD:C_0402_1005Metric"
 			(at 87.63 93.98 0)
 			(effects
@@
 			)
 		)
+		(property "Part #" "Generic 100nF 6.3V X7R 0402 MLCC"
+			(at 87.63 93.98 0)
+			(effects
+				(font
+					(size 1.27 1.27)
+				)
+				(hide yes)
+			)
+		)
 		(pin "1"
 		)
@@
 			(project "rocket2-ecu"
 				(path "/02606b2c-b376-4ffb-9781-f9cea3f70994/fc637a4d-3fde-405d-ae60-ec7da7a8a72d"
-					(reference "C97")
+					(reference "C96")
 					(unit 1)
 				)
@@
 		(on_board yes)
 		(dnp no)
-		(property "Reference" "#PWR0322"
+		(property "Reference" "#PWR0316"
 			(at 195.58 96.52 0)
 			(effects
@@
 			(project "rocket2-ecu"
 				(path "/02606b2c-b376-4ffb-9781-f9cea3f70994/fc637a4d-3fde-405d-ae60-ec7da7a8a72d"
-					(reference "#PWR0322")
+					(reference "#PWR0316")
 					(unit 1)
 				)
@@
 		(on_board yes)
 		(dnp no)
-		(property "Reference" "#PWR0319"
+		(property "Reference" "#PWR0313"
 			(at 166.37 96.52 0)
 			(effects
@@
 			(project "rocket2-ecu"
 				(path "/02606b2c-b376-4ffb-9781-f9cea3f70994/fc637a4d-3fde-405d-ae60-ec7da7a8a72d"
-					(reference "#PWR0319")
+					(reference "#PWR0313")
 					(unit 1)
 				)
@@
 		(on_board yes)
 		(dnp no)
-		(property "Reference" "R120"
+		(property "Reference" "R119"
 			(at 101.346 84.328 0)
 			(effects
@@
 			)
 		)
-		(property "Value" "100k"
+		(property "Value" "100K"
 			(at 101.346 86.868 0)
 			(effects
@@
 			)
 		)
-		(property "Footprint" "Resistor_SMD:R_0603_1608Metric_Pad0.98x0.95mm_HandSolder"
+		(property "Footprint" "Resistor_SMD:R_0402_1005Metric"
 			(at 107.95 86.36 0)
 			(effects
@@
 			)
 		)
-		(property "Part #" "Generic 100k 1% 0402 Chip Resistor"
+		(property "Part #" "Generic 100K 5% 0402 Resistor"
 			(at 107.95 86.36 0)
 			(effects
@@
 			(project "rocket2-ecu"
 				(path "/02606b2c-b376-4ffb-9781-f9cea3f70994/fc637a4d-3fde-405d-ae60-ec7da7a8a72d"
-					(reference "R120")
+					(reference "R119")
 					(unit 1)
 				)
@@
 		(on_board yes)
 		(dnp no)
-		(property "Reference" "#PWR0315"
+		(property "Reference" "#PWR0309"
 			(at 115.57 96.52 0)
 			(effects
@@
 			(project "rocket2-ecu"
 				(path "/02606b2c-b376-4ffb-9781-f9cea3f70994/fc637a4d-3fde-405d-ae60-ec7da7a8a72d"
-					(reference "#PWR0315")
+					(reference "#PWR0309")
 					(unit 1)
 				)
@@
 		(on_board yes)
 		(dnp no)
-		(property "Reference" "#PWR0323"
+		(property "Reference" "#PWR0317"
 			(at 185.42 99.06 0)
 			(effects
@@
 			(project "rocket2-ecu"
 				(path "/02606b2c-b376-4ffb-9781-f9cea3f70994/fc637a4d-3fde-405d-ae60-ec7da7a8a72d"
-					(reference "#PWR0323")
+					(reference "#PWR0317")
 					(unit 1)
 				)
@@
 		(on_board yes)
 		(dnp no)
-		(property "Reference" "R121"
+		(property "Reference" "R120"
 			(at 181.356 84.328 0)
 			(effects
@@
 			)
 		)
-		(property "Value" "100k"
+		(property "Value" "100K"
 			(at 181.356 86.868 0)
 			(effects
@@
 			)
 		)
-		(property "Footprint" "Resistor_SMD:R_0603_1608Metric_Pad0.98x0.95mm_HandSolder"
+		(property "Footprint" "Resistor_SMD:R_0402_1005Metric"
 			(at 187.96 86.36 0)
 			(effects
@@
 			)
 		)
-		(property "Part #" "Generic 100k 1% 0402 Chip Resistor"
+		(property "Part #" "Generic 100K 5% 0402 Resistor"
 			(at 187.96 86.36 0)
 			(effects
@@
 			(project "rocket2-ecu"
 				(path "/02606b2c-b376-4ffb-9781-f9cea3f70994/fc637a4d-3fde-405d-ae60-ec7da7a8a72d"
-					(reference "R121")
+					(reference "R120")
 					(unit 1)
 				)
@@
 		(on_board yes)
 		(dnp no)
-		(property "Reference" "#PWR0325"
+		(property "Reference" "#PWR0319"
 			(at 210.82 93.98 0)
 			(effects
@@
 			(project "rocket2-ecu"
 				(path "/02606b2c-b376-4ffb-9781-f9cea3f70994/fc637a4d-3fde-405d-ae60-ec7da7a8a72d"
-					(reference "#PWR0325")
+					(reference "#PWR0319")
 					(unit 1)
 				)
@@
 		(on_board yes)
 		(dnp no)
-		(property "Reference" "#PWR0320"
+		(property "Reference" "#PWR0314"
 			(at 166.37 104.14 0)
 			(effects
@@
 			(project "rocket2-ecu"
 				(path "/02606b2c-b376-4ffb-9781-f9cea3f70994/fc637a4d-3fde-405d-ae60-ec7da7a8a72d"
-					(reference "#PWR0320")
+					(reference "#PWR0314")
 					(unit 1)
 				)
@@
 		(on_board yes)
 		(dnp no)
-		(property "Reference" "#PWR0317"
+		(property "Reference" "#PWR0311"
 			(at 125.73 93.98 0)
 			(effects
@@
 			(project "rocket2-ecu"
 				(path "/02606b2c-b376-4ffb-9781-f9cea3f70994/fc637a4d-3fde-405d-ae60-ec7da7a8a72d"
-					(reference "#PWR0317")
-					(unit 1)
-				)
+					(reference "#PWR0311")
+					(unit 1)
+				)

Commit message: new BOM
Parts:
- C96, C97: Manufacturer (none) -> Generic; Part # Generic 100nF 6.3V X7R 0402 MLCC -> Generic CAP CER 0.1UF 6.3V X7R 0402
- R119, R120: Part # Generic 100K 5% 0402 Resistor -> Generic RES SMD 100K OHM 1% 1/16W 0402
Changed lines of the file:
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@@
 			)
 		)
-		(property "Part #" "Generic 100nF 6.3V X7R 0402 MLCC"
+		(property "Part #" "Generic CAP CER 0.1UF 6.3V X7R 0402"
+			(at 166.37 95.25 0)
+			(effects
+				(font
+					(size 1.27 1.27)
+				)
+				(hide yes)
+			)
+		)
+		(property "Manufacturer" "Generic"
 			(at 166.37 95.25 0)
 			(effects
@@
 			)
 		)
-		(property "Part #" "Generic 100nF 6.3V X7R 0402 MLCC"
+		(property "Part #" "Generic CAP CER 0.1UF 6.3V X7R 0402"
+			(at 87.63 93.98 0)
+			(effects
+				(font
+					(size 1.27 1.27)
+				)
+				(hide yes)
+			)
+		)
+		(property "Manufacturer" "Generic"
 			(at 87.63 93.98 0)
 			(effects
@@
 			)
 		)
-		(property "Part #" "Generic 100K 5% 0402 Resistor"
+		(property "Part #" "Generic RES SMD 100K OHM 1% 1/16W 0402"
 			(at 107.95 86.36 0)
 			(effects
@@
 			)
 		)
-		(property "Part #" "Generic 100K 5% 0402 Resistor"
+		(property "Part #" "Generic RES SMD 100K OHM 1% 1/16W 0402"
 			(at 187.96 86.36 0)
 			(effects

Commit message: idk what I changed tbh
Parts:
- U46, U47: footprint Package_SO:SOIC-8W_5.3x5.3mm_P1.27mm -> Package_SON:WSON-8-1EP_8x6mm_P1.27mm_EP3.4x4.3mm
Changed lines of the file:
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@@
 			)
 		)
-		(property "Footprint" "Package_SO:SOIC-8W_5.3x5.3mm_P1.27mm"
+		(property "Footprint" "Package_SON:WSON-8-1EP_8x6mm_P1.27mm_EP3.4x4.3mm"
 			(at 120.65 95.25 0)
 			(effects
@@
 			)
 		)
-		(property "Footprint" "Package_SO:SOIC-8W_5.3x5.3mm_P1.27mm"
+		(property "Footprint" "Package_SON:WSON-8-1EP_8x6mm_P1.27mm_EP3.4x4.3mm"
 			(at 200.66 95.25 0)
 			(effects
