File: ECU_Radios.kicad_sch (KiCad schematic)
At the start: 12 parts, among them J20 SMA, J22 SMA

Commit message: layout done
Parts:
- J20, J22: footprint Connector_Coaxial:SMA_Molex_73251-2200_Horizontal -> 0UCIRP-KiCAD-Lib:CONN_73391-0070_MOL
Changed lines of the file:
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@@
 			)
 		)
-		(property "Footprint" "Connector_Coaxial:SMA_Molex_73251-2200_Horizontal"
+		(property "Footprint" "0UCIRP-KiCAD-Lib:CONN_73391-0070_MOL"
 			(at 158.75 77.47 0)
 			(effects
@@
 			)
 		)
-		(property "Datasheet" "https://www.molex.com/en-us/products/part-detail/732512200?display=pdf"
+		(property "Datasheet" "https://www.molex.com/en-us/products/part-detail/733910070?display=pdf"
 			(at 158.75 77.47 0)
 			(effects
@@
 			)
 		)
-		(property "Footprint" "Connector_Coaxial:SMA_Molex_73251-2200_Horizontal"
+		(property "Footprint" "0UCIRP-KiCAD-Lib:CONN_73391-0070_MOL"
 			(at 58.42 77.47 0)
 			(effects
@@
 			)
 		)
-		(property "Datasheet" "https://www.molex.com/en-us/products/part-detail/732512200?display=pdf"
+		(property "Datasheet" "https://www.molex.com/en-us/products/part-detail/733910070?display=pdf"
 			(at 58.42 77.47 0)
 			(effects

Commit message: version in PCBway 12/12/2025
Parts:
- U43, U45: now not fitted
Changed lines of the file:
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@@
 		(in_bom yes)
 		(on_board yes)
-		(dnp no)
+		(dnp yes)
 		(property "Reference" "U43"
 			(at 96.52 49.53 0)
@@
 		(in_bom yes)
 		(on_board yes)
-		(dnp no)
+		(dnp yes)
 		(property "Reference" "U45"
 			(at 196.85 49.53 0)

Commit message: changed charging circuit for Insta360, gonna send in now on JLCPCB
Parts:
- R13, R9: value 100 -> 470
- U43, U45: now fitted
Other:
- note added: "TRS Radio Module 0"
- note added: "TRS Radio Module 1"
- note removed: "Removed DIO0 so we have vsense"
- note removed: "TRS Radio Module"
- note removed: "TRS Radio Module 2"
Changed lines of the file:
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@@
 	(generator_version "9.0")
 	(paper "A4")
-	(text "TRS Radio Module 2"
+	(text "TRS Radio Module 1"
 		(exclude_from_sim no)
 		(at 201.676 93.98 0)
@@
 		)
 	)
-	(text "Removed DIO0 so we have vsense"
-		(exclude_from_sim no)
-		(at 249.682 61.976 0)
-		(effects
-			(font
-				(size 1.27 1.27)
-				(color 255 40 86 1)
-			)
-		)
-	)
-	(text "TRS Radio Module"
+	(text "TRS Radio Module 0"
 		(exclude_from_sim no)
 		(at 101.346 92.456 0)
@@
 			)
 		)
-		(property "Datasheet" "https://www.molex.com/en-us/products/part-detail/733910070?display=pdf"
+		(property "Datasheet" "~"
 			(at 158.75 77.47 0)
 			(effects
@@
 			)
 		)
-		(property "Description" ""
+		(property "Description" "coaxial connector (BNC, SMA, SMB, SMC, Cinch/RCA, LEMO, ...)"
 			(at 158.75 77.47 0)
 			(effects
@@
 			)
 		)
-		(property "Description" ""
+		(property "Description" "Light emitting diode, small symbol"
 			(at 137.16 72.39 0)
 			(effects
@@
 		)
 		(property "Part #" "Generic 0603 Red LED"
+			(at 137.16 72.39 0)
+			(effects
+				(font
+					(size 1.27 1.27)
+				)
+				(hide yes)
+			)
+		)
+		(property "Sim.Pin" "1=K 2=A"
 			(at 137.16 72.39 0)
 			(effects
@@
 			)
 		)
-		(property "Description" ""
+		(property "Description" "Power symbol creates a global label with name \"+3.3V\""
 			(at 191.77 53.34 0)
 			(effects
@@
 			)
 		)
-		(property "Description" ""
+		(property "Description" "Power symbol creates a global label with name \"GND\" , ground"
 			(at 158.75 82.55 0)
 			(effects
@@
 			)
 		)
-		(property "Description" ""
+		(property "Description" "Power symbol creates a global label with name \"GND\" , ground"
 			(at 227.33 59.69 0)
 			(effects
@@
 			)
 		)
-		(property "Value" "100"
+		(property "Value" "470"
 			(at 141.986 68.58 0)
 			(effects
@@
 			)
 		)
-		(property "Description" ""
+		(property "Description" "Resistor, small US symbol"
 			(at 137.16 67.31 0)
 			(effects
@@
 			)
 		)
-		(property "Description" ""
+		(property "Description" "Power symbol creates a global label with name \"GND\" , ground"
 			(at 137.16 74.93 0)
 			(effects
@@
 			)
 		)
-		(property "Description" ""
+		(property "Description" "Power symbol creates a global label with name \"+3.3V\""
 			(at 91.44 53.34 0)
 			(effects
@@
 		(in_bom yes)
 		(on_board yes)
-		(dnp yes)
+		(dnp no)
 		(property "Reference" "U43"
 			(at 96.52 49.53 0)
@@
 			)
 		)
-		(property "Description" ""
+		(property "Description" "Resistor, small US symbol"
 			(at 59.69 57.15 0)
 			(effects
@@
 			)
 		)
-		(property "Description" ""
+		(property "Description" "Power symbol creates a global label with name \"+3.3V\""
 			(at 127 54.61 0)
 			(effects
@@
 			)
 		)
-		(property "Description" ""
+		(property "Description" "Unpolarized capacitor, small symbol"
 			(at 127 57.15 0)
 			(effects
@@
 			)
 		)
-		(property "Description" ""
+		(property "Description" "Power symbol creates a global label with name \"GND\" , ground"
 			(at 191.77 88.9 0)
 			(effects
@@
 			)
 		)
-		(property "Description" ""
+		(property "Description" "Light emitting diode, small symbol"
 			(at 36.83 71.12 0)
 			(effects
@@
 		)
 		(property "Part #" "Generic 0603 Red LED"
+			(at 36.83 71.12 0)
+			(effects
+				(font
+					(size 1.27 1.27)
+				)
+				(hide yes)
+			)
+		)
+		(property "Sim.Pin" "1=K 2=A"
 			(at 36.83 71.12 0)
 			(effects
@@
 			)
 		)
-		(property "Description" ""
+		(property "Description" "Power symbol creates a global label with name \"GND\" , ground"
 			(at 127 59.69 0)
 			(effects
@@
 			)
 		)
-		(property "Datasheet" "https://www.molex.com/en-us/products/part-detail/733910070?display=pdf"
+		(property "Datasheet" "~"
 			(at 58.42 77.47 0)
 			(effects
@@
 			)
 		)
-		(property "Description" ""
+		(property "Description" "coaxial connector (BNC, SMA, SMB, SMC, Cinch/RCA, LEMO, ...)"
 			(at 58.42 77.47 0)
 			(effects
@@
 			)
 		)
-		(property "Value" "100"
+		(property "Value" "470"
 			(at 41.656 67.31 0)
 			(effects
@@
 			)
 		)
-		(property "Description" ""
+		(property "Description" "Resistor, small US symbol"
 			(at 36.83 66.04 0)
 			(effects
@@
 			)
 		)
-		(property "Description" ""
+		(property "Description" "Resistor, small US symbol"
 			(at 160.02 57.15 0)
 			(effects
@@
 		(in_bom yes)
 		(on_board yes)
-		(dnp yes)
+		(dnp no)
 		(property "Reference" "U45"
 			(at 196.85 49.53 0)
@@
 			)
 		)
-		(property "Description" ""
+		(property "Description" "Power symbol creates a global label with name \"GND\" , ground"
 			(at 36.83 73.66 0)
 			(effects
@@
 			)
 		)
-		(property "Description" ""
+		(property "Description" "Power symbol creates a global label with name \"GND\" , ground"
 			(at 91.44 88.9 0)
 			(effects
@@
 			)
 		)
-		(property "Description" ""
+		(property "Description" "Power symbol creates a global label with name \"GND\" , ground"
 			(at 58.42 82.55 0)
 			(effects
@@
 			)
 		)
-		(property "Description" ""
+		(property "Description" "Unpolarized capacitor, small symbol"
 			(at 227.33 57.15 0)
 			(effects
@@
 			)
 		)
-		(property "Description" ""
+		(property "Description" "Power symbol creates a global label with name \"+3.3V\""
 			(at 227.33 54.61 0)
 			(effects
