File: PowerReg.kicad_sch (KiCad schematic)
At the start: 17 parts, among them U7 24V->3.3V 3A

Commit message: added some production files
Parts:
- L2: Manufacturer Vishay Dale -> TDK Corporation; Part # IHLP1212BZER2R2M11 -> VLS3012HBX-2R2M
Changed lines of the file:
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@@
 			)
 		)
-		(property "Datasheet" "https://www.vishay.com/docs/34289/lp12bz11.pdf"
+		(property "Datasheet" "https://product.tdk.com/en/system/files/dam/doc/product/inductor/inductor/smd/catalog/inductor_commercial_power_vls3012hbx_en.pdf"
 			(at 177.8 88.9 0)
 			(effects
@@
 			)
 		)
-		(property "Part #" "IHLP1212BZER2R2M11"
+		(property "Part #" "VLS3012HBX-2R2M"
 			(at 177.8 88.9 90)
 			(effects
@@
 			)
 		)
-		(property "Manufacturer" "Vishay Dale"
+		(property "Manufacturer" "  TDK Corporation"
 			(at 177.8 88.9 90)
 			(effects

Commit message: changed charging circuit for Insta360, gonna send in now on JLCPCB
Parts:
- L2: Manufacturer TDK Corporation -> Vishay Dale; Part # VLS3012HBX-2R2M -> IHLP1212BZEV2R2MA1
Changed lines of the file:
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@@
 			)
 		)
-		(property "Description" ""
+		(property "Description" "Power symbol creates a global label with name \"GND\" , ground"
 			(at 179.07 43.18 0)
 			(effects
@@
 	)
 	(symbol
-		(lib_name "GND_7")
 		(lib_id "power:GND")
 		(at 219.71 93.98 0)
@@
 	)
 	(symbol
-		(lib_name "GND_6")
 		(lib_id "power:GND")
 		(at 223.52 101.6 90)
@@
 	)
 	(symbol
-		(lib_name "GND_9")
 		(lib_id "power:GND")
 		(at 163.83 93.98 0)
@@
 			)
 		)
-		(property "Description" ""
+		(property "Description" "Resistor, small US symbol"
 			(at 241.3 88.9 0)
 			(effects
@@
 			)
 		)
-		(property "Datasheet" "https://product.tdk.com/en/system/files/dam/doc/product/inductor/inductor/smd/catalog/inductor_commercial_power_vls3012hbx_en.pdf"
+		(property "Datasheet" "~"
 			(at 177.8 88.9 0)
 			(effects
@@
 			)
 		)
-		(property "Part #" "VLS3012HBX-2R2M"
+		(property "Part #" "IHLP1212BZEV2R2MA1"
 			(at 177.8 88.9 90)
 			(effects
@@
 			)
 		)
-		(property "Manufacturer" "  TDK Corporation"
+		(property "Manufacturer" "Vishay Dale"
 			(at 177.8 88.9 90)
 			(effects
@@
 			)
 		)
-		(property "Description" "10uF 50V X7R Generic"
+		(property "Description" "Unpolarized capacitor, small symbol"
 			(at 156.21 91.44 0)
 			(effects
@@
 			)
 		)
-		(property "Description" ""
+		(property "Description" "Power symbol creates a global label with name \"GND\" , ground"
 			(at 48.26 96.52 0)
 			(effects
@@
 			)
 		)
-		(property "Description" "10uF 25V X7R Generic"
+		(property "Description" "Unpolarized capacitor, small symbol"
 			(at 219.71 91.44 0)
 			(effects
@@
 	)
 	(symbol
-		(lib_name "GND_8")
 		(lib_id "power:GND")
 		(at 187.96 97.79 0)
@@
 	)
 	(symbol
-		(lib_name "GND_9")
 		(lib_id "power:GND")
 		(at 171.45 93.98 0)
@@
 	)
 	(symbol
-		(lib_name "GND_9")
 		(lib_id "power:GND")
 		(at 184.15 93.98 0)
@@
 			)
 		)
-		(property "Description" "10uF 50V X7R Generic"
+		(property "Description" "Unpolarized capacitor, small symbol"
 			(at 171.45 91.44 0)
 			(effects
@@
 	)
 	(symbol
-		(lib_name "GND_6")
 		(lib_id "power:GND")
 		(at 200.66 110.49 0)
@@
 			)
 		)
-		(property "Description" "10uF 50V X7R Generic"
+		(property "Description" "Unpolarized capacitor, small symbol"
 			(at 184.15 91.44 0)
 			(effects
@@
 			)
 		)
-		(property "Description" "10uF 50V X7R Generic"
+		(property "Description" "Unpolarized capacitor, small symbol"
 			(at 163.83 91.44 0)
 			(effects
@@
 			)
 		)
-		(property "Description" ""
+		(property "Description" "Light emitting diode, small symbol"
 			(at 220.98 101.6 0)
 			(effects
@@
 		)
 		(property "Part #" "Generic 0603 Yellow-Green LED"
+			(at 220.98 101.6 0)
+			(effects
+				(font
+					(size 1.27 1.27)
+				)
+				(hide yes)
+			)
+		)
+		(property "Sim.Pin" "1=K 2=A"
 			(at 220.98 101.6 0)
 			(effects
@@
 			)
 		)
-		(property "Description" ""
+		(property "Description" "Power symbol creates a global label with name \"GND\" , ground"
 			(at 135.89 43.18 0)
 			(effects
@@
 	)
 	(symbol
-		(lib_name "GND_9")
 		(lib_id "power:GND")
 		(at 156.21 93.98 0)
@@
 			)
 		)
-		(property "Datasheet" "https://www.mouser.com/datasheet/2/468/RPMB_3_0-1670415.pdf"
+		(property "Datasheet" "https://www.recom-power.com/pdf/Innoline/RPM-6.0.pdf"
 			(at 200.025 95.25 0)
 			(effects
@@
 			)
 		)
-		(property "Description" ""
+		(property "Description" "6A non-isolated switching regulator power module, 4-15V input voltage, 3.3V output voltage, DOSA"
 			(at 200.66 96.52 0)
 			(effects
@@
 			)
 		)
-		(property "Description" ""
+		(property "Description" "Resistor, small US symbol"
 			(at 214.63 101.6 0)
 			(effects
