File: single-cell-charger.kicad_sch (KiCad schematic)
At the start: 15 parts, among them U12 VOS615A-1

Commit message: REDS updated with diodes and hierarchy to main micro
Parts:
- renumbered C36 to C21, C37 to C22, C38 to C23, D21 to D16
Connections:
- net +3V3 renamed +3V3_REDS

Commit message: Added power sense to rocket2-battery with voltage follower, added +1 solenoids and PT circuit, made new gx connectors
Parts:
- removed JP1: Bridge, Jumper:SolderJumper-2_P1.3mm_Open_RoundedPad1.0x1.5mm, symbol Jumper:SolderJumper_2_Bridged
- added TP1: ISO_5V, TestPoint:TestPoint_Plated_Hole_D2.0mm, symbol Connector:TestPoint
- added TP13: BAT-, TestPoint:TestPoint_Plated_Hole_D2.0mm, symbol Connector:TestPoint
- added TP7: BAT+, TestPoint:TestPoint_Plated_Hole_D2.0mm, symbol Connector:TestPoint
Connections:
- net BAT+: now also TP7.1
- net BAT-: now also TP13.1
- net ISO_5V: now also TP1.1
- net stat: now also D16.1 (K)
Changed lines of the file:
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@@
+	)
+	(junction
+		(at 180.34 88.9)
+		(diameter 0)
+		(color 0 0 0 0)
 	)
 	(junction
@@
 	)
 	(junction
+		(at 181.61 111.76)
+		(diameter 0)
+		(color 0 0 0 0)
+	)
+	(junction
 		(at 148.59 111.76)
 		(diameter 0)
@@
 	(wire
 		(pts
-			(xy 165.1 106.68) (xy 165.1 105.41)
-		)
-		(stroke
-			(width 0)
-			(type default)
-		)
-	)
-	(wire
-		(pts
 			(xy 147.32 111.76) (xy 148.59 111.76)
 		)
@@
 	(wire
 		(pts
-			(xy 165.1 96.52) (xy 165.1 97.79)
+			(xy 165.1 96.52) (xy 165.1 106.68)
 		)
 		(stroke
@@
 	(wire
 		(pts
-			(xy 149.86 111.76) (xy 191.77 111.76)
+			(xy 149.86 111.76) (xy 181.61 111.76)
 		)
 		(stroke
@@
 	(wire
 		(pts
+			(xy 181.61 111.76) (xy 191.77 111.76)
+		)
+		(stroke
+			(width 0)
+			(type default)
+		)
+	)
+	(wire
+		(pts
 			(xy 180.34 53.34) (xy 185.42 53.34)
 		)
@@
 	(wire
 		(pts
-			(xy 161.29 88.9) (xy 191.77 88.9)
+			(xy 161.29 88.9) (xy 180.34 88.9)
 		)
 		(stroke
@@
 		(pts
 			(xy 124.46 111.76) (xy 129.54 111.76)
+		)
+		(stroke
+			(width 0)
+			(type default)
+		)
+	)
+	(wire
+		(pts
+			(xy 180.34 88.9) (xy 191.77 88.9)
 		)
 		(stroke
@@
 	)
 	(symbol
+		(lib_id "Connector:TestPoint")
+		(at 180.34 88.9 0)
+		(unit 1)
+		(exclude_from_sim no)
+		(in_bom yes)
+		(on_board yes)
+		(dnp no)
+		(fields_autoplaced yes)
+		(property "Reference" "TP7"
+			(at 182.88 84.3279 0)
+			(effects
+				(font
+					(size 1.27 1.27)
+				)
+				(justify left)
+			)
+		)
+		(property "Value" "BAT+"
+			(at 182.88 86.8679 0)
+			(effects
+				(font
+					(size 1.27 1.27)
+				)
+				(justify left)
+			)
+		)
+		(property "Footprint" "TestPoint:TestPoint_Plated_Hole_D2.0mm"
+			(at 185.42 88.9 0)
+			(effects
+				(font
+					(size 1.27 1.27)
+				)
+				(hide yes)
+			)
+		)
+		(property "Datasheet" "~"
+			(at 185.42 88.9 0)
+			(effects
+				(font
+					(size 1.27 1.27)
+				)
+				(hide yes)
+			)
+		)
+		(property "Description" "test point"
+			(at 180.34 88.9 0)
+			(effects
+				(font
+					(size 1.27 1.27)
+				)
+				(hide yes)
+			)
+		)
+		(pin "1"
+		)
+		(instances
+			(project "rocket2-ecu"
+				(path "/02606b2c-b376-4ffb-9781-f9cea3f70994/c8976b66-9d7c-47d1-8ab5-e6fd9c707361/1a39f8df-dcec-4a97-951c-60148a5067ca"
+					(reference "TP8")
+					(unit 1)
+				)
+				(path "/02606b2c-b376-4ffb-9781-f9cea3f70994/c8976b66-9d7c-47d1-8ab5-e6fd9c707361/218966e8-0599-4bad-8241-95ca09109d89"
+					(reference "TP7")
+					(unit 1)
+				)
+				(path "/02606b2c-b376-4ffb-9781-f9cea3f70994/c8976b66-9d7c-47d1-8ab5-e6fd9c707361/5c1dbfcc-3925-4da2-a038-2c416606c068"
+					(reference "TP12")
+					(unit 1)
+				)
+				(path "/02606b2c-b376-4ffb-9781-f9cea3f70994/c8976b66-9d7c-47d1-8ab5-e6fd9c707361/8ab1e7d4-e52f-422c-912d-30fd70001231"
+					(reference "TP11")
+					(unit 1)
+				)
+				(path "/02606b2c-b376-4ffb-9781-f9cea3f70994/c8976b66-9d7c-47d1-8ab5-e6fd9c707361/b5f91759-085b-4a53-bede-6cb17536657b"
+					(reference "TP10")
+					(unit 1)
+				)
+				(path "/02606b2c-b376-4ffb-9781-f9cea3f70994/c8976b66-9d7c-47d1-8ab5-e6fd9c707361/eb655268-f2ac-4ac0-945d-2ba286ede0a5"
+					(reference "TP9")
+					(unit 1)
+				)
+			)
+		)
+	)
+	(symbol
 		(lib_id "UCIRP-KiCAD-Lib:EC4SAW-xxSxxN")
 		(at 81.915 100.33 0)
@@
 				(path "/453543af-7e3c-49a0-a644-4bd49c4f86f8/eb655268-f2ac-4ac0-945d-2ba286ede0a5"
 					(reference "R33")
+					(unit 1)
+				)
+			)
+		)
+	)
+	(symbol
+		(lib_id "Connector:TestPoint")
+		(at 125.73 80.01 0)
+		(unit 1)
+		(exclude_from_sim no)
+		(in_bom yes)
+		(on_board yes)
+		(dnp no)
+		(fields_autoplaced yes)
+		(property "Reference" "TP1"
+			(at 128.27 75.4379 0)
+			(effects
+				(font
+					(size 1.27 1.27)
+				)
+				(justify left)
+			)
+		)
+		(property "Value" "ISO_5V"
+			(at 128.27 77.9779 0)
+			(effects
+				(font
+					(size 1.27 1.27)
+				)
+				(justify left)
+			)
+		)
+		(property "Footprint" "TestPoint:TestPoint_Plated_Hole_D2.0mm"
+			(at 130.81 80.01 0)
+			(effects
+				(font
+					(size 1.27 1.27)
+				)
+				(hide yes)
+			)
+		)
+		(property "Datasheet" "~"
+			(at 130.81 80.01 0)
+			(effects
+				(font
+					(size 1.27 1.27)
+				)
+				(hide yes)
+			)
+		)
+		(property "Description" "test point"
+			(at 125.73 80.01 0)
+			(effects
+				(font
+					(size 1.27 1.27)
+				)
+				(hide yes)
+			)
+		)
+		(pin "1"
+		)
+		(instances
+			(project ""
+				(path "/02606b2c-b376-4ffb-9781-f9cea3f70994/c8976b66-9d7c-47d1-8ab5-e6fd9c707361/1a39f8df-dcec-4a97-951c-60148a5067ca"
+					(reference "TP2")
+					(unit 1)
+				)
+				(path "/02606b2c-b376-4ffb-9781-f9cea3f70994/c8976b66-9d7c-47d1-8ab5-e6fd9c707361/218966e8-0599-4bad-8241-95ca09109d89"
+					(reference "TP1")
+					(unit 1)
+				)
+				(path "/02606b2c-b376-4ffb-9781-f9cea3f70994/c8976b66-9d7c-47d1-8ab5-e6fd9c707361/5c1dbfcc-3925-4da2-a038-2c416606c068"
+					(reference "TP6")
+					(unit 1)
+				)
+				(path "/02606b2c-b376-4ffb-9781-f9cea3f70994/c8976b66-9d7c-47d1-8ab5-e6fd9c707361/8ab1e7d4-e52f-422c-912d-30fd70001231"
+					(reference "TP5")
+					(unit 1)
+				)
+				(path "/02606b2c-b376-4ffb-9781-f9cea3f70994/c8976b66-9d7c-47d1-8ab5-e6fd9c707361/b5f91759-085b-4a53-bede-6cb17536657b"
+					(reference "TP4")
+					(unit 1)
+				)
+				(path "/02606b2c-b376-4ffb-9781-f9cea3f70994/c8976b66-9d7c-47d1-8ab5-e6fd9c707361/eb655268-f2ac-4ac0-945d-2ba286ede0a5"
+					(reference "TP3")
 					(unit 1)
 				)
@@
 				(path "/02606b2c-b376-4ffb-9781-f9cea3f70994/c8976b66-9d7c-47d1-8ab5-e6fd9c707361/eb655268-f2ac-4ac0-945d-2ba286ede0a5"
 					(reference "R50")
-					(unit 1)
-				)
-			)
-		)
-	)
-	(symbol
-		(lib_id "Jumper:SolderJumper_2_Bridged")
-		(at 165.1 101.6 90)
-		(unit 1)
-		(exclude_from_sim no)
-		(in_bom yes)
-		(on_board yes)
-		(dnp no)
-		(property "Reference" "JP1"
-			(at 157.48 100.33 90)
-			(effects
-				(font
-					(size 1.27 1.27)
-				)
-				(justify right)
-			)
-		)
-		(property "Value" "Bridge"
-			(at 157.48 102.87 90)
-			(effects
-				(font
-					(size 1.27 1.27)
-				)
-				(justify right)
-			)
-		)
-		(property "Footprint" "Jumper:SolderJumper-2_P1.3mm_Open_RoundedPad1.0x1.5mm"
-			(at 165.1 101.6 0)
-			(effects
-				(font
-					(size 1.27 1.27)
-				)
-				(hide yes)
-			)
-		)
-		(property "Datasheet" "~"
-			(at 165.1 101.6 0)
-			(effects
-				(font
-					(size 1.27 1.27)
-				)
-				(hide yes)
-			)
-		)
-		(property "Description" ""
-			(at 165.1 101.6 0)
-			(effects
-				(font
-					(size 1.27 1.27)
-				)
-				(hide yes)
-			)
-		)
-		(pin "1"
-		)
-		(pin "2"
-		)
-		(instances
-			(project "rocket2-ecu"
-				(path "/02606b2c-b376-4ffb-9781-f9cea3f70994/c8976b66-9d7c-47d1-8ab5-e6fd9c707361/1a39f8df-dcec-4a97-951c-60148a5067ca"
-					(reference "JP2")
-					(unit 1)
-				)
-				(path "/02606b2c-b376-4ffb-9781-f9cea3f70994/c8976b66-9d7c-47d1-8ab5-e6fd9c707361/218966e8-0599-4bad-8241-95ca09109d89"
-					(reference "JP1")
-					(unit 1)
-				)
-				(path "/02606b2c-b376-4ffb-9781-f9cea3f70994/c8976b66-9d7c-47d1-8ab5-e6fd9c707361/5c1dbfcc-3925-4da2-a038-2c416606c068"
-					(reference "JP6")
-					(unit 1)
-				)
-				(path "/02606b2c-b376-4ffb-9781-f9cea3f70994/c8976b66-9d7c-47d1-8ab5-e6fd9c707361/8ab1e7d4-e52f-422c-912d-30fd70001231"
-					(reference "JP5")
-					(unit 1)
-				)
-				(path "/02606b2c-b376-4ffb-9781-f9cea3f70994/c8976b66-9d7c-47d1-8ab5-e6fd9c707361/b5f91759-085b-4a53-bede-6cb17536657b"
-					(reference "JP4")
-					(unit 1)
-				)
-				(path "/02606b2c-b376-4ffb-9781-f9cea3f70994/c8976b66-9d7c-47d1-8ab5-e6fd9c707361/eb655268-f2ac-4ac0-945d-2ba286ede0a5"
-					(reference "JP3")
 					(unit 1)
 				)
@@
 					(unit 1)
 				)
+			)
+		)
+	)
+	(symbol
+		(lib_id "Connector:TestPoint")
+		(at 181.61 111.76 180)
+		(unit 1)
+		(exclude_from_sim no)
+		(in_bom yes)
+		(on_board yes)
+		(dnp no)
+		(fields_autoplaced yes)
+		(property "Reference" "TP13"
+			(at 184.15 113.7919 0)
+			(effects
+				(font
+					(size 1.27 1.27)
+				)
+				(justify right)
+			)
+		)
+		(property "Value" "BAT-"
+			(at 184.15 116.3319 0)
+			(effects
+				(font
+					(size 1.27 1.27)
+				)
+				(justify right)
+			)
+		)
+		(property "Footprint" "TestPoint:TestPoint_Plated_Hole_D2.0mm"
+			(at 176.53 111.76 0)
+			(effects
+				(font
+					(size 1.27 1.27)
+				)
+				(hide yes)
+			)
+		)
+		(property "Datasheet" "~"
+			(at 176.53 111.76 0)
+			(effects
+				(font
+					(size 1.27 1.27)
+				)
+				(hide yes)
+			)
+		)
+		(property "Description" "test point"
+			(at 181.61 111.76 0)
+			(effects
+				(font
+					(size 1.27 1.27)
+				)
+				(hide yes)
+			)
+		)
+		(pin "1"
+		)
+		(instances
+			(project "rocket2-ecu"
+				(path "/02606b2c-b376-4ffb-9781-f9cea3f70994/c8976b66-9d7c-47d1-8ab5-e6fd9c707361/1a39f8df-dcec-4a97-951c-60148a5067ca"
+					(reference "TP14")
+					(unit 1)
+				)
+				(path "/02606b2c-b376-4ffb-9781-f9cea3f70994/c8976b66-9d7c-47d1-8ab5-e6fd9c707361/218966e8-0599-4bad-8241-95ca09109d89"
+					(reference "TP13")
+					(unit 1)
+				)
+				(path "/02606b2c-b376-4ffb-9781-f9cea3f70994/c8976b66-9d7c-47d1-8ab5-e6fd9c707361/5c1dbfcc-3925-4da2-a038-2c416606c068"
+					(reference "TP18")
+					(unit 1)
+				)
+				(path "/02606b2c-b376-4ffb-9781-f9cea3f70994/c8976b66-9d7c-47d1-8ab5-e6fd9c707361/8ab1e7d4-e52f-422c-912d-30fd70001231"
+					(reference "TP17")
+					(unit 1)
+				)
+				(path "/02606b2c-b376-4ffb-9781-f9cea3f70994/c8976b66-9d7c-47d1-8ab5-e6fd9c707361/b5f91759-085b-4a53-bede-6cb17536657b"
+					(reference "TP16")
+					(unit 1)
+				)
+				(path "/02606b2c-b376-4ffb-9781-f9cea3f70994/c8976b66-9d7c-47d1-8ab5-e6fd9c707361/eb655268-f2ac-4ac0-945d-2ba286ede0a5"
+					(reference "TP15")
+					(unit 1)
+				)

Commit message: Component placement halfway done
Parts:
- removed TP13: BAT-, TestPoint:TestPoint_Plated_Hole_D2.0mm, symbol Connector:TestPoint
- added D43: LED, LED_SMD:LED_0603_1608Metric_Pad1.05x0.95mm_HandSolder, symbol Device:LED_Small
Connections:
- net at R33.1: now also D43.2 (A); no longer U11.6 (~{PG})
- new net: D43.1 (K), U11.6 (~{PG})
Changed lines of the file:
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@@
-	)
-	(junction
-		(at 181.61 111.76)
-		(diameter 0)
-		(color 0 0 0 0)
 	)
 	(junction
@@
 	(wire
 		(pts
+			(xy 161.29 92.71) (xy 166.37 92.71)
+		)
+		(stroke
+			(width 0)
+			(type default)
+		)
+	)
+	(wire
+		(pts
 			(xy 161.29 95.25) (xy 165.1 95.25)
 		)
@@
 	(wire
 		(pts
-			(xy 149.86 111.76) (xy 181.61 111.76)
-		)
-		(stroke
-			(width 0)
-			(type default)
-		)
-	)
-	(wire
-		(pts
 			(xy 179.07 96.52) (xy 186.69 96.52)
 		)
@@
 	(wire
 		(pts
-			(xy 161.29 92.71) (xy 171.45 92.71)
-		)
-		(stroke
-			(width 0)
-			(type default)
-		)
-	)
-	(wire
-		(pts
 			(xy 114.3 77.47) (xy 114.3 80.01)
 		)
@@
 	(wire
 		(pts
-			(xy 181.61 111.76) (xy 191.77 111.76)
+			(xy 149.86 111.76) (xy 191.77 111.76)
 		)
 		(stroke
@@
 				(path "/453543af-7e3c-49a0-a644-4bd49c4f86f8/eb655268-f2ac-4ac0-945d-2ba286ede0a5"
 					(reference "R28")
+					(unit 1)
+				)
+			)
+		)
+	)
+	(symbol
+		(lib_id "Device:LED_Small")
+		(at 168.91 92.71 0)
+		(unit 1)
+		(exclude_from_sim no)
+		(in_bom yes)
+		(on_board yes)
+		(dnp no)
+		(property "Reference" "D43"
+			(at 172.72 91.186 0)
+			(effects
+				(font
+					(size 1.27 1.27)
+				)
+				(justify left)
+			)
+		)
+		(property "Value" "LED"
+			(at 172.72 92.964 0)
+			(effects
+				(font
+					(size 1.27 1.27)
+				)
+				(justify left)
+			)
+		)
+		(property "Footprint" "LED_SMD:LED_0603_1608Metric_Pad1.05x0.95mm_HandSolder"
+			(at 168.91 92.71 90)
+			(effects
+				(font
+					(size 1.27 1.27)
+				)
+				(hide yes)
+			)
+		)
+		(property "Datasheet" "~"
+			(at 168.91 92.71 90)
+			(effects
+				(font
+					(size 1.27 1.27)
+				)
+				(hide yes)
+			)
+		)
+		(property "Description" ""
+			(at 168.91 92.71 0)
+			(effects
+				(font
+					(size 1.27 1.27)
+				)
+				(hide yes)
+			)
+		)
+		(property "Manufacturer" "Generic"
+			(at 168.91 92.71 0)
+			(effects
+				(font
+					(size 1.27 1.27)
+				)
+				(hide yes)
+			)
+		)
+		(property "Part #" "Generic 0603 Blue LED"
+			(at 168.91 92.71 0)
+			(effects
+				(font
+					(size 1.27 1.27)
+				)
+				(hide yes)
+			)
+		)
+		(pin "1"
+		)
+		(pin "2"
+		)
+		(instances
+			(project "rocket2-ecu"
+				(path "/02606b2c-b376-4ffb-9781-f9cea3f70994/c8976b66-9d7c-47d1-8ab5-e6fd9c707361/1a39f8df-dcec-4a97-951c-60148a5067ca"
+					(reference "D44")
+					(unit 1)
+				)
+				(path "/02606b2c-b376-4ffb-9781-f9cea3f70994/c8976b66-9d7c-47d1-8ab5-e6fd9c707361/218966e8-0599-4bad-8241-95ca09109d89"
+					(reference "D43")
+					(unit 1)
+				)
+				(path "/02606b2c-b376-4ffb-9781-f9cea3f70994/c8976b66-9d7c-47d1-8ab5-e6fd9c707361/5c1dbfcc-3925-4da2-a038-2c416606c068"
+					(reference "D48")
+					(unit 1)
+				)
+				(path "/02606b2c-b376-4ffb-9781-f9cea3f70994/c8976b66-9d7c-47d1-8ab5-e6fd9c707361/8ab1e7d4-e52f-422c-912d-30fd70001231"
+					(reference "D47")
+					(unit 1)
+				)
+				(path "/02606b2c-b376-4ffb-9781-f9cea3f70994/c8976b66-9d7c-47d1-8ab5-e6fd9c707361/b5f91759-085b-4a53-bede-6cb17536657b"
+					(reference "D46")
+					(unit 1)
+				)
+				(path "/02606b2c-b376-4ffb-9781-f9cea3f70994/c8976b66-9d7c-47d1-8ab5-e6fd9c707361/eb655268-f2ac-4ac0-945d-2ba286ede0a5"
+					(reference "D45")
 					(unit 1)
 				)
@@
 					(unit 1)
 				)
-			)
-		)
-	)
-	(symbol
-		(lib_id "Connector:TestPoint")
-		(at 181.61 111.76 180)
-		(unit 1)
-		(exclude_from_sim no)
-		(in_bom yes)
-		(on_board yes)
-		(dnp no)
-		(fields_autoplaced yes)
-		(property "Reference" "TP13"
-			(at 184.15 113.7919 0)
-			(effects
-				(font
-					(size 1.27 1.27)
-				)
-				(justify right)
-			)
-		)
-		(property "Value" "BAT-"
-			(at 184.15 116.3319 0)
-			(effects
-				(font
-					(size 1.27 1.27)
-				)
-				(justify right)
-			)
-		)
-		(property "Footprint" "TestPoint:TestPoint_Plated_Hole_D2.0mm"
-			(at 176.53 111.76 0)
-			(effects
-				(font
-					(size 1.27 1.27)
-				)
-				(hide yes)
-			)
-		)
-		(property "Datasheet" "~"
-			(at 176.53 111.76 0)
-			(effects
-				(font
-					(size 1.27 1.27)
-				)
-				(hide yes)
-			)
-		)
-		(property "Description" "test point"
-			(at 181.61 111.76 0)
-			(effects
-				(font
-					(size 1.27 1.27)
-				)
-				(hide yes)
-			)
-		)
-		(pin "1"
-		)
-		(instances
-			(project "rocket2-ecu"
-				(path "/02606b2c-b376-4ffb-9781-f9cea3f70994/c8976b66-9d7c-47d1-8ab5-e6fd9c707361/1a39f8df-dcec-4a97-951c-60148a5067ca"
-					(reference "TP14")
-					(unit 1)
-				)
-				(path "/02606b2c-b376-4ffb-9781-f9cea3f70994/c8976b66-9d7c-47d1-8ab5-e6fd9c707361/218966e8-0599-4bad-8241-95ca09109d89"
-					(reference "TP13")
-					(unit 1)
-				)
-				(path "/02606b2c-b376-4ffb-9781-f9cea3f70994/c8976b66-9d7c-47d1-8ab5-e6fd9c707361/5c1dbfcc-3925-4da2-a038-2c416606c068"
-					(reference "TP18")
-					(unit 1)
-				)
-				(path "/02606b2c-b376-4ffb-9781-f9cea3f70994/c8976b66-9d7c-47d1-8ab5-e6fd9c707361/8ab1e7d4-e52f-422c-912d-30fd70001231"
-					(reference "TP17")
-					(unit 1)
-				)
-				(path "/02606b2c-b376-4ffb-9781-f9cea3f70994/c8976b66-9d7c-47d1-8ab5-e6fd9c707361/b5f91759-085b-4a53-bede-6cb17536657b"
-					(reference "TP16")
-					(unit 1)
-				)
-				(path "/02606b2c-b376-4ffb-9781-f9cea3f70994/c8976b66-9d7c-47d1-8ab5-e6fd9c707361/eb655268-f2ac-4ac0-945d-2ba286ede0a5"
-					(reference "TP15")
-					(unit 1)
-				)

Commit message: version in PCBway 12/12/2025
Parts:
- R31: value 375 -> 500; Part # Generic RES SMD 375 OHM 0.1% 1/16W 0402 -> Generic RES SMD 500 OHM 0.1% 1/16W 0402
- U10: Part # EC4SAW-xxSxxN -> EC4SAW-24S05N
Changed lines of the file:
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@@
+		)
+	)
+	(text_box "ISET should be 375ohm, using 500 bc jlcpcb didn't have 375"
+		(exclude_from_sim no)
+		(at 119.38 114.3 0)
+		(size 7.62 3.81)
+		(margins 0.375 0.375 0.375 0.375)
+		(stroke
+			(width 0)
+			(type solid)
+		)
+		(fill
+			(type none)
+		)
+		(effects
+			(font
+				(size 0.5 0.5)
+			)
+			(justify left top)
 		)
 	)
@@
 			)
 		)
-		(property "Part #" "EC4SAW-xxSxxN"
+		(property "Part #" "EC4SAW-24S05N"
 			(at 81.915 93.98 0)
 			(effects
@@
 			)
 		)
-		(property "Value" "375"
+		(property "Value" "500"
 			(at 119.38 105.41 0)
 			(effects
@@
 			)
 		)
-		(property "Part #" "Generic RES SMD 375 OHM 0.1% 1/16W 0402"
+		(property "Part #" "Generic RES SMD 500 OHM 0.1% 1/16W 0402"
 			(at 124.46 104.14 0)
 			(effects

Commit message: added some production files
Parts:
- U12: value VOS615A-1 -> PS2811-1-F3-A; Manufacturer Vishay -> CEL; Part # VOS615A-1X001T -> PS2811-1-F3-A
Changed lines of the file:
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@@
 			)
 		)
-		(property "Value" "VOS615A-1"
+		(property "Value" "PS2811-1-F3-A"
 			(at 193.04 50.8 0)
 			(effects
@@
 			)
 		)
-		(property "Datasheet" "https://www.vishay.com/docs/85373/vos615a.pdf"
+		(property "Datasheet" "https://mm.digikey.com/Volume0/opasdata/d220001/medias/docus/2583/PS2811-1%2C%20PS2811-4%20Rev2006.pdf"
 			(at 193.04 55.88 0)
 			(effects
@@
 			)
 		)
-		(property "Manufacturer" "Vishay"
+		(property "Manufacturer" "  CEL"
 			(at 193.04 55.88 0)
 			(effects
@@
 			)
 		)
-		(property "Part #" "VOS615A-1X001T"
+		(property "Part #" "PS2811-1-F3-A"
 			(at 193.04 55.88 0)
 			(effects
